Commit message: modified:   ada.srdf 	modified:   ada_srdf.xacro

File: robots/ada_srdf.xacro (robot description, xacro)
@@ -1,17 +1,17 @@
 <robot xmlns:xacro="http://www.ros.org/wiki/xacro" name="ada">
     <group name="manipulator">
-      <chain base_link="j2n6s200_link_base" tip_link="j2n6s200_link_6/INPUT_INTERFACE"/>
+      <chain base_link="j2n6s200_link_base" tip_link="j2n6s200_link_6"/>
     </group>
     <!-- ADA self collisions -->
-    <disable_collisions link1="j2n6s200_link_base" link2="j2n6s200_link_1/INPUT_INTERFACE"/>
-    <disable_collisions link1="j2n6s200_link_1/INPUT_INTERFACE" link2="j2n6s200_link_2/INPUT_INTERFACE"/>
-    <disable_collisions link1="j2n6s200_link_2/INPUT_INTERFACE" link2="j2n6s200_link_3/INPUT_INTERFACE"/>
-    <disable_collisions link1="j2n6s200_link_3/INPUT_INTERFACE" link2="j2n6s200_link_4/INPUT_INTERFACE"/>
-    <disable_collisions link1="j2n6s200_link_4/INPUT_INTERFACE" link2="j2n6s200_link_5/INPUT_INTERFACE"/>
-    <disable_collisions link1="j2n6s200_link_5/INPUT_INTERFACE" link2="j2n6s200_link_6/INPUT_INTERFACE"/>
-    <disable_collisions link1="j2n6s200_link_6/INPUT_INTERFACE" link2="j2n6s200_end_effector/INPUT_INTERFACE"/>
+    <disable_collisions link1="j2n6s200_link_base" link2="j2n6s200_link_1"/>
+    <disable_collisions link1="j2n6s200_link_1" link2="j2n6s200_link_2"/>
+    <disable_collisions link1="j2n6s200_link_2" link2="j2n6s200_link_3"/>
+    <disable_collisions link1="j2n6s200_link_3" link2="j2n6s200_link_4"/>
+    <disable_collisions link1="j2n6s200_link_4" link2="j2n6s200_link_5"/>
+    <disable_collisions link1="j2n6s200_link_5" link2="j2n6s200_link_6"/>
+    <disable_collisions link1="j2n6s200_link_6" link2="j2n6s200_end_effector"/>
     <group name="endEffector">
-      <link name="j2n6s200_end_effector/INPUT_INTERFACE"/>
+      <link name="j2n6s200_end_effector"/>
     </group>
-    <end_effector name="end_effector" parent_link="j2n6s200_end_effector/INPUT_INTERFACE" group="endEffector"/>
+    <end_effector name="end_effector" parent_link="j2n6s200_end_effector" group="endEffector"/>
 </robot>

Commit message: added hand dofs 	modified:   ada.srdf 	modified:   ada_srdf.xacro

File: robots/ada_srdf.xacro (robot description, xacro)
@@ -14,4 +14,14 @@
       <link name="j2n6s200_end_effector"/>
     </group>
+    <group name="j2n6s200_hand">
+      <link name="j2n6s200_link_finger_1"/>
+      <link name="j2n6s200_link_finger_tip_1"/>
+      <link name="j2n6s200_link_finger_2"/>
+      <link name="j2n6s200_link_finger_tip_2"/>
+    </group>
+    <!--<group name="j2n6s200_hand">
+      <chain base_link="j2n6s200_link_finger_1" tip_link="j2n6s200_link_finger_tip_1"/>
+      <chain base_link="j2n6s200_link_finger_2" tip_link="j2n6s200_link_finger_tip_2"/>
+    </group>-->
     <end_effector name="end_effector" parent_link="j2n6s200_end_effector" group="endEffector"/>
 </robot>
