Commit message: add camera at the end of ada_accessories.urdf

File: robots/ada_accessories.urdf (robot description, URDF)
Before this commit: robot j2n6s200, 13 links, 12 joints
Links:
- added link joule; collision mesh filename=package://ada_description/meshes/camera_joule_tex.dae scale=0.001 0.001 0.00094; visual mesh filename=package://ada_description/meshes/camera_joule_tex.STL scale=0.001 0.001 0.001
Joints:
- added joint joule: type continuous, parent j2n6s200_link_6, child joule, origin xyz=0.06 0.051 0.0163 rpy=1.57079632679 1.57079632679 0, axis 0 0 1, limit lower=-6.28318530718 upper=6.28318530718 effort=2000 velocity=1

Commit message: modified:   meshes/camera_joule_tex.STL 	new file:   meshes/forque_kinova.dae 	modified:   robots/ada_accessories.urdf

File: robots/ada_accessories.urdf (robot description, URDF)
Before this commit: robot j2n6s200, 14 links, 13 joints
Links:
- removed link joule
- added link j2n6s200_joule; collision mesh filename=package://ada_description/meshes/camera_joule_tex.dae scale=0.001 0.001 0.00094; visual mesh filename=package://ada_description/meshes/camera_joule_tex.STL scale=0.001 0.001 0.001
- link j2n6s200_forque: geometry collision mesh filename=package://ada_description/meshes/forque_kinova.dae scale=0.001 0.001 0.001; visual mesh filename=package://ada_description/meshes/forque_kinova.dae scale=0.001 0.001 0.001
Joints:
- removed joint joule
- added joint j2n6s200_joule: type continuous, parent j2n6s200_link_6, child j2n6s200_joule, origin xyz=0.06 0.051 0.0163 rpy=1.57079632679 1.57079632679 0, axis 0 0 1, limit lower=-6.28318530718 upper=6.28318530718 effort=2000 velocity=1
- joint j2n6s200_joint_forque: parent j2n6s200_end_effector -> j2n6s200_link_6

Commit message: minor changes to forque urdf

File: robots/ada_accessories.urdf (robot description, URDF)
Before this commit: robot j2n6s200, 14 links, 13 joints
Joints:
- joint j2n6s200_joint_finger_1: origin xyz=-0.0025 0.03095 -0.11482 rpy=-1.570796327 .649262481663582 1.57079632679490 -> xyz=-0.0025 0.03095 -0.11482 rpy=-1.570796327 1.75 1.57079632679490
- joint j2n6s200_joint_finger_2: origin xyz=-0.0025 -0.03095 -0.11482 rpy=-1.570796327 .649262481663582 -1.57079632679490 -> xyz=-0.0025 -0.03095 -0.11482 rpy=-1.570796327 1.75 -1.57079632679490
- joint j2n6s200_joint_forque: origin xyz=0.044 -0.003 0 rpy=0 0 0 -> xyz=-0.001 -0.000 0.09 rpy=3.14 0 0; parent j2n6s200_link_6 -> j2n6s200_end_effector

Commit message: adapted robot accessories so that planning works

File: robots/ada_accessories.urdf (robot description, URDF)
Before this commit: robot j2n6s200, 14 links, 13 joints
Links:
- added link j2n6s200_forque_end_effector; visual box size=0.0001 0.0001 0.0001
- link j2n6s200_forque: geometry visual mesh filename=package://ada_description/meshes/forque_kinova.dae scale=0.001 0.001 0.001
- link j2n6s200_joule: geometry visual mesh filename=package://ada_description/meshes/camera_joule_tex.STL scale=0.001 0.001 0.001
Joints:
- added joint j2n6s200_joint_forque_end_effector: type fixed, parent j2n6s200_forque, child j2n6s200_forque_end_effector, origin xyz=0 0 -0.1 rpy=3.1415 0 0, axis 0 0 0, limit lower=0 upper=0 effort=2000 velocity=1
- joint j2n6s200_joule: type continuous -> fixed

Commit message: disabled collision for forque and joule

File: robots/ada_accessories.urdf (robot description, URDF)
Before this commit: robot j2n6s200, 15 links, 14 joints
Joints:
- joint j2n6s200_joule: origin xyz=0.06 0.051 0.0163 rpy=1.57079632679 1.57079632679 0 -> xyz=-0.06 -0.051 -0.0163 rpy=-1.57079632679 1.57079632679 0

Commit message: reenabled collision for forque and camera

File: robots/ada_accessories.urdf (robot description, URDF)
Before this commit: robot j2n6s200, 15 links, 14 joints
Links:
- link j2n6s200_forque: geometry collision mesh filename=package://ada_description/meshes/forque_kinova.dae scale=0.001 0.001 0.001; visual mesh filename=package://ada_description/meshes/forque_kinova.dae scale=0.001 0.001 0.001
- link j2n6s200_joule: geometry collision mesh filename=package://ada_description/meshes/camera_joule_tex.dae scale=0.001 0.001 0.00094; visual mesh filename=package://ada_description/meshes/camera_joule_tex.STL scale=0.001 0.001 0.001

Commit message: colors for ada rings

File: robots/ada_accessories.urdf (robot description, URDF)
Before this commit: robot j2n6s200, 15 links, 14 joints
Links:
- link j2n6s200_link_1: geometry collision mesh filename=package://ada_description/meshes/shoulder.dae; visual mesh filename=package://ada_description/meshes/ring_big.dae
- link j2n6s200_link_2: geometry collision mesh filename=package://ada_description/meshes/arm.dae; visual mesh filename=package://ada_description/meshes/arm.dae
- link j2n6s200_link_3: geometry collision mesh filename=package://ada_description/meshes/forearm.dae; visual mesh filename=package://ada_description/meshes/forearm.dae
- link j2n6s200_link_4: geometry collision mesh filename=package://ada_description/meshes/wrist.dae; visual mesh filename=package://ada_description/meshes/ring_small.dae
- link j2n6s200_link_5: geometry collision mesh filename=package://ada_description/meshes/wrist.dae; visual mesh filename=package://ada_description/meshes/ring_small.dae
- link j2n6s200_link_6: geometry collision mesh filename=package://ada_description/meshes/hand_2finger.dae; visual mesh filename=package://ada_description/meshes/hand_2finger.dae
