Commit message: some changes to urdf and srdf with different models for different accessories

File: robots/ada_with_camera.urdf (robot description, URDF)
Before this commit: robot j2n6s200, 12 links, 11 joints
Links:
- added link j2n6s200_joule; collision mesh filename=package://ada_description/meshes/camera_joule_tex.dae scale=0.001 0.001 0.00094; visual mesh filename=package://ada_description/meshes/camera_joule_tex.STL scale=0.001 0.001 0.001
Joints:
- added joint j2n6s200_joule: type fixed, parent j2n6s200_link_6, child j2n6s200_joule, origin xyz=-0.06 -0.051 -0.0163 rpy=-1.57079632679 1.57079632679 0, axis 0 0 1, limit lower=-6.28318530718 upper=6.28318530718 effort=2000 velocity=1

File: robots/ada_with_camera_forque.urdf (robot description, URDF)
Before this commit: robot j2n6s200, 12 links, 11 joints
Links:
- added link j2n6s200_forque; collision mesh filename=package://ada_description/meshes/collision_forque_kinova.dae scale=0.001 0.001 0.001; visual mesh filename=package://ada_description/meshes/forque_kinova.dae scale=0.001 0.001 0.001
- added link j2n6s200_forque_end_effector; visual box size=0.0001 0.0001 0.0001
- added link j2n6s200_joule; collision mesh filename=package://ada_description/meshes/camera_joule_tex.dae scale=0.001 0.001 0.00094; visual mesh filename=package://ada_description/meshes/camera_joule_tex.STL scale=0.001 0.001 0.001
Joints:
- added joint j2n6s200_joint_forque: type fixed, parent j2n6s200_end_effector, child j2n6s200_forque, origin xyz=-0.001 -0.000 0.09 rpy=3.14 0 0, axis 0 0 1, limit lower=0 upper=2 effort=2000 velocity=1
- added joint j2n6s200_joint_forque_end_effector: type fixed, parent j2n6s200_forque, child j2n6s200_forque_end_effector, origin xyz=0 0 -0.1 rpy=3.1415 0 0, axis 0 0 0, limit lower=0 upper=0 effort=2000 velocity=1
- added joint j2n6s200_joule: type fixed, parent j2n6s200_link_6, child j2n6s200_joule, origin xyz=-0.06 -0.051 -0.0163 rpy=-1.57079632679 1.57079632679 0, axis 0 0 1, limit lower=-6.28318530718 upper=6.28318530718 effort=2000 velocity=1
- joint j2n6s200_joint_finger_1: origin xyz=-0.0025 0.03095 -0.11482 rpy=-1.570796327 .649262481663582 1.57079632679490 -> xyz=-0.0025 0.03095 -0.11482 rpy=-1.570796327 1.75 1.57079632679490
- joint j2n6s200_joint_finger_2: origin xyz=-0.0025 -0.03095 -0.11482 rpy=-1.570796327 .649262481663582 -1.57079632679490 -> xyz=-0.0025 -0.03095 -0.11482 rpy=-1.570796327 1.75 -1.57079632679490
