Commit message: modified:   ada.urdf 	modified:   ada_urdf.xacro 	modified:   kinova_common.xacro

File: robots/ada.urdf (robot description, URDF)
Before this commit: robot j2n6s200, 14 links, 13 joints
Links:
- link j2n6s200_end_effector: geometry collision box size=0.01 0.01 0.01; visual box size=0.01 0.01 0.01
- link root: geometry collision box size=0.01 0.01 0.01; visual box size=0.01 0.01 0.01

File: robots/ada_urdf.xacro (robot description, xacro)
@@ -19,5 +19,5 @@
       <origin xyz="0 0 0" rpy="0 0 0" />
       <geometry>
-        <box size = "0 0 0"/>
+        <box size = "0.01 0.01 0.01"/>
       </geometry>
     <!--<material name="Black" /> -->
@@ -26,5 +26,5 @@
       <origin xyz="0 0 0" rpy="0 0 0" />
       <geometry>
-        <box size = "0 0 0"/>
+        <box size = "0.01 0.01 0.01"/>
       </geometry>
     </collision>

File: robots/kinova_common.xacro (robot description, xacro)
@@ -70,10 +70,10 @@
             <visual>
                 <geometry>
-                    <box size = "0 0 0"/>
+                    <box size = "0.01 0.01 0.01"/>
                 </geometry>
             </visual>
             <collision>
                 <geometry>
-                    <box size = "0 0 0"/>
+                    <box size = "0.01 0.01 0.01"/>
                 </geometry>
             </collision>

Commit message: On branch robot 	modified:   ada.urdf 	modified:   ada_urdf.xacro 	modified:   kinova_common.xacro

File: robots/ada.urdf (robot description, URDF)
Before this commit: robot j2n6s200, 14 links, 13 joints
Links:
- link j2n6s200_end_effector: geometry collision box size=0.01 0.01 0.01; visual box size=0.0001 0.0001 0.0001
- link root: geometry collision box size=0.01 0.01 0.01; visual box size=0.0001 0.0001 0.0001

File: robots/ada_urdf.xacro (robot description, xacro)
@@ -19,5 +19,5 @@
       <origin xyz="0 0 0" rpy="0 0 0" />
       <geometry>
-        <box size = "0.01 0.01 0.01"/>
+        <box size = "0.0001 0.0001 0.0001"/>
       </geometry>
     <!--<material name="Black" /> -->

File: robots/kinova_common.xacro (robot description, xacro)
@@ -70,5 +70,5 @@
             <visual>
                 <geometry>
-                    <box size = "0.01 0.01 0.01"/>
+                    <box size = "0.0001 0.0001 0.0001"/>
                 </geometry>
             </visual>

Commit message: changes to the urdf and srdf and cleaned it up..

File: robots/ada.urdf (robot description, URDF)
Before this commit: robot j2n6s200, 14 links, 13 joints
Links:
- removed link root
- removed link world
Joints:
- removed joint connect_root_and_world

Commit message: minor changes to the urdf 	deleted:    README.txt 	modified:   ada.urdf

File: robots/ada.urdf (robot description, URDF)
Before this commit: robot j2n6s200, 12 links, 12 joints
Joints:
- removed joint j2n6s200_joint_base

Commit message: change URDF to finger-distal joints to revolute

File: robots/ada.urdf (robot description, URDF)
Before this commit: robot j2n6s200, 12 links, 11 joints
Joints:
- joint j2n6s200_joint_finger_tip_1: type fixed -> revolute
- joint j2n6s200_joint_finger_tip_2: type fixed -> revolute

Commit message: Set joint limits

File: robots/ada.urdf (robot description, URDF)
Before this commit: robot j2n6s200, 12 links, 11 joints
Joints:
- joint j2n6s200_joint_1: limit lower=-6.28318530718 upper=6.28318530718 effort=2000 velocity=1 -> lower=-3.141592 upper=3.141592 effort=2000 velocity=1
- joint j2n6s200_joint_2: limit lower=0.820304748437 upper=5.46288055874 effort=2000 velocity=1 -> lower=-3.8451785 upper=0.7035858 effort=2000 velocity=1
- joint j2n6s200_joint_3: limit lower=0.331612557879 upper=5.9515727493 effort=2000 velocity=1 -> lower=-4.104090 upper=0.9515727493 effort=2000 velocity=1
- joint j2n6s200_joint_4: limit lower=-6.28318530718 upper=6.28318530718 effort=2000 velocity=1 -> lower=-3.141592 upper=3.141592 effort=2000 velocity=1
- joint j2n6s200_joint_5: limit lower=-6.28318530718 upper=6.28318530718 effort=2000 velocity=1 -> lower=-3.141592 upper=3.141592 effort=2000 velocity=1
- joint j2n6s200_joint_6: limit lower=-6.28318530718 upper=6.28318530718 effort=2000 velocity=1 -> lower=-3.141592 upper=3.141592 effort=2000 velocity=1

Commit message: Forque added to mesh and urdf

File: robots/ada.urdf (robot description, URDF)
Before this commit: robot j2n6s200, 12 links, 11 joints
Links:
- added link j2n6s200_forque; collision mesh filename=package://ada_description/meshes/forque_kinova.STL; visual mesh filename=package://ada_description/meshes/forque_kinova.STL
Joints:
- added joint j2n6s200_joint_forque: type fixed, parent j2n6s200_end_effector, child j2n6s200_forque, origin xyz=0.044 -0.003 0 rpy=0 0 0, axis 0 0 1, limit lower=0 upper=2 effort=2000 velocity=1

Commit message: ring color and camera for ada without accessories

File: robots/ada.urdf (robot description, URDF)
Before this commit: robot j2n6s200, 12 links, 11 joints
Links:
- added link j2n6s200_joule; collision mesh filename=package://ada_description/meshes/camera_joule_tex.dae scale=0.001 0.001 0.00094; visual mesh filename=package://ada_description/meshes/camera_joule_tex.STL scale=0.001 0.001 0.001
- link j2n6s200_link_1: geometry collision mesh filename=package://ada_description/meshes/shoulder.dae; visual mesh filename=package://ada_description/meshes/ring_big.dae
- link j2n6s200_link_2: geometry collision mesh filename=package://ada_description/meshes/arm.dae; visual mesh filename=package://ada_description/meshes/arm.dae
- link j2n6s200_link_3: geometry collision mesh filename=package://ada_description/meshes/forearm.dae; visual mesh filename=package://ada_description/meshes/forearm.dae
- link j2n6s200_link_4: geometry collision mesh filename=package://ada_description/meshes/wrist.dae; visual mesh filename=package://ada_description/meshes/ring_small.dae
- link j2n6s200_link_5: geometry collision mesh filename=package://ada_description/meshes/wrist.dae; visual mesh filename=package://ada_description/meshes/ring_small.dae
- link j2n6s200_link_6: geometry collision mesh filename=package://ada_description/meshes/hand_2finger.dae; visual mesh filename=package://ada_description/meshes/hand_2finger.dae
Joints:
- added joint j2n6s200_joule: type fixed, parent j2n6s200_link_6, child j2n6s200_joule, origin xyz=-0.06 -0.051 -0.0163 rpy=-1.57079632679 1.57079632679 0, axis 0 0 1, limit lower=-6.28318530718 upper=6.28318530718 effort=2000 velocity=1

Commit message: simpler collision meshes for ada

File: robots/ada.urdf (robot description, URDF)
Before this commit: robot j2n6s200, 13 links, 12 joints
Links:
- link j2n6s200_link_1: geometry collision mesh filename=package://ada_description/meshes/collision_shoulder.dae; visual mesh filename=package://ada_description/meshes/ring_big.dae
- link j2n6s200_link_2: geometry collision mesh filename=package://ada_description/meshes/collision_arm.dae; visual mesh filename=package://ada_description/meshes/arm.dae
- link j2n6s200_link_3: geometry collision mesh filename=package://ada_description/meshes/collision_forearm.dae; visual mesh filename=package://ada_description/meshes/forearm.dae
- link j2n6s200_link_4: geometry collision mesh filename=package://ada_description/meshes/collision_wrist.dae; visual mesh filename=package://ada_description/meshes/ring_small.dae
- link j2n6s200_link_5: geometry collision mesh filename=package://ada_description/meshes/collision_wrist.dae; visual mesh filename=package://ada_description/meshes/ring_small.dae
- link j2n6s200_link_6: geometry collision mesh filename=package://ada_description/meshes/collision_hand_2finger.dae; visual mesh filename=package://ada_description/meshes/hand_2finger.dae
- link j2n6s200_link_base: geometry collision mesh filename=package://ada_description/meshes/collision_base.dae; visual mesh filename=package://ada_description/meshes/base.dae
- link j2n6s200_link_finger_1: geometry collision mesh filename=package://ada_description/meshes/collision_finger_proximal.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; visual mesh filename=package://ada_description/meshes/finger_proximal.dae
- link j2n6s200_link_finger_2: geometry collision mesh filename=package://ada_description/meshes/collision_finger_proximal.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; visual mesh filename=package://ada_description/meshes/finger_proximal.dae
- link j2n6s200_link_finger_tip_1: geometry collision mesh filename=package://ada_description/meshes/collision_finger_distal.dae; visual mesh filename=package://ada_description/meshes/finger_distal.dae
- link j2n6s200_link_finger_tip_2: geometry collision mesh filename=package://ada_description/meshes/collision_finger_distal.dae; visual mesh filename=package://ada_description/meshes/finger_distal.dae

File: robots/ada_accessories.urdf (robot description, URDF)
Before this commit: robot j2n6s200, 15 links, 14 joints
Links:
- link j2n6s200_forque: geometry collision mesh filename=package://ada_description/meshes/collision_forque_kinova.dae scale=0.001 0.001 0.001; visual mesh filename=package://ada_description/meshes/forque_kinova.dae scale=0.001 0.001 0.001
- link j2n6s200_link_1: geometry collision mesh filename=package://ada_description/meshes/collision_shoulder.dae; visual mesh filename=package://ada_description/meshes/ring_big.dae
- link j2n6s200_link_2: geometry collision mesh filename=package://ada_description/meshes/collision_arm.dae; visual mesh filename=package://ada_description/meshes/arm.dae
- link j2n6s200_link_3: geometry collision mesh filename=package://ada_description/meshes/collision_forearm.dae; visual mesh filename=package://ada_description/meshes/forearm.dae
- link j2n6s200_link_4: geometry collision mesh filename=package://ada_description/meshes/collision_wrist.dae; visual mesh filename=package://ada_description/meshes/ring_small.dae
- link j2n6s200_link_5: geometry collision mesh filename=package://ada_description/meshes/collision_wrist.dae; visual mesh filename=package://ada_description/meshes/ring_small.dae
- link j2n6s200_link_6: geometry collision mesh filename=package://ada_description/meshes/collision_hand_2finger.dae; visual mesh filename=package://ada_description/meshes/hand_2finger.dae
- link j2n6s200_link_base: geometry collision mesh filename=package://ada_description/meshes/collision_base.dae; visual mesh filename=package://ada_description/meshes/base.dae
- link j2n6s200_link_finger_1: geometry collision mesh filename=package://ada_description/meshes/collision_finger_proximal.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; visual mesh filename=package://ada_description/meshes/finger_proximal.dae
- link j2n6s200_link_finger_2: geometry collision mesh filename=package://ada_description/meshes/collision_finger_proximal.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; visual mesh filename=package://ada_description/meshes/finger_proximal.dae
- link j2n6s200_link_finger_tip_1: geometry collision mesh filename=package://ada_description/meshes/collision_finger_distal.dae; visual mesh filename=package://ada_description/meshes/finger_distal.dae
- link j2n6s200_link_finger_tip_2: geometry collision mesh filename=package://ada_description/meshes/collision_finger_distal.dae; visual mesh filename=package://ada_description/meshes/finger_distal.dae

Commit message: Add hand base to urdf

File: robots/ada.urdf (robot description, URDF)
Before this commit: robot j2n6s200, 14 links, 13 joints
Links:
- added link j2n6s200_hand_base
- link j2n6s200_end_effector: geometry 
Joints:
- added joint j2n6s200_joint_hand_base: type fixed, parent j2n6s200_link_6, child j2n6s200_hand_base, origin xyz=0 0 0 rpy=0 0 0, axis 0 0 0
- joint j2n6s200_joint_finger_1: parent j2n6s200_link_6 -> j2n6s200_hand_base
- joint j2n6s200_joint_finger_2: parent j2n6s200_link_6 -> j2n6s200_hand_base

Commit message: Fix urdf joint limits

File: robots/ada.urdf (robot description, URDF)
Before this commit: robot j2n6s200, 14 links, 13 joints
Joints:
- joint j2n6s200_joint_2: limit lower=-3.8451785 upper=0.7035858 effort=2000 velocity=1 -> lower=0.82030474843 upper=5.46288055874 effort=2000 velocity=1
- joint j2n6s200_joint_3: limit lower=-4.104090 upper=0.9515727493 effort=2000 velocity=1 -> lower=0.33161255787 upper=5.9515727493 effort=2000 velocity=1
- joint j2n6s200_joint_finger_tip_1: type revolute -> fixed
- joint j2n6s200_joint_finger_tip_2: type revolute -> fixed
