Commit message: added hand_base to ada with camera forque

File: robots/ada_with_camera_forque.urdf (robot description, URDF)
Before this commit: robot j2n6s200, 15 links, 14 joints
Links:
- added link j2n6s200_hand_base
- added link world
- link j2n6s200_end_effector: geometry 
- link j2n6s200_forque_end_effector: geometry 
Joints:
- added joint j2n6s200_joint_base: type fixed, parent world, child j2n6s200_link_base, origin xyz=0 0 0 rpy=0 0 0
- added joint j2n6s200_joint_hand_base: type fixed, parent j2n6s200_link_6, child j2n6s200_hand_base, origin xyz=0 0 0 rpy=0 0 0, axis 0 0 0
- joint j2n6s200_joint_finger_1: parent j2n6s200_link_6 -> j2n6s200_hand_base
- joint j2n6s200_joint_finger_2: limit lower=0 upper=2 effort=2000 velocity=1 -> lower=0 upper=2 effort=0 velocity=1; parent j2n6s200_link_6 -> j2n6s200_hand_base
- joint j2n6s200_joint_finger_tip_1: limit lower=0 upper=2 effort=2000 velocity=1 -> lower=0 upper=2 effort=0 velocity=1

Commit message: Revert changes on camera_forque

File: robots/ada_with_camera_forque.urdf (robot description, URDF)
Before this commit: robot j2n6s200, 17 links, 16 joints
Links:
- removed link j2n6s200_hand_base
- removed link world
- link j2n6s200_end_effector: geometry collision box size=0.01 0.01 0.01; visual box size=0.0001 0.0001 0.0001
- link j2n6s200_forque_end_effector: geometry visual box size=0.0001 0.0001 0.0001
Joints:
- removed joint j2n6s200_joint_base
- removed joint j2n6s200_joint_hand_base
- joint j2n6s200_joint_finger_1: parent j2n6s200_hand_base -> j2n6s200_link_6
- joint j2n6s200_joint_finger_2: limit lower=0 upper=2 effort=0 velocity=1 -> lower=0 upper=2 effort=2000 velocity=1; parent j2n6s200_hand_base -> j2n6s200_link_6
- joint j2n6s200_joint_finger_tip_1: limit lower=0 upper=2 effort=0 velocity=1 -> lower=0 upper=2 effort=2000 velocity=1

Commit message: gilwoos joint limits update

File: robots/ada_with_camera_forque.urdf (robot description, URDF)
Before this commit: robot j2n6s200, 17 links, 16 joints
Joints:
- joint j2n6s200_joint_3: limit lower=-4.104090 upper=0.9515727493 effort=2000 velocity=1 -> lower=0.33161255787 upper=5.9515727493 effort=2000 velocity=1
- joint j2n6s200_joint_finger_2: type revolute -> fixed
- joint j2n6s200_joint_finger_tip_1: type revolute -> fixed

Commit message: corrected small stuff

File: robots/ada_with_camera_forque.urdf (robot description, URDF)
Before this commit: robot j2n6s200, 17 links, 16 joints
Joints:
- joint j2n6s200_joint_finger_1: origin xyz=-0.0025 0.03095 -0.11482 rpy=-1.570796327 1.75 1.57079632679490 -> xyz=-0.0025 0.03095 -0.11482 rpy=-1.570796327 .649262481663582 1.57079632679490
- joint j2n6s200_joint_finger_2: limit lower=0 upper=2 effort=0 velocity=1 -> lower=0 upper=2 effort=2000 velocity=1; origin xyz=-0.0025 -0.03095 -0.11482 rpy=-1.570796327 1.75 -1.57079632679490 -> xyz=-0.0025 -0.03095 -0.11482 rpy=-1.570796327 .649262481663582 -1.57079632679490; type fixed -> revolute
- joint j2n6s200_joint_finger_tip_2: limit lower=0 upper=2 effort=2000 velocity=1 -> lower=0 upper=2 effort=0 velocity=1; type revolute -> fixed

Commit message: corrections

File: robots/ada_with_camera_forque.urdf (robot description, URDF)
Before this commit: robot j2n6s200, 17 links, 16 joints
Joints:
- joint j2n6s200_joint_2: limit lower=-3.8451785 upper=0.7035858 effort=2000 velocity=1 -> lower=0.82030474843 upper=5.46288055874 effort=2000 velocity=1
- joint j2n6s200_joint_base: type floating -> fixed

Commit message: quick hack joint limits

File: robots/ada_with_camera_forque.urdf (robot description, URDF)
Before this commit: robot j2n6s200, 17 links, 16 joints
Joints:
- joint j2n6s200_joint_1: limit lower=-3.141592 upper=3.141592 effort=2000 velocity=1 -> lower=-10 upper=10 effort=2000 velocity=1; type continuous -> revolute
- joint j2n6s200_joint_4: limit lower=-3.141592 upper=3.141592 effort=2000 velocity=1 -> lower=-10 upper=10 effort=2000 velocity=1; type continuous -> revolute
- joint j2n6s200_joint_5: limit lower=-3.141592 upper=3.141592 effort=2000 velocity=1 -> lower=-10 upper=10 effort=2000 velocity=1; type continuous -> revolute
- joint j2n6s200_joint_6: limit lower=-3.141592 upper=3.141592 effort=2000 velocity=1 -> lower=-10 upper=10 effort=2000 velocity=1; type continuous -> revolute
