Commit message: changed forque end effector offset

File: robots/forque.xacro (robot description, xacro)
@@ -33,5 +33,15 @@
       <axis xyz="0 0 0"/>
       <limit effort="2000" lower="0" upper="0" velocity="1"/>
-      <origin rpy="3.1415 0 0" xyz="0 0 -0.1"/>
+      <origin rpy="3.1415 0 0" xyz="0 -0.007 -0.093"/>
+      <!-- Rotation consistent with pointers of forque: -->
+      <!-- <origin rpy="2.6415 0 0" xyz="0 -0.007 -0.093"/> -->
+    </joint>
+    <link name="j2n6s200_forque_tip">
+  </link>
+    <joint name="j2n6s200_joint_forque_tip" type="fixed">
+      <parent link="j2n6s200_forque"/>
+      <child link="j2n6s200_forque_tip"/>
+      <axis xyz="0 0 0"/>
+      <limit effort="2000" lower="0" upper="0" velocity="1"/>
     </joint>
   </xacro:macro>

File: robots_urdf/ada_with_camera_forque.urdf (robot description, URDF)
Before this commit: robot j2n6s200, 17 links, 16 joints
Links:
- added link j2n6s200_forque_tip
Joints:
- added joint j2n6s200_joint_forque_tip: type fixed, parent j2n6s200_forque, child j2n6s200_forque_tip, axis 0 0 0, limit lower=0 upper=0 effort=2000 velocity=1
- joint j2n6s200_joint_forque_end_effector: origin xyz=0 0 -0.1 rpy=3.1415 0 0 -> xyz=0 -0.007 -0.093 rpy=3.1415 0 0

File: robots_urdf/ada_with_forque.urdf (robot description, URDF)
Before this commit: robot j2n6s200, 16 links, 15 joints
Links:
- added link j2n6s200_forque_tip
Joints:
- added joint j2n6s200_joint_forque_tip: type fixed, parent j2n6s200_forque, child j2n6s200_forque_tip, axis 0 0 0, limit lower=0 upper=0 effort=2000 velocity=1
- joint j2n6s200_joint_forque_end_effector: origin xyz=0 0 -0.1 rpy=3.1415 0 0 -> xyz=0 -0.007 -0.093 rpy=3.1415 0 0

Commit message: fixed the forque's frame

File: robots/forque.xacro (robot description, xacro)
@@ -23,5 +23,5 @@
       <child link="j2n6s200_forque"/>
       <axis xyz="0 0 1"/>
-      <origin rpy="3.14 0 0" xyz="-0.001 -0.000 0.09"/>
+      <origin rpy="3.14 0 0" xyz="-0.003 -0.000 0.078"/>
       <limit effort="2000" lower="0" upper="2" velocity="1"/>
     </joint>
@@ -34,6 +34,4 @@
       <limit effort="2000" lower="0" upper="0" velocity="1"/>
       <origin rpy="3.1415 0 0" xyz="0 -0.007 -0.093"/>
-      <!-- Rotation consistent with pointers of forque: -->
-      <!-- <origin rpy="2.6415 0 0" xyz="0 -0.007 -0.093"/> -->
     </joint>
     <link name="j2n6s200_forque_tip">
@@ -44,4 +42,6 @@
       <axis xyz="0 0 0"/>
       <limit effort="2000" lower="0" upper="0" velocity="1"/>
+      <!-- Rotation consistent with pointers of forque: -->
+      <origin rpy="2.6415 0 0" xyz="0 -0.007 -0.093"/>
     </joint>
   </xacro:macro>

File: robots_urdf/ada_with_camera_forque.urdf (robot description, URDF)
Before this commit: robot j2n6s200, 19 links, 18 joints
Joints:
- joint j2n6s200_joint_forque: origin xyz=-0.001 -0.000 0.09 rpy=3.14 0 0 -> xyz=-0.003 -0.000 0.078 rpy=3.14 0 0
- joint j2n6s200_joint_forque_tip: origin (none) -> xyz=0 -0.007 -0.093 rpy=2.6415 0 0

File: robots_urdf/ada_with_forque.urdf (robot description, URDF)
Before this commit: robot j2n6s200, 18 links, 17 joints
Joints:
- joint j2n6s200_joint_forque: origin xyz=-0.001 -0.000 0.09 rpy=3.14 0 0 -> xyz=-0.003 -0.000 0.078 rpy=3.14 0 0
- joint j2n6s200_joint_forque_tip: origin (none) -> xyz=0 -0.007 -0.093 rpy=2.6415 0 0

Commit message: translated forque to match model in camera

File: robots/forque.xacro (robot description, xacro)
@@ -23,5 +23,5 @@
       <child link="j2n6s200_forque"/>
       <axis xyz="0 0 1"/>
-      <origin rpy="3.14 0 0" xyz="-0.003 -0.000 0.078"/>
+      <origin rpy="3.14 0 0" xyz="0.01 -0.000 0.078"/>
       <limit effort="2000" lower="0" upper="2" velocity="1"/>
     </joint>
@@ -33,5 +33,5 @@
       <axis xyz="0 0 0"/>
       <limit effort="2000" lower="0" upper="0" velocity="1"/>
-      <origin rpy="3.1415 0 0" xyz="0 -0.007 -0.093"/>
+      <origin rpy="3.1415 0 1.57075" xyz="0.007 0 -0.093"/>
     </joint>
     <link name="j2n6s200_forque_tip">
@@ -43,5 +43,5 @@
       <limit effort="2000" lower="0" upper="0" velocity="1"/>
       <!-- Rotation consistent with pointers of forque: -->
-      <origin rpy="2.6415 0 0" xyz="0 -0.007 -0.093"/>
+      <origin rpy="2.6415 0 1.57075" xyz="0.007 0 -0.093"/>
     </joint>
   </xacro:macro>

File: robots/kinova_common.xacro (robot description, xacro)
@@ -38,5 +38,5 @@
         <child link="${child}"/>
         <axis xyz="${joint_axis_xyz}"/>
-        <limit effort="2000" velocity="1.5" lower="${joint_lower_limit}" upper="${joint_upper_limit}"/>
+        <limit effort="2000" velocity="0.8" lower="${joint_lower_limit}" upper="${joint_upper_limit}"/>
         <origin xyz="${joint_origin_xyz}" rpy="${joint_origin_rpy}"/>
         <dynamics damping="0.0" friction="0.0"/>

File: robots_urdf/ada.urdf (robot description, URDF)
Before this commit: robot j2n6s200, 15 links, 14 joints
Joints:
- joint j2n6s200_joint_1: limit lower=-6.28318530718 upper=6.28318530718 effort=2000 velocity=1.5 -> lower=-6.28318530718 upper=6.28318530718 effort=2000 velocity=0.8
- joint j2n6s200_joint_2: limit lower=0.820304748437 upper=5.46288055874 effort=2000 velocity=1.5 -> lower=0.820304748437 upper=5.46288055874 effort=2000 velocity=0.8
- joint j2n6s200_joint_3: limit lower=0.331612557879 upper=5.9515727493 effort=2000 velocity=1.5 -> lower=0.331612557879 upper=5.9515727493 effort=2000 velocity=0.8
- joint j2n6s200_joint_4: limit lower=-6.28318530718 upper=6.28318530718 effort=2000 velocity=1.5 -> lower=-6.28318530718 upper=6.28318530718 effort=2000 velocity=0.8
- joint j2n6s200_joint_5: limit lower=-6.28318530718 upper=6.28318530718 effort=2000 velocity=1.5 -> lower=-6.28318530718 upper=6.28318530718 effort=2000 velocity=0.8
- joint j2n6s200_joint_6: limit lower=-6.28318530718 upper=6.28318530718 effort=2000 velocity=1.5 -> lower=-6.28318530718 upper=6.28318530718 effort=2000 velocity=0.8
- joint j2n6s200_joint_base: limit lower=0 upper=0 effort=2000 velocity=1.5 -> lower=0 upper=0 effort=2000 velocity=0.8

File: robots_urdf/ada_with_camera.urdf (robot description, URDF)
Before this commit: robot j2n6s200, 16 links, 15 joints
Joints:
- joint j2n6s200_joint_1: limit lower=-6.28318530718 upper=6.28318530718 effort=2000 velocity=1.5 -> lower=-6.28318530718 upper=6.28318530718 effort=2000 velocity=0.8
- joint j2n6s200_joint_2: limit lower=0.820304748437 upper=5.46288055874 effort=2000 velocity=1.5 -> lower=0.820304748437 upper=5.46288055874 effort=2000 velocity=0.8
- joint j2n6s200_joint_3: limit lower=0.331612557879 upper=5.9515727493 effort=2000 velocity=1.5 -> lower=0.331612557879 upper=5.9515727493 effort=2000 velocity=0.8
- joint j2n6s200_joint_4: limit lower=-6.28318530718 upper=6.28318530718 effort=2000 velocity=1.5 -> lower=-6.28318530718 upper=6.28318530718 effort=2000 velocity=0.8
- joint j2n6s200_joint_5: limit lower=-6.28318530718 upper=6.28318530718 effort=2000 velocity=1.5 -> lower=-6.28318530718 upper=6.28318530718 effort=2000 velocity=0.8
- joint j2n6s200_joint_6: limit lower=-6.28318530718 upper=6.28318530718 effort=2000 velocity=1.5 -> lower=-6.28318530718 upper=6.28318530718 effort=2000 velocity=0.8
- joint j2n6s200_joint_base: limit lower=0 upper=0 effort=2000 velocity=1.5 -> lower=0 upper=0 effort=2000 velocity=0.8

File: robots_urdf/ada_with_camera_forque.urdf (robot description, URDF)
Before this commit: robot j2n6s200, 19 links, 18 joints
Joints:
- joint j2n6s200_joint_1: limit lower=-6.28318530718 upper=6.28318530718 effort=2000 velocity=1.5 -> lower=-6.28318530718 upper=6.28318530718 effort=2000 velocity=0.8
- joint j2n6s200_joint_2: limit lower=0.820304748437 upper=5.46288055874 effort=2000 velocity=1.5 -> lower=0.820304748437 upper=5.46288055874 effort=2000 velocity=0.8
- joint j2n6s200_joint_3: limit lower=0.331612557879 upper=5.9515727493 effort=2000 velocity=1.5 -> lower=0.331612557879 upper=5.9515727493 effort=2000 velocity=0.8
- joint j2n6s200_joint_4: limit lower=-6.28318530718 upper=6.28318530718 effort=2000 velocity=1.5 -> lower=-6.28318530718 upper=6.28318530718 effort=2000 velocity=0.8
- joint j2n6s200_joint_5: limit lower=-6.28318530718 upper=6.28318530718 effort=2000 velocity=1.5 -> lower=-6.28318530718 upper=6.28318530718 effort=2000 velocity=0.8
- joint j2n6s200_joint_6: limit lower=-6.28318530718 upper=6.28318530718 effort=2000 velocity=1.5 -> lower=-6.28318530718 upper=6.28318530718 effort=2000 velocity=0.8
- joint j2n6s200_joint_base: limit lower=0 upper=0 effort=2000 velocity=1.5 -> lower=0 upper=0 effort=2000 velocity=0.8
- joint j2n6s200_joint_forque: origin xyz=-0.003 -0.000 0.078 rpy=3.14 0 0 -> xyz=0.01 -0.000 0.078 rpy=3.14 0 0
- joint j2n6s200_joint_forque_end_effector: origin xyz=0 -0.007 -0.093 rpy=3.1415 0 0 -> xyz=0.007 0 -0.093 rpy=3.1415 0 1.57075
- joint j2n6s200_joint_forque_tip: origin xyz=0 -0.007 -0.093 rpy=2.6415 0 0 -> xyz=0.007 0 -0.093 rpy=2.6415 0 1.57075

File: robots_urdf/ada_with_forque.urdf (robot description, URDF)
Before this commit: robot j2n6s200, 18 links, 17 joints
Joints:
- joint j2n6s200_joint_1: limit lower=-6.28318530718 upper=6.28318530718 effort=2000 velocity=1.5 -> lower=-6.28318530718 upper=6.28318530718 effort=2000 velocity=0.8
- joint j2n6s200_joint_2: limit lower=0.820304748437 upper=5.46288055874 effort=2000 velocity=1.5 -> lower=0.820304748437 upper=5.46288055874 effort=2000 velocity=0.8
- joint j2n6s200_joint_3: limit lower=0.331612557879 upper=5.9515727493 effort=2000 velocity=1.5 -> lower=0.331612557879 upper=5.9515727493 effort=2000 velocity=0.8
- joint j2n6s200_joint_4: limit lower=-6.28318530718 upper=6.28318530718 effort=2000 velocity=1.5 -> lower=-6.28318530718 upper=6.28318530718 effort=2000 velocity=0.8
- joint j2n6s200_joint_5: limit lower=-6.28318530718 upper=6.28318530718 effort=2000 velocity=1.5 -> lower=-6.28318530718 upper=6.28318530718 effort=2000 velocity=0.8
- joint j2n6s200_joint_6: limit lower=-6.28318530718 upper=6.28318530718 effort=2000 velocity=1.5 -> lower=-6.28318530718 upper=6.28318530718 effort=2000 velocity=0.8
- joint j2n6s200_joint_base: limit lower=0 upper=0 effort=2000 velocity=1.5 -> lower=0 upper=0 effort=2000 velocity=0.8
- joint j2n6s200_joint_forque: origin xyz=-0.003 -0.000 0.078 rpy=3.14 0 0 -> xyz=0.01 -0.000 0.078 rpy=3.14 0 0
- joint j2n6s200_joint_forque_end_effector: origin xyz=0 -0.007 -0.093 rpy=3.1415 0 0 -> xyz=0.007 0 -0.093 rpy=3.1415 0 1.57075
- joint j2n6s200_joint_forque_tip: origin xyz=0 -0.007 -0.093 rpy=2.6415 0 0 -> xyz=0.007 0 -0.093 rpy=2.6415 0 1.57075

Commit message: fork adaptions

File: robots/forque.xacro (robot description, xacro)
@@ -23,5 +23,6 @@
       <child link="j2n6s200_forque"/>
       <axis xyz="0 0 1"/>
-      <origin rpy="3.14 0 0" xyz="-0.003 -0.0013 0.065"/>
+      <!-- <origin rpy="3.14 0 0" xyz="-0.003 -0.0013 0.065"/> -->
+      <origin rpy="3.14 0 0" xyz="-0.013 0.0163 0.065"/>
       <limit effort="2000" lower="0" upper="2" velocity="1"/>
     </joint>

File: robots/kinova_common.xacro (robot description, xacro)
@@ -38,5 +38,5 @@
         <child link="${child}"/>
         <axis xyz="${joint_axis_xyz}"/>
-        <limit effort="2000" velocity="0.8" lower="${joint_lower_limit}" upper="${joint_upper_limit}"/>
+        <limit effort="2000" velocity="1.0" lower="${joint_lower_limit}" upper="${joint_upper_limit}"/>
         <origin xyz="${joint_origin_xyz}" rpy="${joint_origin_rpy}"/>
         <dynamics damping="0.0" friction="0.0"/>

File: robots_urdf/ada.urdf (robot description, URDF)
Before this commit: robot j2n6s200, 15 links, 14 joints
Joints:
- joint j2n6s200_joint_1: limit lower=-6.28318530718 upper=6.28318530718 effort=2000 velocity=0.8 -> lower=-6.28318530718 upper=6.28318530718 effort=2000 velocity=1.0
- joint j2n6s200_joint_2: limit lower=0.820304748437 upper=5.46288055874 effort=2000 velocity=0.8 -> lower=0.820304748437 upper=5.46288055874 effort=2000 velocity=1.0
- joint j2n6s200_joint_3: limit lower=0.331612557879 upper=5.9515727493 effort=2000 velocity=0.8 -> lower=0.331612557879 upper=5.9515727493 effort=2000 velocity=1.0
- joint j2n6s200_joint_4: limit lower=-6.28318530718 upper=6.28318530718 effort=2000 velocity=0.8 -> lower=-6.28318530718 upper=6.28318530718 effort=2000 velocity=1.0
- joint j2n6s200_joint_5: limit lower=-6.28318530718 upper=6.28318530718 effort=2000 velocity=0.8 -> lower=-6.28318530718 upper=6.28318530718 effort=2000 velocity=1.0
- joint j2n6s200_joint_6: limit lower=-6.28318530718 upper=6.28318530718 effort=2000 velocity=0.8 -> lower=-6.28318530718 upper=6.28318530718 effort=2000 velocity=1.0
- joint j2n6s200_joint_base: limit lower=0 upper=0 effort=2000 velocity=0.8 -> lower=0 upper=0 effort=2000 velocity=1.0

File: robots_urdf/ada_with_camera.urdf (robot description, URDF)
Before this commit: robot j2n6s200, 16 links, 15 joints
Joints:
- joint j2n6s200_joint_1: limit lower=-6.28318530718 upper=6.28318530718 effort=2000 velocity=0.8 -> lower=-6.28318530718 upper=6.28318530718 effort=2000 velocity=1.0
- joint j2n6s200_joint_2: limit lower=0.820304748437 upper=5.46288055874 effort=2000 velocity=0.8 -> lower=0.820304748437 upper=5.46288055874 effort=2000 velocity=1.0
- joint j2n6s200_joint_3: limit lower=0.331612557879 upper=5.9515727493 effort=2000 velocity=0.8 -> lower=0.331612557879 upper=5.9515727493 effort=2000 velocity=1.0
- joint j2n6s200_joint_4: limit lower=-6.28318530718 upper=6.28318530718 effort=2000 velocity=0.8 -> lower=-6.28318530718 upper=6.28318530718 effort=2000 velocity=1.0
- joint j2n6s200_joint_5: limit lower=-6.28318530718 upper=6.28318530718 effort=2000 velocity=0.8 -> lower=-6.28318530718 upper=6.28318530718 effort=2000 velocity=1.0
- joint j2n6s200_joint_6: limit lower=-6.28318530718 upper=6.28318530718 effort=2000 velocity=0.8 -> lower=-6.28318530718 upper=6.28318530718 effort=2000 velocity=1.0
- joint j2n6s200_joint_base: limit lower=0 upper=0 effort=2000 velocity=0.8 -> lower=0 upper=0 effort=2000 velocity=1.0

File: robots_urdf/ada_with_camera_forque.urdf (robot description, URDF)
Before this commit: robot j2n6s200, 19 links, 18 joints
Joints:
- joint j2n6s200_joint_1: limit lower=-6.28318530718 upper=6.28318530718 effort=2000 velocity=0.8 -> lower=-6.28318530718 upper=6.28318530718 effort=2000 velocity=1.0
- joint j2n6s200_joint_2: limit lower=0.820304748437 upper=5.46288055874 effort=2000 velocity=0.8 -> lower=0.820304748437 upper=5.46288055874 effort=2000 velocity=1.0
- joint j2n6s200_joint_3: limit lower=0.331612557879 upper=5.9515727493 effort=2000 velocity=0.8 -> lower=0.331612557879 upper=5.9515727493 effort=2000 velocity=1.0
- joint j2n6s200_joint_4: limit lower=-6.28318530718 upper=6.28318530718 effort=2000 velocity=0.8 -> lower=-6.28318530718 upper=6.28318530718 effort=2000 velocity=1.0
- joint j2n6s200_joint_5: limit lower=-6.28318530718 upper=6.28318530718 effort=2000 velocity=0.8 -> lower=-6.28318530718 upper=6.28318530718 effort=2000 velocity=1.0
- joint j2n6s200_joint_6: limit lower=-6.28318530718 upper=6.28318530718 effort=2000 velocity=0.8 -> lower=-6.28318530718 upper=6.28318530718 effort=2000 velocity=1.0
- joint j2n6s200_joint_base: limit lower=0 upper=0 effort=2000 velocity=0.8 -> lower=0 upper=0 effort=2000 velocity=1.0
- joint j2n6s200_joint_forque: origin xyz=-0.003 -0.0013 0.065 rpy=3.14 0 0 -> xyz=-0.013 0.0163 0.065 rpy=3.14 0 0

File: robots_urdf/ada_with_forque.urdf (robot description, URDF)
Before this commit: robot j2n6s200, 18 links, 17 joints
Joints:
- joint j2n6s200_joint_1: limit lower=-6.28318530718 upper=6.28318530718 effort=2000 velocity=0.8 -> lower=-6.28318530718 upper=6.28318530718 effort=2000 velocity=1.0
- joint j2n6s200_joint_2: limit lower=0.820304748437 upper=5.46288055874 effort=2000 velocity=0.8 -> lower=0.820304748437 upper=5.46288055874 effort=2000 velocity=1.0
- joint j2n6s200_joint_3: limit lower=0.331612557879 upper=5.9515727493 effort=2000 velocity=0.8 -> lower=0.331612557879 upper=5.9515727493 effort=2000 velocity=1.0
- joint j2n6s200_joint_4: limit lower=-6.28318530718 upper=6.28318530718 effort=2000 velocity=0.8 -> lower=-6.28318530718 upper=6.28318530718 effort=2000 velocity=1.0
- joint j2n6s200_joint_5: limit lower=-6.28318530718 upper=6.28318530718 effort=2000 velocity=0.8 -> lower=-6.28318530718 upper=6.28318530718 effort=2000 velocity=1.0
- joint j2n6s200_joint_6: limit lower=-6.28318530718 upper=6.28318530718 effort=2000 velocity=0.8 -> lower=-6.28318530718 upper=6.28318530718 effort=2000 velocity=1.0
- joint j2n6s200_joint_base: limit lower=0 upper=0 effort=2000 velocity=0.8 -> lower=0 upper=0 effort=2000 velocity=1.0
- joint j2n6s200_joint_forque: origin xyz=-0.003 -0.0013 0.065 rpy=3.14 0 0 -> xyz=-0.013 0.0163 0.065 rpy=3.14 0 0

Commit message: more 3 finger gripper stuff

File: robots/forque.xacro (robot description, xacro)
@@ -23,5 +23,9 @@
       <child link="j2n6s200_forque"/>
       <axis xyz="0 0 1"/>
-      <origin rpy="3.14 0 0" xyz="-0.003 -0.0013 0.065"/>
+      <!-- <origin rpy="3.14 0 0" xyz="-0.003 -0.0013 0.065"/> -->
+      <!-- was perfect -->
+      <!-- <origin rpy="3.14 0 0" xyz="0.02 -0.0026 0.065"/> -->
+      <!-- <origin rpy="3.14 0 0" xyz="0.02556679118 -0.00332368285 0.08309207135"/> -->
+      <origin rpy="3.14 0 -0.31" xyz="0.02556679118 -0.00332368285 0.08309207135"/>
       <limit effort="2000" lower="0" upper="2" velocity="1"/>
     </joint>

File: robots/j2n6s200.xacro (robot description, xacro)
@@ -74,6 +74,7 @@
     <property name="joint_hand_tip_type" value="fixed" />
     <property name="joint_hand_tip_axis_xyz" value="0 0 0" />
-    <property name="joint_hand_tip_origin_xyz" value="0 0 0.0370" />
+    <property name="joint_hand_tip_origin_xyz" value="0.016 -0.009 0.0370" />
     <property name="joint_hand_tip_origin_rpy" value="0 0 0" />
+    <!--property name="joint_hand_tip_origin_rpy" value="0 0 -0.314" /-->
     <property name="joint_hand_base" value="hand_base" />
     <property name="joint_hand_base_type" value="fixed" />

File: robots/kinova_finger_set.xacro (robot description, xacro)
@@ -21,5 +21,7 @@
         <xacro:kinova_finger prefix="${prefix}" finger_number="2" hand="${link_hand}" finger_origin_xyz="0.02226 -0.02707 -0.11482" finger_origin_rpy="-1.570796327 .649262481663582 -1.38614049188413"/>
         <!-- finger3 Rot := Ry((1/2)*Pi) . Rx(-10.58*((1/180)*Pi)) . Rz(-52.8*((1/180)*Pi)) -->
+<!--
         <xacro:kinova_finger prefix="${prefix}" finger_number="3" hand="${link_hand}" finger_origin_xyz="-0.02226 -0.02707 -0.11482" finger_origin_rpy="-1.570796327 .649262481663582 -1.75545216211587"/>
+-->
     </xacro:macro>
     <xacro:macro name="kinova_2fingers" params="link_hand prefix">

File: robots_urdf/ada.urdf (robot description, URDF)
Before this commit: robot j2n6s200, 15 links, 14 joints
Links:
- link j2n6s200_link_6: geometry collision mesh filename=package://ada_description/meshes/collision_hand_3finger.dae; visual mesh filename=package://ada_description/meshes/hand_3finger.dae
Joints:
- joint j2n6s200_joint_finger_1: origin xyz=-0.0025 0.03095 -0.11482 rpy=-1.570796327 .649262481663582 1.57079632679490 -> xyz=0.00279 0.03126 -0.11467 rpy=-1.570796327 .649262481663582 1.35961148639407
- joint j2n6s200_joint_finger_2: origin xyz=-0.0025 -0.03095 -0.11482 rpy=-1.570796327 .649262481663582 -1.57079632679490 -> xyz=0.02226 -0.02707 -0.11482 rpy=-1.570796327 .649262481663582 -1.38614049188413
- joint j2n6s200_joint_hand_tip: origin xyz=0 0 0.0370 rpy=0 0 0 -> xyz=0.016 -0.009 0.0370 rpy=0 0 0

File: robots_urdf/ada_with_camera.urdf (robot description, URDF)
Before this commit: robot j2n6s200, 16 links, 15 joints
Links:
- link j2n6s200_link_6: geometry collision mesh filename=package://ada_description/meshes/collision_hand_3finger.dae; visual mesh filename=package://ada_description/meshes/hand_3finger.dae
Joints:
- joint j2n6s200_joint_finger_1: origin xyz=-0.0025 0.03095 -0.11482 rpy=-1.570796327 .649262481663582 1.57079632679490 -> xyz=0.00279 0.03126 -0.11467 rpy=-1.570796327 .649262481663582 1.35961148639407
- joint j2n6s200_joint_finger_2: origin xyz=-0.0025 -0.03095 -0.11482 rpy=-1.570796327 .649262481663582 -1.57079632679490 -> xyz=0.02226 -0.02707 -0.11482 rpy=-1.570796327 .649262481663582 -1.38614049188413
- joint j2n6s200_joint_hand_tip: origin xyz=0 0 0.0370 rpy=0 0 0 -> xyz=0.016 -0.009 0.0370 rpy=0 0 0

File: robots_urdf/ada_with_camera_forque.urdf (robot description, URDF)
Before this commit: robot j2n6s200, 19 links, 18 joints
Links:
- link j2n6s200_link_6: geometry collision mesh filename=package://ada_description/meshes/collision_hand_3finger.dae; visual mesh filename=package://ada_description/meshes/hand_3finger.dae
Joints:
- joint j2n6s200_joint_finger_1: origin xyz=-0.0025 0.03095 -0.11482 rpy=-1.570796327 .649262481663582 1.57079632679490 -> xyz=0.00279 0.03126 -0.11467 rpy=-1.570796327 .649262481663582 1.35961148639407
- joint j2n6s200_joint_finger_2: origin xyz=-0.0025 -0.03095 -0.11482 rpy=-1.570796327 .649262481663582 -1.57079632679490 -> xyz=0.02226 -0.02707 -0.11482 rpy=-1.570796327 .649262481663582 -1.38614049188413
- joint j2n6s200_joint_forque: origin xyz=-0.003 -0.0013 0.065 rpy=3.14 0 0 -> xyz=0.02556679118 -0.00332368285 0.08309207135 rpy=3.14 0 -0.31
- joint j2n6s200_joint_hand_tip: origin xyz=0 0 0.0370 rpy=0 0 0 -> xyz=0.016 -0.009 0.0370 rpy=0 0 0

File: robots_urdf/ada_with_forque.urdf (robot description, URDF)
Before this commit: robot j2n6s200, 18 links, 17 joints
Links:
- link j2n6s200_link_6: geometry collision mesh filename=package://ada_description/meshes/collision_hand_3finger.dae; visual mesh filename=package://ada_description/meshes/hand_3finger.dae
Joints:
- joint j2n6s200_joint_finger_1: origin xyz=-0.0025 0.03095 -0.11482 rpy=-1.570796327 .649262481663582 1.57079632679490 -> xyz=0.00279 0.03126 -0.11467 rpy=-1.570796327 .649262481663582 1.35961148639407
- joint j2n6s200_joint_finger_2: origin xyz=-0.0025 -0.03095 -0.11482 rpy=-1.570796327 .649262481663582 -1.57079632679490 -> xyz=0.02226 -0.02707 -0.11482 rpy=-1.570796327 .649262481663582 -1.38614049188413
- joint j2n6s200_joint_forque: origin xyz=-0.003 -0.0013 0.065 rpy=3.14 0 0 -> xyz=0.02556679118 -0.00332368285 0.08309207135 rpy=3.14 0 -0.31
- joint j2n6s200_joint_hand_tip: origin xyz=0 0 0.0370 rpy=0 0 0 -> xyz=0.016 -0.009 0.0370 rpy=0 0 0
