Commit message: fixed typo

File: robots/j2n6s200.xacro (robot description, xacro)
@@ -94,5 +94,5 @@
     <property name="joint_hand_base_axis_xyz" value="0 0 0" />
     <property name="joint_hand_base_origin_xyz" value="0 0 0" />
-    <property name="joint_hand_base_origin_rpy" value="$0 0 0" />
+    <property name="joint_hand_base_origin_rpy" value="0 0 0" />
     <xacro:macro name="j2n6s200" params="base_parent prefix:=j2n6s200">
         <!--xacro:gazebo_config robot_namespace="${prefix}"/-->

File: robots_urdf/ada.urdf (robot description, URDF)
Before this commit: robot j2n6s200, 14 links, 13 joints
Joints:
- joint j2n6s200_joint_hand_base: origin xyz=0 0 0 rpy=$0 0 0 -> xyz=0 0 0 rpy=0 0 0

File: robots_urdf/ada_with_camera.urdf (robot description, URDF)
Before this commit: robot j2n6s200, 15 links, 14 joints
Joints:
- joint j2n6s200_joint_hand_base: origin xyz=0 0 0 rpy=$0 0 0 -> xyz=0 0 0 rpy=0 0 0

File: robots_urdf/ada_with_camera_forque.urdf (robot description, URDF)
Before this commit: robot j2n6s200, 17 links, 16 joints
Joints:
- joint j2n6s200_joint_hand_base: origin xyz=0 0 0 rpy=$0 0 0 -> xyz=0 0 0 rpy=0 0 0

File: robots_urdf/ada_with_forque.urdf (robot description, URDF)
Before this commit: robot j2n6s200, 16 links, 15 joints
Joints:
- joint j2n6s200_joint_hand_base: origin xyz=0 0 0 rpy=$0 0 0 -> xyz=0 0 0 rpy=0 0 0

Commit message: added finger_tips joint

File: robots/j2n6s200.xacro (robot description, xacro)
@@ -71,4 +71,9 @@
     <property name="joint_end_effector_origin_xyz" value="0 0 -0.1600" />
     <property name="joint_end_effector_origin_rpy" value="${J_PI} 0 0" />
+    <property name="joint_finger_tips" value="end_effector_offset" />
+    <property name="joint_finger_tips_type" value="fixed" />
+    <property name="joint_finger_tips_axis_xyz" value="0 0 0" />
+    <property name="joint_finger_tips_origin_xyz" value="0 0 -0.1970" />
+    <property name="joint_finger_tips_origin_rpy" value="${J_PI} 0 0" />
     <property name="joint_hand_base" value="hand_base" />
     <property name="joint_hand_base_type" value="fixed" />
@@ -94,4 +99,6 @@
         <xacro:kinova_virtual_link link_name="${prefix}_end_effector"/>
         <xacro:kinova_virtual_joint joint_name="${prefix}_joint_end_effector" type="${joint_end_effector_type}" parent="${prefix}_link_6" child="${prefix}_end_effector" joint_axis_xyz="${joint_end_effector_axis_xyz}" joint_origin_xyz="${joint_end_effector_origin_xyz}" joint_origin_rpy="${joint_end_effector_origin_rpy}" joint_lower_limit="0" joint_upper_limit="0"/>
+        <xacro:kinova_virtual_link link_name="${prefix}_finger_tips"/>
+        <xacro:kinova_virtual_joint joint_name="${prefix}_joint_finter_tips" type="${joint_finger_tips_type}" parent="${prefix}_link_6" child="${prefix}_finger_tips" joint_axis_xyz="${joint_finger_tips_axis_xyz}" joint_origin_xyz="${joint_finger_tips_origin_xyz}" joint_origin_rpy="${joint_finger_tips_origin_rpy}" joint_lower_limit="0" joint_upper_limit="0"/>
         <xacro:kinova_virtual_link link_name="${prefix}_hand_base"/>
         <xacro:kinova_virtual_joint joint_name="${prefix}_joint_hand_base" type="${joint_hand_base_type}" parent="${prefix}_link_6" child="${prefix}_hand_base" joint_axis_xyz="${joint_hand_base_axis_xyz}" joint_origin_xyz="${joint_hand_base_origin_xyz}" joint_origin_rpy="${joint_hand_base_origin_rpy}" joint_lower_limit="0" joint_upper_limit="0"/>

File: robots_urdf/ada.urdf (robot description, URDF)
Before this commit: robot j2n6s200, 14 links, 13 joints
Links:
- added link j2n6s200_finger_tips
Joints:
- added joint j2n6s200_joint_finter_tips: type fixed, parent j2n6s200_link_6, child j2n6s200_finger_tips, origin xyz=0 0 -0.1970 rpy=3.14159265359 0 0, axis 0 0 0, limit lower=0 upper=0 effort=2000 velocity=1

File: robots_urdf/ada_with_camera.urdf (robot description, URDF)
Before this commit: robot j2n6s200, 15 links, 14 joints
Links:
- added link j2n6s200_finger_tips
Joints:
- added joint j2n6s200_joint_finter_tips: type fixed, parent j2n6s200_link_6, child j2n6s200_finger_tips, origin xyz=0 0 -0.1970 rpy=3.14159265359 0 0, axis 0 0 0, limit lower=0 upper=0 effort=2000 velocity=1

File: robots_urdf/ada_with_camera_forque.urdf (robot description, URDF)
Before this commit: robot j2n6s200, 18 links, 17 joints
Links:
- added link j2n6s200_finger_tips
Joints:
- added joint j2n6s200_joint_finter_tips: type fixed, parent j2n6s200_link_6, child j2n6s200_finger_tips, origin xyz=0 0 -0.1970 rpy=3.14159265359 0 0, axis 0 0 0, limit lower=0 upper=0 effort=2000 velocity=1

File: robots_urdf/ada_with_forque.urdf (robot description, URDF)
Before this commit: robot j2n6s200, 17 links, 16 joints
Links:
- added link j2n6s200_finger_tips
Joints:
- added joint j2n6s200_joint_finter_tips: type fixed, parent j2n6s200_link_6, child j2n6s200_finger_tips, origin xyz=0 0 -0.1970 rpy=3.14159265359 0 0, axis 0 0 0, limit lower=0 upper=0 effort=2000 velocity=1

Commit message: parent of finger_tips is hand_base

File: robots/j2n6s200.xacro (robot description, xacro)
@@ -100,5 +100,5 @@
         <xacro:kinova_virtual_joint joint_name="${prefix}_joint_end_effector" type="${joint_end_effector_type}" parent="${prefix}_link_6" child="${prefix}_end_effector" joint_axis_xyz="${joint_end_effector_axis_xyz}" joint_origin_xyz="${joint_end_effector_origin_xyz}" joint_origin_rpy="${joint_end_effector_origin_rpy}" joint_lower_limit="0" joint_upper_limit="0"/>
         <xacro:kinova_virtual_link link_name="${prefix}_finger_tips"/>
-        <xacro:kinova_virtual_joint joint_name="${prefix}_joint_finter_tips" type="${joint_finger_tips_type}" parent="${prefix}_link_6" child="${prefix}_finger_tips" joint_axis_xyz="${joint_finger_tips_axis_xyz}" joint_origin_xyz="${joint_finger_tips_origin_xyz}" joint_origin_rpy="${joint_finger_tips_origin_rpy}" joint_lower_limit="0" joint_upper_limit="0"/>
+        <xacro:kinova_virtual_joint joint_name="${prefix}_joint_finter_tips" type="${joint_finger_tips_type}" parent="${prefix}_hand_base" child="${prefix}_finger_tips" joint_axis_xyz="${joint_finger_tips_axis_xyz}" joint_origin_xyz="${joint_finger_tips_origin_xyz}" joint_origin_rpy="${joint_finger_tips_origin_rpy}" joint_lower_limit="0" joint_upper_limit="0"/>
         <xacro:kinova_virtual_link link_name="${prefix}_hand_base"/>
         <xacro:kinova_virtual_joint joint_name="${prefix}_joint_hand_base" type="${joint_hand_base_type}" parent="${prefix}_link_6" child="${prefix}_hand_base" joint_axis_xyz="${joint_hand_base_axis_xyz}" joint_origin_xyz="${joint_hand_base_origin_xyz}" joint_origin_rpy="${joint_hand_base_origin_rpy}" joint_lower_limit="0" joint_upper_limit="0"/>

File: robots_urdf/ada.urdf (robot description, URDF)
Before this commit: robot j2n6s200, 15 links, 14 joints
Joints:
- joint j2n6s200_joint_finter_tips: parent j2n6s200_link_6 -> j2n6s200_hand_base

File: robots_urdf/ada_with_camera.urdf (robot description, URDF)
Before this commit: robot j2n6s200, 16 links, 15 joints
Joints:
- joint j2n6s200_joint_finter_tips: parent j2n6s200_link_6 -> j2n6s200_hand_base

File: robots_urdf/ada_with_camera_forque.urdf (robot description, URDF)
Before this commit: robot j2n6s200, 19 links, 18 joints
Joints:
- joint j2n6s200_joint_finter_tips: parent j2n6s200_link_6 -> j2n6s200_hand_base

File: robots_urdf/ada_with_forque.urdf (robot description, URDF)
Before this commit: robot j2n6s200, 18 links, 17 joints
Joints:
- joint j2n6s200_joint_finter_tips: parent j2n6s200_link_6 -> j2n6s200_hand_base

Commit message: some renaming

File: robots/j2n6s200.xacro (robot description, xacro)
@@ -71,9 +71,9 @@
     <property name="joint_end_effector_origin_xyz" value="0 0 -0.1600" />
     <property name="joint_end_effector_origin_rpy" value="${J_PI} 0 0" />
-    <property name="joint_finger_tips" value="end_effector_offset" />
-    <property name="joint_finger_tips_type" value="fixed" />
-    <property name="joint_finger_tips_axis_xyz" value="0 0 0" />
-    <property name="joint_finger_tips_origin_xyz" value="0 0 -0.1970" />
-    <property name="joint_finger_tips_origin_rpy" value="${J_PI} 0 0" />
+    <property name="joint_hand_tip" value="end_effector_offset" />
+    <property name="joint_hand_tip_type" value="fixed" />
+    <property name="joint_hand_tip_axis_xyz" value="0 0 0" />
+    <property name="joint_hand_tip_origin_xyz" value="0 0 -0.1970" />
+    <property name="joint_hand_tip_origin_rpy" value="${J_PI} 0 0" />
     <property name="joint_hand_base" value="hand_base" />
     <property name="joint_hand_base_type" value="fixed" />
@@ -99,6 +99,6 @@
         <xacro:kinova_virtual_link link_name="${prefix}_end_effector"/>
         <xacro:kinova_virtual_joint joint_name="${prefix}_joint_end_effector" type="${joint_end_effector_type}" parent="${prefix}_link_6" child="${prefix}_end_effector" joint_axis_xyz="${joint_end_effector_axis_xyz}" joint_origin_xyz="${joint_end_effector_origin_xyz}" joint_origin_rpy="${joint_end_effector_origin_rpy}" joint_lower_limit="0" joint_upper_limit="0"/>
-        <xacro:kinova_virtual_link link_name="${prefix}_finger_tips"/>
-        <xacro:kinova_virtual_joint joint_name="${prefix}_joint_finter_tips" type="${joint_finger_tips_type}" parent="${prefix}_hand_base" child="${prefix}_finger_tips" joint_axis_xyz="${joint_finger_tips_axis_xyz}" joint_origin_xyz="${joint_finger_tips_origin_xyz}" joint_origin_rpy="${joint_finger_tips_origin_rpy}" joint_lower_limit="0" joint_upper_limit="0"/>
+        <xacro:kinova_virtual_link link_name="${prefix}_hand_tip"/>
+        <xacro:kinova_virtual_joint joint_name="${prefix}_joint_hand_tip" type="${joint_hand_tip_type}" parent="${prefix}_hand_base" child="${prefix}_hand_tip" joint_axis_xyz="${joint_hand_tip_axis_xyz}" joint_origin_xyz="${joint_hand_tip_origin_xyz}" joint_origin_rpy="${joint_hand_tip_origin_rpy}" joint_lower_limit="0" joint_upper_limit="0"/>
         <xacro:kinova_virtual_link link_name="${prefix}_hand_base"/>
         <xacro:kinova_virtual_joint joint_name="${prefix}_joint_hand_base" type="${joint_hand_base_type}" parent="${prefix}_link_6" child="${prefix}_hand_base" joint_axis_xyz="${joint_hand_base_axis_xyz}" joint_origin_xyz="${joint_hand_base_origin_xyz}" joint_origin_rpy="${joint_hand_base_origin_rpy}" joint_lower_limit="0" joint_upper_limit="0"/>

File: robots_urdf/ada.urdf (robot description, URDF)
Before this commit: robot j2n6s200, 15 links, 14 joints
Links:
- removed link j2n6s200_finger_tips
- added link j2n6s200_hand_tip
Joints:
- removed joint j2n6s200_joint_finter_tips
- added joint j2n6s200_joint_hand_tip: type fixed, parent j2n6s200_hand_base, child j2n6s200_hand_tip, origin xyz=0 0 -0.1970 rpy=3.14159265359 0 0, axis 0 0 0, limit lower=0 upper=0 effort=2000 velocity=1

File: robots_urdf/ada_with_camera.urdf (robot description, URDF)
Before this commit: robot j2n6s200, 16 links, 15 joints
Links:
- removed link j2n6s200_finger_tips
- added link j2n6s200_hand_tip
Joints:
- removed joint j2n6s200_joint_finter_tips
- added joint j2n6s200_joint_hand_tip: type fixed, parent j2n6s200_hand_base, child j2n6s200_hand_tip, origin xyz=0 0 -0.1970 rpy=3.14159265359 0 0, axis 0 0 0, limit lower=0 upper=0 effort=2000 velocity=1

File: robots_urdf/ada_with_camera_forque.urdf (robot description, URDF)
Before this commit: robot j2n6s200, 19 links, 18 joints
Links:
- removed link j2n6s200_finger_tips
- added link j2n6s200_hand_tip
Joints:
- removed joint j2n6s200_joint_finter_tips
- added joint j2n6s200_joint_hand_tip: type fixed, parent j2n6s200_hand_base, child j2n6s200_hand_tip, origin xyz=0 0 -0.1970 rpy=3.14159265359 0 0, axis 0 0 0, limit lower=0 upper=0 effort=2000 velocity=1

File: robots_urdf/ada_with_forque.urdf (robot description, URDF)
Before this commit: robot j2n6s200, 18 links, 17 joints
Links:
- removed link j2n6s200_finger_tips
- added link j2n6s200_hand_tip
Joints:
- removed joint j2n6s200_joint_finter_tips
- added joint j2n6s200_joint_hand_tip: type fixed, parent j2n6s200_hand_base, child j2n6s200_hand_tip, origin xyz=0 0 -0.1970 rpy=3.14159265359 0 0, axis 0 0 0, limit lower=0 upper=0 effort=2000 velocity=1

Commit message: changed handTip parent

File: robots/j2n6s200.xacro (robot description, xacro)
@@ -74,6 +74,6 @@
     <property name="joint_hand_tip_type" value="fixed" />
     <property name="joint_hand_tip_axis_xyz" value="0 0 0" />
-    <property name="joint_hand_tip_origin_xyz" value="0 0 -0.1970" />
-    <property name="joint_hand_tip_origin_rpy" value="${J_PI} 0 0" />
+    <property name="joint_hand_tip_origin_xyz" value="0 0 0.0370" />
+    <property name="joint_hand_tip_origin_rpy" value="0 0 0" />
     <property name="joint_hand_base" value="hand_base" />
     <property name="joint_hand_base_type" value="fixed" />
@@ -100,5 +100,5 @@
         <xacro:kinova_virtual_joint joint_name="${prefix}_joint_end_effector" type="${joint_end_effector_type}" parent="${prefix}_link_6" child="${prefix}_end_effector" joint_axis_xyz="${joint_end_effector_axis_xyz}" joint_origin_xyz="${joint_end_effector_origin_xyz}" joint_origin_rpy="${joint_end_effector_origin_rpy}" joint_lower_limit="0" joint_upper_limit="0"/>
         <xacro:kinova_virtual_link link_name="${prefix}_hand_tip"/>
-        <xacro:kinova_virtual_joint joint_name="${prefix}_joint_hand_tip" type="${joint_hand_tip_type}" parent="${prefix}_hand_base" child="${prefix}_hand_tip" joint_axis_xyz="${joint_hand_tip_axis_xyz}" joint_origin_xyz="${joint_hand_tip_origin_xyz}" joint_origin_rpy="${joint_hand_tip_origin_rpy}" joint_lower_limit="0" joint_upper_limit="0"/>
+        <xacro:kinova_virtual_joint joint_name="${prefix}_joint_hand_tip" type="${joint_hand_tip_type}" parent="${prefix}_end_effector" child="${prefix}_hand_tip" joint_axis_xyz="${joint_hand_tip_axis_xyz}" joint_origin_xyz="${joint_hand_tip_origin_xyz}" joint_origin_rpy="${joint_hand_tip_origin_rpy}" joint_lower_limit="0" joint_upper_limit="0"/>
         <xacro:kinova_virtual_link link_name="${prefix}_hand_base"/>
         <xacro:kinova_virtual_joint joint_name="${prefix}_joint_hand_base" type="${joint_hand_base_type}" parent="${prefix}_link_6" child="${prefix}_hand_base" joint_axis_xyz="${joint_hand_base_axis_xyz}" joint_origin_xyz="${joint_hand_base_origin_xyz}" joint_origin_rpy="${joint_hand_base_origin_rpy}" joint_lower_limit="0" joint_upper_limit="0"/>

File: robots_urdf/ada.urdf (robot description, URDF)
Before this commit: robot j2n6s200, 15 links, 14 joints
Joints:
- joint j2n6s200_joint_hand_tip: origin xyz=0 0 -0.1970 rpy=3.14159265359 0 0 -> xyz=0 0 0.0370 rpy=0 0 0; parent j2n6s200_hand_base -> j2n6s200_end_effector

File: robots_urdf/ada_with_camera.urdf (robot description, URDF)
Before this commit: robot j2n6s200, 16 links, 15 joints
Joints:
- joint j2n6s200_joint_hand_tip: origin xyz=0 0 -0.1970 rpy=3.14159265359 0 0 -> xyz=0 0 0.0370 rpy=0 0 0; parent j2n6s200_hand_base -> j2n6s200_end_effector

File: robots_urdf/ada_with_camera_forque.urdf (robot description, URDF)
Before this commit: robot j2n6s200, 19 links, 18 joints
Joints:
- joint j2n6s200_joint_hand_tip: origin xyz=0 0 -0.1970 rpy=3.14159265359 0 0 -> xyz=0 0 0.0370 rpy=0 0 0; parent j2n6s200_hand_base -> j2n6s200_end_effector

File: robots_urdf/ada_with_forque.urdf (robot description, URDF)
Before this commit: robot j2n6s200, 18 links, 17 joints
Joints:
- joint j2n6s200_joint_hand_tip: origin xyz=0 0 -0.1970 rpy=3.14159265359 0 0 -> xyz=0 0 0.0370 rpy=0 0 0; parent j2n6s200_hand_base -> j2n6s200_end_effector

Commit message: continuous joints in xacro

File: robots/j2n6s200.xacro (robot description, xacro)
@@ -25,5 +25,5 @@
     <property name="joint_base_origin_rpy" value="0 0 0" />
     <property name="joint_1" value="joint_1" />
-    <property name="joint_1_type" value="revolute" />
+    <property name="joint_1_type" value="continuous" />
     <property name="joint_1_axis_xyz" value="0 0 1" />
     <property name="joint_1_origin_xyz" value="0 0 0.15675" />
@@ -46,5 +46,5 @@
     <property name="joint_3_upper_limit" value="${341/180*J_PI}" />
     <property name="joint_4" value="joint_4" />
-    <property name="joint_4_type" value="revolute" />
+    <property name="joint_4_type" value="continuous" />
     <property name="joint_4_axis_xyz" value="0 0 1" />
     <property name="joint_4_origin_xyz" value="0 0.2073 -0.0114" />
@@ -53,5 +53,5 @@
     <property name="joint_4_upper_limit" value="${2*J_PI}" />
     <property name="joint_5" value="joint_5" />
-    <property name="joint_5_type" value="revolute" />
+    <property name="joint_5_type" value="continuous" />
     <property name="joint_5_axis_xyz" value="0 0 1" />
     <property name="joint_5_origin_xyz" value="0 -0.03703 -0.06414" />
@@ -60,5 +60,5 @@
     <property name="joint_5_upper_limit" value="${2*J_PI}" />
     <property name="joint_6" value="joint_6" />
-    <property name="joint_6_type" value="revolute" />
+    <property name="joint_6_type" value="continuous" />
     <property name="joint_6_axis_xyz" value="0 0 1" />
     <property name="joint_6_origin_xyz" value="0 -0.03703 -0.06414" />

File: robots_urdf/ada.urdf (robot description, URDF)
Before this commit: robot j2n6s200, 15 links, 14 joints
Joints:
- joint j2n6s200_joint_1: type revolute -> continuous
- joint j2n6s200_joint_4: type revolute -> continuous
- joint j2n6s200_joint_5: type revolute -> continuous
- joint j2n6s200_joint_6: type revolute -> continuous

File: robots_urdf/ada_with_camera.urdf (robot description, URDF)
Before this commit: robot j2n6s200, 16 links, 15 joints
Joints:
- joint j2n6s200_joint_1: type revolute -> continuous
- joint j2n6s200_joint_4: type revolute -> continuous
- joint j2n6s200_joint_5: type revolute -> continuous
- joint j2n6s200_joint_6: type revolute -> continuous

File: robots_urdf/ada_with_camera_forque.urdf (robot description, URDF)
Before this commit: robot j2n6s200, 19 links, 18 joints
Joints:
- joint j2n6s200_joint_1: type revolute -> continuous
- joint j2n6s200_joint_4: type revolute -> continuous
- joint j2n6s200_joint_5: type revolute -> continuous
- joint j2n6s200_joint_6: type revolute -> continuous

File: robots_urdf/ada_with_forque.urdf (robot description, URDF)
Before this commit: robot j2n6s200, 18 links, 17 joints
Joints:
- joint j2n6s200_joint_1: type revolute -> continuous
- joint j2n6s200_joint_4: type revolute -> continuous
- joint j2n6s200_joint_5: type revolute -> continuous
- joint j2n6s200_joint_6: type revolute -> continuous

Commit message: 3 finger hand

File: robots/j2n6s200.xacro (robot description, xacro)
@@ -11,5 +11,5 @@
     <property name="link_4_mesh" value="wrist" />
     <property name="link_5_mesh" value="wrist" />
-    <property name="link_6_mesh" value="hand_2finger" />
+    <property name="link_6_mesh" value="hand_3finger" />
     <property name="link_base_mesh_no" value="0" />
     <property name="link_1_mesh_no" value="1" />
@@ -103,5 +103,5 @@
         <xacro:kinova_virtual_link link_name="${prefix}_hand_base"/>
         <xacro:kinova_virtual_joint joint_name="${prefix}_joint_hand_base" type="${joint_hand_base_type}" parent="${prefix}_link_6" child="${prefix}_hand_base" joint_axis_xyz="${joint_hand_base_axis_xyz}" joint_origin_xyz="${joint_hand_base_origin_xyz}" joint_origin_rpy="${joint_hand_base_origin_rpy}" joint_lower_limit="0" joint_upper_limit="0"/>
-        <xacro:kinova_2fingers link_hand="${prefix}_hand_base" prefix="${prefix}_"/>
+        <xacro:kinova_3fingers link_hand="${prefix}_hand_base" prefix="${prefix}_"/>
     </xacro:macro>
 </root>

File: robots/kinova_finger_set.xacro (robot description, xacro)
@@ -15,4 +15,12 @@
     xmlns:xacro="http://ros.org/wiki/xacro">
     <xacro:include filename="$(find ada_description)/robots/kinova_common.xacro" />
+    <xacro:macro name="kinova_3fingers" params="link_hand prefix">
+        <!-- finger1 Rot := Ry((1/2)*Pi) . Rx(12.1*((1/180)*Pi)+Pi) . Rz(-52.8*((1/180)*Pi)) -->
+        <xacro:kinova_finger prefix="${prefix}" finger_number="1" hand="${link_hand}" finger_origin_xyz="0.00279 0.03126 -0.11467" finger_origin_rpy="-1.570796327 .649262481663582 1.35961148639407"/>
+        <!-- finger2 Rot := Ry((1/2)*Pi) . Rx(10.58*((1/180)*Pi)) . Rz(-52.8*((1/180)*Pi)) -->
+        <xacro:kinova_finger prefix="${prefix}" finger_number="2" hand="${link_hand}" finger_origin_xyz="0.02226 -0.02707 -0.11482" finger_origin_rpy="-1.570796327 .649262481663582 -1.38614049188413"/>
+        <!-- finger3 Rot := Ry((1/2)*Pi) . Rx(-10.58*((1/180)*Pi)) . Rz(-52.8*((1/180)*Pi)) -->
+        <xacro:kinova_finger prefix="${prefix}" finger_number="3" hand="${link_hand}" finger_origin_xyz="-0.02226 -0.02707 -0.11482" finger_origin_rpy="-1.570796327 .649262481663582 -1.75545216211587"/>
+    </xacro:macro>
     <xacro:macro name="kinova_2fingers" params="link_hand prefix">
         <!-- finger1 Rot := Ry((1/2)*Pi) . Rx(Pi) . Rz(-52.8*((1/180)*Pi)) -->

File: robots/kinova_inertial.xacro (robot description, xacro)
@@ -21,4 +21,5 @@
    wrist_spherical_1  8
    wrist_spherical_2  9
+   hand 3 finger  		55
    hand_2finger   		56
    finger_proximal		57
@@ -118,4 +119,12 @@
     </inertial>
   </xacro:unless>
+  <!-- hand 3 finger = 55 -->
+  <xacro:unless value="${mesh_no - 55}">
+    <inertial>
+        <mass value="0.99" />
+        <origin xyz="0 0 -0.06" />
+        <xacro:inertia_cylinder height="0.03"  radius = "0.04" mass="0.727"/>
+    </inertial>
+  </xacro:unless>
   <!-- hand 2 finger = 56 -->
   <xacro:unless value="${mesh_no - 56}">
