Commit message: speed changes

File: robots/kinova_common.xacro (robot description, xacro)
@@ -49,5 +49,5 @@
         <child link="${child}"/>
         <axis xyz="${joint_axis_xyz}"/>
-        <limit effort="2000" velocity="1" lower="${joint_lower_limit}" upper="${joint_upper_limit}"/>
+        <limit effort="2000" velocity="1.6" lower="${joint_lower_limit}" upper="${joint_upper_limit}"/>
         <origin xyz="${joint_origin_xyz}" rpy="${joint_origin_rpy}"/>
         <dynamics damping="0.0" friction="0.0"/>

File: robots_urdf/ada.urdf (robot description, URDF)
Before this commit: robot j2n6s200, 14 links, 13 joints
Joints:
- joint j2n6s200_joint_1: limit lower=-6.28318530718 upper=6.28318530718 effort=2000 velocity=1 -> lower=-6.28318530718 upper=6.28318530718 effort=2000 velocity=1.6
- joint j2n6s200_joint_2: limit lower=0.820304748437 upper=5.46288055874 effort=2000 velocity=1 -> lower=0.820304748437 upper=5.46288055874 effort=2000 velocity=1.6
- joint j2n6s200_joint_3: limit lower=0.331612557879 upper=5.9515727493 effort=2000 velocity=1 -> lower=0.331612557879 upper=5.9515727493 effort=2000 velocity=1.6
- joint j2n6s200_joint_4: limit lower=-6.28318530718 upper=6.28318530718 effort=2000 velocity=1 -> lower=-6.28318530718 upper=6.28318530718 effort=2000 velocity=1.6
- joint j2n6s200_joint_5: limit lower=-6.28318530718 upper=6.28318530718 effort=2000 velocity=1 -> lower=-6.28318530718 upper=6.28318530718 effort=2000 velocity=1.6
- joint j2n6s200_joint_6: limit lower=-6.28318530718 upper=6.28318530718 effort=2000 velocity=1 -> lower=-6.28318530718 upper=6.28318530718 effort=2000 velocity=1.6
- joint j2n6s200_joint_base: limit lower=0 upper=0 effort=2000 velocity=1 -> lower=0 upper=0 effort=2000 velocity=1.6

File: robots_urdf/ada_with_camera.urdf (robot description, URDF)
Before this commit: robot j2n6s200, 15 links, 14 joints
Joints:
- joint j2n6s200_joint_1: limit lower=-6.28318530718 upper=6.28318530718 effort=2000 velocity=1 -> lower=-6.28318530718 upper=6.28318530718 effort=2000 velocity=1.6
- joint j2n6s200_joint_2: limit lower=0.820304748437 upper=5.46288055874 effort=2000 velocity=1 -> lower=0.820304748437 upper=5.46288055874 effort=2000 velocity=1.6
- joint j2n6s200_joint_3: limit lower=0.331612557879 upper=5.9515727493 effort=2000 velocity=1 -> lower=0.331612557879 upper=5.9515727493 effort=2000 velocity=1.6
- joint j2n6s200_joint_4: limit lower=-6.28318530718 upper=6.28318530718 effort=2000 velocity=1 -> lower=-6.28318530718 upper=6.28318530718 effort=2000 velocity=1.6
- joint j2n6s200_joint_5: limit lower=-6.28318530718 upper=6.28318530718 effort=2000 velocity=1 -> lower=-6.28318530718 upper=6.28318530718 effort=2000 velocity=1.6
- joint j2n6s200_joint_6: limit lower=-6.28318530718 upper=6.28318530718 effort=2000 velocity=1 -> lower=-6.28318530718 upper=6.28318530718 effort=2000 velocity=1.6
- joint j2n6s200_joint_base: limit lower=0 upper=0 effort=2000 velocity=1 -> lower=0 upper=0 effort=2000 velocity=1.6

File: robots_urdf/ada_with_camera_forque.urdf (robot description, URDF)
Before this commit: robot j2n6s200, 17 links, 16 joints
Joints:
- joint j2n6s200_joint_1: limit lower=-6.28318530718 upper=6.28318530718 effort=2000 velocity=1 -> lower=-6.28318530718 upper=6.28318530718 effort=2000 velocity=1.6
- joint j2n6s200_joint_2: limit lower=0.820304748437 upper=5.46288055874 effort=2000 velocity=1 -> lower=0.820304748437 upper=5.46288055874 effort=2000 velocity=1.6
- joint j2n6s200_joint_3: limit lower=0.331612557879 upper=5.9515727493 effort=2000 velocity=1 -> lower=0.331612557879 upper=5.9515727493 effort=2000 velocity=1.6
- joint j2n6s200_joint_4: limit lower=-6.28318530718 upper=6.28318530718 effort=2000 velocity=1 -> lower=-6.28318530718 upper=6.28318530718 effort=2000 velocity=1.6
- joint j2n6s200_joint_5: limit lower=-6.28318530718 upper=6.28318530718 effort=2000 velocity=1 -> lower=-6.28318530718 upper=6.28318530718 effort=2000 velocity=1.6
- joint j2n6s200_joint_6: limit lower=-6.28318530718 upper=6.28318530718 effort=2000 velocity=1 -> lower=-6.28318530718 upper=6.28318530718 effort=2000 velocity=1.6
- joint j2n6s200_joint_base: limit lower=0 upper=0 effort=2000 velocity=1 -> lower=0 upper=0 effort=2000 velocity=1.6

File: robots_urdf/ada_with_forque.urdf (robot description, URDF)
Before this commit: robot j2n6s200, 16 links, 15 joints
Joints:
- joint j2n6s200_joint_1: limit lower=-6.28318530718 upper=6.28318530718 effort=2000 velocity=1 -> lower=-6.28318530718 upper=6.28318530718 effort=2000 velocity=1.6
- joint j2n6s200_joint_2: limit lower=0.820304748437 upper=5.46288055874 effort=2000 velocity=1 -> lower=0.820304748437 upper=5.46288055874 effort=2000 velocity=1.6
- joint j2n6s200_joint_3: limit lower=0.331612557879 upper=5.9515727493 effort=2000 velocity=1 -> lower=0.331612557879 upper=5.9515727493 effort=2000 velocity=1.6
- joint j2n6s200_joint_4: limit lower=-6.28318530718 upper=6.28318530718 effort=2000 velocity=1 -> lower=-6.28318530718 upper=6.28318530718 effort=2000 velocity=1.6
- joint j2n6s200_joint_5: limit lower=-6.28318530718 upper=6.28318530718 effort=2000 velocity=1 -> lower=-6.28318530718 upper=6.28318530718 effort=2000 velocity=1.6
- joint j2n6s200_joint_6: limit lower=-6.28318530718 upper=6.28318530718 effort=2000 velocity=1 -> lower=-6.28318530718 upper=6.28318530718 effort=2000 velocity=1.6
- joint j2n6s200_joint_base: limit lower=0 upper=0 effort=2000 velocity=1 -> lower=0 upper=0 effort=2000 velocity=1.6

Commit message: bigger camera collision box

File: robots/kinova_common.xacro (robot description, xacro)
@@ -38,5 +38,5 @@
         <child link="${child}"/>
         <axis xyz="${joint_axis_xyz}"/>
-        <limit effort="2000" velocity="1.5" lower="${joint_lower_limit}" upper="${joint_upper_limit}"/>
+        <limit effort="2000" velocity="1.0" lower="${joint_lower_limit}" upper="${joint_upper_limit}"/>
         <origin xyz="${joint_origin_xyz}" rpy="${joint_origin_rpy}"/>
         <dynamics damping="0.0" friction="0.0"/>

File: robots_urdf/ada.urdf (robot description, URDF)
Before this commit: robot j2n6s200, 15 links, 14 joints
Joints:
- joint j2n6s200_joint_1: limit lower=-6.28318530718 upper=6.28318530718 effort=2000 velocity=1.5 -> lower=-6.28318530718 upper=6.28318530718 effort=2000 velocity=1.0
- joint j2n6s200_joint_2: limit lower=0.820304748437 upper=5.46288055874 effort=2000 velocity=1.5 -> lower=0.820304748437 upper=5.46288055874 effort=2000 velocity=1.0
- joint j2n6s200_joint_3: limit lower=0.331612557879 upper=5.9515727493 effort=2000 velocity=1.5 -> lower=0.331612557879 upper=5.9515727493 effort=2000 velocity=1.0
- joint j2n6s200_joint_4: limit lower=-6.28318530718 upper=6.28318530718 effort=2000 velocity=1.5 -> lower=-6.28318530718 upper=6.28318530718 effort=2000 velocity=1.0
- joint j2n6s200_joint_5: limit lower=-6.28318530718 upper=6.28318530718 effort=2000 velocity=1.5 -> lower=-6.28318530718 upper=6.28318530718 effort=2000 velocity=1.0
- joint j2n6s200_joint_6: limit lower=-6.28318530718 upper=6.28318530718 effort=2000 velocity=1.5 -> lower=-6.28318530718 upper=6.28318530718 effort=2000 velocity=1.0
- joint j2n6s200_joint_base: limit lower=0 upper=0 effort=2000 velocity=1.5 -> lower=0 upper=0 effort=2000 velocity=1.0

File: robots_urdf/ada_with_camera.urdf (robot description, URDF)
Before this commit: robot j2n6s200, 16 links, 15 joints
Links:
- link j2n6s200_joule: geometry collision mesh filename=package://ada_description/meshes/collision_camera_joule.dae scale=0.001 0.001 0.00098; visual mesh filename=package://ada_description/meshes/collision_camera_joule.dae scale=0.001 0.001 0.00098
Joints:
- joint j2n6s200_joint_1: limit lower=-6.28318530718 upper=6.28318530718 effort=2000 velocity=1.5 -> lower=-6.28318530718 upper=6.28318530718 effort=2000 velocity=1.0
- joint j2n6s200_joint_2: limit lower=0.820304748437 upper=5.46288055874 effort=2000 velocity=1.5 -> lower=0.820304748437 upper=5.46288055874 effort=2000 velocity=1.0
- joint j2n6s200_joint_3: limit lower=0.331612557879 upper=5.9515727493 effort=2000 velocity=1.5 -> lower=0.331612557879 upper=5.9515727493 effort=2000 velocity=1.0
- joint j2n6s200_joint_4: limit lower=-6.28318530718 upper=6.28318530718 effort=2000 velocity=1.5 -> lower=-6.28318530718 upper=6.28318530718 effort=2000 velocity=1.0
- joint j2n6s200_joint_5: limit lower=-6.28318530718 upper=6.28318530718 effort=2000 velocity=1.5 -> lower=-6.28318530718 upper=6.28318530718 effort=2000 velocity=1.0
- joint j2n6s200_joint_6: limit lower=-6.28318530718 upper=6.28318530718 effort=2000 velocity=1.5 -> lower=-6.28318530718 upper=6.28318530718 effort=2000 velocity=1.0
- joint j2n6s200_joint_base: limit lower=0 upper=0 effort=2000 velocity=1.5 -> lower=0 upper=0 effort=2000 velocity=1.0

File: robots_urdf/ada_with_camera_forque.urdf (robot description, URDF)
Before this commit: robot j2n6s200, 19 links, 18 joints
Links:
- link j2n6s200_joule: geometry collision mesh filename=package://ada_description/meshes/collision_camera_joule.dae scale=0.001 0.001 0.00098; visual mesh filename=package://ada_description/meshes/collision_camera_joule.dae scale=0.001 0.001 0.00098
Joints:
- joint j2n6s200_joint_1: limit lower=-6.28318530718 upper=6.28318530718 effort=2000 velocity=1.5 -> lower=-6.28318530718 upper=6.28318530718 effort=2000 velocity=1.0
- joint j2n6s200_joint_2: limit lower=0.820304748437 upper=5.46288055874 effort=2000 velocity=1.5 -> lower=0.820304748437 upper=5.46288055874 effort=2000 velocity=1.0
- joint j2n6s200_joint_3: limit lower=0.331612557879 upper=5.9515727493 effort=2000 velocity=1.5 -> lower=0.331612557879 upper=5.9515727493 effort=2000 velocity=1.0
- joint j2n6s200_joint_4: limit lower=-6.28318530718 upper=6.28318530718 effort=2000 velocity=1.5 -> lower=-6.28318530718 upper=6.28318530718 effort=2000 velocity=1.0
- joint j2n6s200_joint_5: limit lower=-6.28318530718 upper=6.28318530718 effort=2000 velocity=1.5 -> lower=-6.28318530718 upper=6.28318530718 effort=2000 velocity=1.0
- joint j2n6s200_joint_6: limit lower=-6.28318530718 upper=6.28318530718 effort=2000 velocity=1.5 -> lower=-6.28318530718 upper=6.28318530718 effort=2000 velocity=1.0
- joint j2n6s200_joint_base: limit lower=0 upper=0 effort=2000 velocity=1.5 -> lower=0 upper=0 effort=2000 velocity=1.0

File: robots_urdf/ada_with_forque.urdf (robot description, URDF)
Before this commit: robot j2n6s200, 18 links, 17 joints
Joints:
- joint j2n6s200_joint_1: limit lower=-6.28318530718 upper=6.28318530718 effort=2000 velocity=1.5 -> lower=-6.28318530718 upper=6.28318530718 effort=2000 velocity=1.0
- joint j2n6s200_joint_2: limit lower=0.820304748437 upper=5.46288055874 effort=2000 velocity=1.5 -> lower=0.820304748437 upper=5.46288055874 effort=2000 velocity=1.0
- joint j2n6s200_joint_3: limit lower=0.331612557879 upper=5.9515727493 effort=2000 velocity=1.5 -> lower=0.331612557879 upper=5.9515727493 effort=2000 velocity=1.0
- joint j2n6s200_joint_4: limit lower=-6.28318530718 upper=6.28318530718 effort=2000 velocity=1.5 -> lower=-6.28318530718 upper=6.28318530718 effort=2000 velocity=1.0
- joint j2n6s200_joint_5: limit lower=-6.28318530718 upper=6.28318530718 effort=2000 velocity=1.5 -> lower=-6.28318530718 upper=6.28318530718 effort=2000 velocity=1.0
- joint j2n6s200_joint_6: limit lower=-6.28318530718 upper=6.28318530718 effort=2000 velocity=1.5 -> lower=-6.28318530718 upper=6.28318530718 effort=2000 velocity=1.0
- joint j2n6s200_joint_base: limit lower=0 upper=0 effort=2000 velocity=1.5 -> lower=0 upper=0 effort=2000 velocity=1.0

Commit message: Use random inertia/mass for dummy links in virtual link macro

File: robots/kinova_common.xacro (robot description, xacro)
@@ -57,5 +57,15 @@
     <xacro:macro name="kinova_virtual_link" params="link_name">
       <link name="${link_name}">
-  </link>
+        <!--
+        In order to model the link in simulation it must have an inertial tag, even
+        though it is only a dummy link. Furthermore, it must have a non-zero mass/inertia,
+        so just use random values.
+        -->
+        <inertial>
+          <origin xyz="0.0 0.0 0.0" rpy="0 0 0"/>
+          <mass value="0.3"/>
+          <inertia ixx="0.1" ixy="0.4" ixz="0.1" iyy="0.5" iyz="0.9" izz="0.2"/>
+        </inertial>
+      </link>
     </xacro:macro>
     <xacro:macro name="kinova_virtual_joint" params="joint_name type parent child joint_axis_xyz joint_origin_xyz joint_origin_rpy joint_lower_limit joint_upper_limit">
