Commit message: new camera model

File: robots/camera.xacro (robot description, xacro)
@@ -19,5 +19,5 @@
         <origin rpy="0 0 0" xyz="0 0 0"/>
         <geometry>
-          <mesh filename="package://ada_description/meshes/camera_joule_tex.STL" scale="0.001 0.001 0.001"/>
+          <mesh filename="package://ada_description/meshes/joule_text.dae" scale="0.001 0.001 0.001"/>
         </geometry>
       <material name="carbon_fiber">
@@ -26,7 +26,7 @@
       </visual>
       <collision>
-      <origin xyz="-0.014 -0.072 -0.025" rpy="0 0 0"/>
+        <origin  rpy="0 0 0" xyz="-0.014 -0.072 -0.033"/>
         <geometry>
-          <mesh filename="package://ada_description/meshes/camera_joule_tex.dae" scale="0.001 0.001 0.00094"/>
+          <mesh filename="package://ada_description/meshes/collision_camera_joule_tex.dae" scale="0.001 0.001 0.00098"/>
         </geometry>
       </collision>
@@ -37,5 +37,5 @@
       <axis xyz="0 0 1"/>
       <limit effort="2000" lower="-6.28318530718" upper="6.28318530718" velocity="1"/>
-    <origin rpy="-1.57079632679 1.57079632679 0" xyz="-0.06 -0.051 -0.0163"/>
+      <origin rpy="1.57079632679 1.57079632679 0" xyz="0.06 0.051 0.0140"/>
       <dynamics damping="0.0" friction="0.0"/>
     </joint>

File: robots/j2n6s200.xacro (robot description, xacro)
@@ -95,5 +95,5 @@
     <property name="joint_hand_base_origin_xyz" value="0 0 0" />
     <property name="joint_hand_base_origin_rpy" value="0 0 0" />
-    <xacro:macro name="j2n6s200" params="base_parent prefix:=j2n6s200">
+    <xacro:macro name="j2n6s200" params="base_parent use_final_ring:=true prefix:=j2n6s200">
         <!--xacro:gazebo_config robot_namespace="${prefix}"/-->
         <xacro:kinova_armlink link_name="${prefix}_link_base" link_mesh="${link_base_mesh}" mesh_no="${link_base_mesh_no}"/>
@@ -109,5 +109,5 @@
         <xacro:kinova_armlink link_name="${prefix}_link_5" link_mesh="${link_5_mesh}" use_ring_mesh="true" ring_mesh="ring_small" mesh_no="${link_5_mesh_no}"/>
         <xacro:kinova_armjoint joint_name="${prefix}_joint_5" type="${joint_5_type}" parent="${prefix}_link_4" child="${prefix}_link_5" joint_axis_xyz="${joint_5_axis_xyz}" joint_origin_xyz="${joint_5_origin_xyz}" joint_origin_rpy="${joint_5_origin_rpy}" joint_lower_limit="${joint_5_lower_limit}" joint_upper_limit="${joint_5_upper_limit}"/>
-        <xacro:kinova_armlink link_name="${prefix}_link_6" link_mesh="${link_6_mesh}" use_ring_mesh="true" ring_mesh="ring_small" mesh_no="${link_6_mesh_no}"/>
+        <xacro:kinova_armlink link_name="${prefix}_link_6" link_mesh="${link_6_mesh}" use_ring_mesh="${use_final_ring}" ring_mesh="ring_small" mesh_no="${link_6_mesh_no}"/>
         <xacro:kinova_armjoint joint_name="${prefix}_joint_6" type="${joint_6_type}" parent="${prefix}_link_5" child="${prefix}_link_6" joint_axis_xyz="${joint_6_axis_xyz}" joint_origin_xyz="${joint_6_origin_xyz}" joint_origin_rpy="${joint_6_origin_rpy}" joint_lower_limit="${joint_6_lower_limit}" joint_upper_limit="${joint_6_upper_limit}"/>
         <xacro:kinova_virtual_link link_name="${prefix}_end_effector"/>

File: robots/j2n6s200_standalone.xacro (robot description, xacro)
@@ -22,5 +22,5 @@
   <property name="robot_root" value="world" />
   <property name="prefix" value="j2n6s200" />
-  <xacro:j2n6s200  base_parent="${robot_root}"/>
+  <xacro:j2n6s200  base_parent="${robot_root}" use_final_ring="'false'"/>
   <xacro:if value="$(arg with_camera)">
     <xacro:camera  camera_parent="${prefix}_link_6"/>

File: robots_urdf/ada.urdf (robot description, URDF)
Before this commit: robot j2n6s200, 14 links, 13 joints
Links:
- link j2n6s200_link_6: geometry collision mesh filename=package://ada_description/meshes/collision_hand_2finger.dae; visual mesh filename=package://ada_description/meshes/hand_2finger.dae

File: robots_urdf/ada_with_camera.urdf (robot description, URDF)
Before this commit: robot j2n6s200, 15 links, 14 joints
Links:
- link j2n6s200_joule: geometry collision mesh filename=package://ada_description/meshes/collision_camera_joule_tex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 scale=0.001 0.001 0.00098; visual mesh filename=package://ada_description/meshes/joule_text.dae scale=0.001 0.001 0.001
- link j2n6s200_link_6: geometry collision mesh filename=package://ada_description/meshes/collision_hand_2finger.dae; visual mesh filename=package://ada_description/meshes/hand_2finger.dae
Joints:
- joint j2n6s200_joule: origin xyz=-0.06 -0.051 -0.0163 rpy=-1.57079632679 1.57079632679 0 -> xyz=0.06 0.051 0.0140 rpy=1.57079632679 1.57079632679 0

File: robots_urdf/ada_with_camera_forque.urdf (robot description, URDF)
Before this commit: robot j2n6s200, 17 links, 16 joints
Links:
- link j2n6s200_joule: geometry collision mesh filename=package://ada_description/meshes/collision_camera_joule_tex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 scale=0.001 0.001 0.00098; visual mesh filename=package://ada_description/meshes/joule_text.dae scale=0.001 0.001 0.001
- link j2n6s200_link_6: geometry collision mesh filename=package://ada_description/meshes/collision_hand_2finger.dae; visual mesh filename=package://ada_description/meshes/hand_2finger.dae
Joints:
- joint j2n6s200_joule: origin xyz=-0.06 -0.051 -0.0163 rpy=-1.57079632679 1.57079632679 0 -> xyz=0.06 0.051 0.0140 rpy=1.57079632679 1.57079632679 0

File: robots_urdf/ada_with_forque.urdf (robot description, URDF)
Before this commit: robot j2n6s200, 16 links, 15 joints
Links:
- link j2n6s200_link_6: geometry collision mesh filename=package://ada_description/meshes/collision_hand_2finger.dae; visual mesh filename=package://ada_description/meshes/hand_2finger.dae

Commit message: new camera model

File: robots/camera.xacro (robot description, xacro)
@@ -17,7 +17,7 @@
     <link name="${prefix}_joule">
       <visual>
-        <origin rpy="0 0 0" xyz="0 0 0"/>
+        <origin  rpy="0 0 0" xyz="-0.014 -0.062 -0.023"  />
         <geometry>
-          <mesh filename="package://ada_description/meshes/joule_text.dae" scale="0.001 0.001 0.001"/>
+          <mesh filename="package://ada_description/meshes/camera_joule.dae" scale="0.001 0.001 0.001"/>
         </geometry>
       <material name="carbon_fiber">
@@ -28,5 +28,5 @@
         <origin  rpy="0 0 0" xyz="-0.014 -0.072 -0.033"/>
         <geometry>
-          <mesh filename="package://ada_description/meshes/collision_camera_joule_tex.dae" scale="0.001 0.001 0.00098"/>
+          <mesh filename="package://ada_description/meshes/collision_camera_joule.dae" scale="0.001 0.001 0.00098"/>
         </geometry>
       </collision>

File: robots/j2n6s200.xacro (robot description, xacro)
@@ -95,5 +95,5 @@
     <property name="joint_hand_base_origin_xyz" value="0 0 0" />
     <property name="joint_hand_base_origin_rpy" value="0 0 0" />
-    <xacro:macro name="j2n6s200" params="base_parent use_final_ring:=true prefix:=j2n6s200">
+    <xacro:macro name="j2n6s200" params="base_parent hide_final_ring:=false prefix:=j2n6s200">
         <!--xacro:gazebo_config robot_namespace="${prefix}"/-->
         <xacro:kinova_armlink link_name="${prefix}_link_base" link_mesh="${link_base_mesh}" mesh_no="${link_base_mesh_no}"/>
@@ -109,5 +109,5 @@
         <xacro:kinova_armlink link_name="${prefix}_link_5" link_mesh="${link_5_mesh}" use_ring_mesh="true" ring_mesh="ring_small" mesh_no="${link_5_mesh_no}"/>
         <xacro:kinova_armjoint joint_name="${prefix}_joint_5" type="${joint_5_type}" parent="${prefix}_link_4" child="${prefix}_link_5" joint_axis_xyz="${joint_5_axis_xyz}" joint_origin_xyz="${joint_5_origin_xyz}" joint_origin_rpy="${joint_5_origin_rpy}" joint_lower_limit="${joint_5_lower_limit}" joint_upper_limit="${joint_5_upper_limit}"/>
-        <xacro:kinova_armlink link_name="${prefix}_link_6" link_mesh="${link_6_mesh}" use_ring_mesh="${use_final_ring}" ring_mesh="ring_small" mesh_no="${link_6_mesh_no}"/>
+        <xacro:kinova_armlink link_name="${prefix}_link_6" link_mesh="${link_6_mesh}" use_ring_mesh="${'false' == hide_final_ring}" ring_mesh="ring_small" mesh_no="${link_6_mesh_no}"/>
         <xacro:kinova_armjoint joint_name="${prefix}_joint_6" type="${joint_6_type}" parent="${prefix}_link_5" child="${prefix}_link_6" joint_axis_xyz="${joint_6_axis_xyz}" joint_origin_xyz="${joint_6_origin_xyz}" joint_origin_rpy="${joint_6_origin_rpy}" joint_lower_limit="${joint_6_lower_limit}" joint_upper_limit="${joint_6_upper_limit}"/>
         <xacro:kinova_virtual_link link_name="${prefix}_end_effector"/>

File: robots/j2n6s200_standalone.xacro (robot description, xacro)
@@ -22,5 +22,6 @@
   <property name="robot_root" value="world" />
   <property name="prefix" value="j2n6s200" />
-  <xacro:j2n6s200  base_parent="${robot_root}" use_final_ring="'false'"/>
+  <xacro:j2n6s200  base_parent="${robot_root}" hide_final_ring="$(arg with_camera)"/>
+  <!--xacro:j2n6s200  base_parent="${robot_root}" /-->
   <xacro:if value="$(arg with_camera)">
     <xacro:camera  camera_parent="${prefix}_link_6"/>

File: robots_urdf/ada.urdf (robot description, URDF)
Before this commit: robot j2n6s200, 14 links, 13 joints
Links:
- link j2n6s200_link_6: geometry collision mesh filename=package://ada_description/meshes/collision_hand_2finger.dae; visual mesh filename=package://ada_description/meshes/hand_2finger.dae

File: robots_urdf/ada_with_camera.urdf (robot description, URDF)
Before this commit: robot j2n6s200, 15 links, 14 joints
Links:
- link j2n6s200_joule: geometry collision mesh filename=package://ada_description/meshes/collision_camera_joule.dae scale=0.001 0.001 0.00098; visual mesh filename=package://ada_description/meshes/camera_joule.dae scale=0.001 0.001 0.001

File: robots_urdf/ada_with_camera_forque.urdf (robot description, URDF)
Before this commit: robot j2n6s200, 17 links, 16 joints
Links:
- link j2n6s200_joule: geometry collision mesh filename=package://ada_description/meshes/collision_camera_joule.dae scale=0.001 0.001 0.00098; visual mesh filename=package://ada_description/meshes/camera_joule.dae scale=0.001 0.001 0.001

File: robots_urdf/ada_with_forque.urdf (robot description, URDF)
Before this commit: robot j2n6s200, 16 links, 15 joints
Links:
- link j2n6s200_link_6: geometry collision mesh filename=package://ada_description/meshes/collision_hand_2finger.dae; visual mesh filename=package://ada_description/meshes/hand_2finger.dae
