Commit message: addressed PR comments

File: robots/camera.xacro (robot description, xacro)
@@ -2,15 +2,4 @@
 <!-- j2_6n refers to jaco v2 6DOF non-spherical -->
 <root xmlns:xi="http://www.w3.org/2001/XInclude"
-    xmlns:gazebo="http://playerstage.sourceforge.net/gazebo/xmlschema/#gz"
-    xmlns:model="http://playerstage.sourceforge.net/gazebo/xmlschema/#model"
-    xmlns:sensor="http://playerstage.sourceforge.net/gazebo/xmlschema/#sensor"
-    xmlns:body="http://playerstage.sourceforge.net/gazebo/xmlschema/#body"
-    xmlns:geom="http://playerstage.sourceforge.net/gazebo/xmlschema/#geom"
-    xmlns:joint="http://playerstage.sourceforge.net/gazebo/xmlschema/#joint"
-    xmlns:controller="http://playerstage.sourceforge.net/gazebo/xmlschema/#controller"
-    xmlns:interface="http://playerstage.sourceforge.net/gazebo/xmlschema/#interface"
-    xmlns:rendering="http://playerstage.sourceforge.net/gazebo/xmlschema/#rendering"
-    xmlns:renderable="http://playerstage.sourceforge.net/gazebo/xmlschema/#renderable"
-    xmlns:physics="http://playerstage.sourceforge.net/gazebo/xmlschema/#physics"
     xmlns:xacro="http://ros.org/wiki/xacro">
   <xacro:macro name="camera" params="camera_parent prefix:=j2n6s200">

File: robots/forque.xacro (robot description, xacro)
@@ -2,15 +2,4 @@
 <!-- j2_6n refers to jaco v2 6DOF non-spherical -->
 <root xmlns:xi="http://www.w3.org/2001/XInclude"
-    xmlns:gazebo="http://playerstage.sourceforge.net/gazebo/xmlschema/#gz"
-    xmlns:model="http://playerstage.sourceforge.net/gazebo/xmlschema/#model"
-    xmlns:sensor="http://playerstage.sourceforge.net/gazebo/xmlschema/#sensor"
-    xmlns:body="http://playerstage.sourceforge.net/gazebo/xmlschema/#body"
-    xmlns:geom="http://playerstage.sourceforge.net/gazebo/xmlschema/#geom"
-    xmlns:joint="http://playerstage.sourceforge.net/gazebo/xmlschema/#joint"
-    xmlns:controller="http://playerstage.sourceforge.net/gazebo/xmlschema/#controller"
-    xmlns:interface="http://playerstage.sourceforge.net/gazebo/xmlschema/#interface"
-    xmlns:rendering="http://playerstage.sourceforge.net/gazebo/xmlschema/#rendering"
-    xmlns:renderable="http://playerstage.sourceforge.net/gazebo/xmlschema/#renderable"
-    xmlns:physics="http://playerstage.sourceforge.net/gazebo/xmlschema/#physics"
     xmlns:xacro="http://ros.org/wiki/xacro">
   <xacro:macro name="forque" params="forque_parent prefix:=j2n6s200">
@@ -29,9 +18,4 @@
         </geometry>
       </collision>
-      <!-- <inertial>
-        <mass value="0.01"/>
-        <origin xyz="0.022 0 0"/>
-        <inertia ixx="7.8999684e-07" ixy="0" ixz="0" iyy="7.8999684e-07" iyz="0" izz="8e-08"/>
-      </inertial> -->
     </link>
     <joint name="j2n6s200_joint_forque" type="fixed">

File: robots/j2n6s200.xacro (robot description, xacro)
@@ -2,20 +2,7 @@
 <!-- j2_6n refers to jaco v2 6DOF non-spherical -->
 <root xmlns:xi="http://www.w3.org/2001/XInclude"
-    xmlns:gazebo="http://playerstage.sourceforge.net/gazebo/xmlschema/#gz"
-    xmlns:model="http://playerstage.sourceforge.net/gazebo/xmlschema/#model"
-    xmlns:sensor="http://playerstage.sourceforge.net/gazebo/xmlschema/#sensor"
-    xmlns:body="http://playerstage.sourceforge.net/gazebo/xmlschema/#body"
-    xmlns:geom="http://playerstage.sourceforge.net/gazebo/xmlschema/#geom"
-    xmlns:joint="http://playerstage.sourceforge.net/gazebo/xmlschema/#joint"
-    xmlns:controller="http://playerstage.sourceforge.net/gazebo/xmlschema/#controller"
-    xmlns:interface="http://playerstage.sourceforge.net/gazebo/xmlschema/#interface"
-    xmlns:rendering="http://playerstage.sourceforge.net/gazebo/xmlschema/#rendering"
-    xmlns:renderable="http://playerstage.sourceforge.net/gazebo/xmlschema/#renderable"
-    xmlns:physics="http://playerstage.sourceforge.net/gazebo/xmlschema/#physics"
     xmlns:xacro="http://ros.org/wiki/xacro">
     <xacro:include filename="$(find ada_description)/robots/kinova_common.xacro" />
     <xacro:include filename="$(find ada_description)/robots/kinova_finger_set.xacro" />
-    <!-- Import all Gazebo-customization elements -->
-    <!--xacro:include filename="$(find ada_description)/robots/kinova.gazebo" /-->
     <property name="link_base_mesh" value="base" />
     <property name="link_1_mesh" value="shoulder" />
@@ -25,10 +12,4 @@
     <property name="link_5_mesh" value="wrist" />
     <property name="link_6_mesh" value="hand_2finger" />
-    <!--Used for conditional arguments for setting inertial parameters
-        base 0, shoulder 1, arm 2, forearm 3, wrist 4, arm_mico 5,
-        arm_half1 (7dof)	6, arm_half2 (7dof) 7, wrist_spherical_1  8, wrist_spherical_2  9
-        fore_arm_mico 10,
-        hand 3 finger 55, hand_2finger 56, finger_proximal 57, finger_distal 58
-    -->
     <property name="link_base_mesh_no" value="0" />
     <property name="link_1_mesh_no" value="1" />

File: robots/j2n6s200_standalone.xacro (robot description, xacro)
@@ -2,15 +2,4 @@
 <!-- j2n6s200 refers to jaco v2 6DOF non-spherical 2fingers -->
 <robot xmlns:xi="http://www.w3.org/2001/XInclude"
-	xmlns:gazebo="http://playerstage.sourceforge.net/gazebo/xmlschema/#gz"
-    xmlns:model="http://playerstage.sourceforge.net/gazebo/xmlschema/#model"
-	xmlns:sensor="http://playerstage.sourceforge.net/gazebo/xmlschema/#sensor"
-	xmlns:body="http://playerstage.sourceforge.net/gazebo/xmlschema/#body"
-    xmlns:geom="http://playerstage.sourceforge.net/gazebo/xmlschema/#geom"
-    xmlns:joint="http://playerstage.sourceforge.net/gazebo/xmlschema/#joint"
-	xmlns:controller="http://playerstage.sourceforge.net/gazebo/xmlschema/#controller"
-	xmlns:interface="http://playerstage.sourceforge.net/gazebo/xmlschema/#interface"
-	xmlns:rendering="http://playerstage.sourceforge.net/gazebo/xmlschema/#rendering"
-    xmlns:renderable="http://playerstage.sourceforge.net/gazebo/xmlschema/#renderable"
-    xmlns:physics="http://playerstage.sourceforge.net/gazebo/xmlschema/#physics"
 	xmlns:xacro="http://ros.org/wiki/xacro" name="j2n6s200">
   <xacro:include filename="$(find ada_description)/robots/j2n6s200.xacro"/>

File: robots/kinova_common.xacro (robot description, xacro)
@@ -1,15 +1,4 @@
 <?xml version="1.0"?>
 <root xmlns:xi="http://www.w3.org/2001/XInclude"
-	xmlns:gazebo="http://playerstage.sourceforge.net/gazebo/xmlschema/#gz"
-    xmlns:model="http://playerstage.sourceforge.net/gazebo/xmlschema/#model"
-	xmlns:sensor="http://playerstage.sourceforge.net/gazebo/xmlschema/#sensor"
-	xmlns:body="http://playerstage.sourceforge.net/gazebo/xmlschema/#body"
-    xmlns:geom="http://playerstage.sourceforge.net/gazebo/xmlschema/#geom"
-    xmlns:joint="http://playerstage.sourceforge.net/gazebo/xmlschema/#joint"
-	xmlns:controller="http://playerstage.sourceforge.net/gazebo/xmlschema/#controller"
-	xmlns:interface="http://playerstage.sourceforge.net/gazebo/xmlschema/#interface"
-	xmlns:rendering="http://playerstage.sourceforge.net/gazebo/xmlschema/#rendering"
-    xmlns:renderable="http://playerstage.sourceforge.net/gazebo/xmlschema/#renderable"
-    xmlns:physics="http://playerstage.sourceforge.net/gazebo/xmlschema/#physics"
 	xmlns:xacro="http://ros.org/wiki/xacro">
 <xacro:include filename="$(find ada_description)/robots/kinova_inertial.xacro" />
@@ -49,5 +38,5 @@
         <child link="${child}"/>
         <axis xyz="${joint_axis_xyz}"/>
-        <limit effort="2000" velocity="1" lower="${joint_lower_limit}" upper="${joint_upper_limit}"/>
+        <limit effort="2000" velocity="1.4" lower="${joint_lower_limit}" upper="${joint_upper_limit}"/>
         <origin xyz="${joint_origin_xyz}" rpy="${joint_origin_rpy}"/>
         <dynamics damping="0.0" friction="0.0"/>

File: robots/kinova_finger_set.xacro (robot description, xacro)
@@ -15,12 +15,4 @@
     xmlns:xacro="http://ros.org/wiki/xacro">
     <xacro:include filename="$(find ada_description)/robots/kinova_common.xacro" />
-    <xacro:macro name="kinova_3fingers" params="link_hand prefix">
-        <!-- finger1 Rot := Ry((1/2)*Pi) . Rx(12.1*((1/180)*Pi)+Pi) . Rz(-52.8*((1/180)*Pi)) -->
-        <xacro:kinova_finger prefix="${prefix}" finger_number="1" hand="${link_hand}" finger_origin_xyz="0.00279 0.03126 -0.11467" finger_origin_rpy="-1.570796327 .649262481663582 1.35961148639407"/>
-        <!-- finger2 Rot := Ry((1/2)*Pi) . Rx(10.58*((1/180)*Pi)) . Rz(-52.8*((1/180)*Pi)) -->
-        <xacro:kinova_finger prefix="${prefix}" finger_number="2" hand="${link_hand}" finger_origin_xyz="0.02226 -0.02707 -0.11482" finger_origin_rpy="-1.570796327 .649262481663582 -1.38614049188413"/>
-        <!-- finger3 Rot := Ry((1/2)*Pi) . Rx(-10.58*((1/180)*Pi)) . Rz(-52.8*((1/180)*Pi)) -->
-        <xacro:kinova_finger prefix="${prefix}" finger_number="3" hand="${link_hand}" finger_origin_xyz="-0.02226 -0.02707 -0.11482" finger_origin_rpy="-1.570796327 .649262481663582 -1.75545216211587"/>
-    </xacro:macro>
     <xacro:macro name="kinova_2fingers" params="link_hand prefix">
         <!-- finger1 Rot := Ry((1/2)*Pi) . Rx(Pi) . Rz(-52.8*((1/180)*Pi)) -->

File: robots/kinova_inertial.xacro (robot description, xacro)
@@ -24,5 +24,4 @@
    wrist_spherical_1  8
    wrist_spherical_2  9
-   hand 3 finger  		55
    hand_2finger   		56
    finger_proximal		57

File: robots_urdf/ada.urdf (robot description, URDF)
Before this commit: robot j2n6s200, 14 links, 13 joints
Joints:
- joint j2n6s200_joint_1: limit lower=-6.28318530718 upper=6.28318530718 effort=2000 velocity=1 -> lower=-6.28318530718 upper=6.28318530718 effort=2000 velocity=1.4
- joint j2n6s200_joint_2: limit lower=0.820304748437 upper=5.46288055874 effort=2000 velocity=1 -> lower=0.820304748437 upper=5.46288055874 effort=2000 velocity=1.4
- joint j2n6s200_joint_3: limit lower=0.331612557879 upper=5.9515727493 effort=2000 velocity=1 -> lower=0.331612557879 upper=5.9515727493 effort=2000 velocity=1.4
- joint j2n6s200_joint_4: limit lower=-6.28318530718 upper=6.28318530718 effort=2000 velocity=1 -> lower=-6.28318530718 upper=6.28318530718 effort=2000 velocity=1.4
- joint j2n6s200_joint_5: limit lower=-6.28318530718 upper=6.28318530718 effort=2000 velocity=1 -> lower=-6.28318530718 upper=6.28318530718 effort=2000 velocity=1.4
- joint j2n6s200_joint_6: limit lower=-6.28318530718 upper=6.28318530718 effort=2000 velocity=1 -> lower=-6.28318530718 upper=6.28318530718 effort=2000 velocity=1.4
- joint j2n6s200_joint_base: limit lower=0 upper=0 effort=2000 velocity=1 -> lower=0 upper=0 effort=2000 velocity=1.4

File: robots_urdf/ada_with_camera.urdf (robot description, URDF)
Before this commit: robot j2n6s200, 15 links, 14 joints
Joints:
- joint j2n6s200_joint_1: limit lower=-6.28318530718 upper=6.28318530718 effort=2000 velocity=1 -> lower=-6.28318530718 upper=6.28318530718 effort=2000 velocity=1.4
- joint j2n6s200_joint_2: limit lower=0.820304748437 upper=5.46288055874 effort=2000 velocity=1 -> lower=0.820304748437 upper=5.46288055874 effort=2000 velocity=1.4
- joint j2n6s200_joint_3: limit lower=0.331612557879 upper=5.9515727493 effort=2000 velocity=1 -> lower=0.331612557879 upper=5.9515727493 effort=2000 velocity=1.4
- joint j2n6s200_joint_4: limit lower=-6.28318530718 upper=6.28318530718 effort=2000 velocity=1 -> lower=-6.28318530718 upper=6.28318530718 effort=2000 velocity=1.4
- joint j2n6s200_joint_5: limit lower=-6.28318530718 upper=6.28318530718 effort=2000 velocity=1 -> lower=-6.28318530718 upper=6.28318530718 effort=2000 velocity=1.4
- joint j2n6s200_joint_6: limit lower=-6.28318530718 upper=6.28318530718 effort=2000 velocity=1 -> lower=-6.28318530718 upper=6.28318530718 effort=2000 velocity=1.4
- joint j2n6s200_joint_base: limit lower=0 upper=0 effort=2000 velocity=1 -> lower=0 upper=0 effort=2000 velocity=1.4

File: robots_urdf/ada_with_camera_forque.urdf (robot description, URDF)
Before this commit: robot j2n6s200, 17 links, 16 joints
Joints:
- joint j2n6s200_joint_1: limit lower=-6.28318530718 upper=6.28318530718 effort=2000 velocity=1 -> lower=-6.28318530718 upper=6.28318530718 effort=2000 velocity=1.4
- joint j2n6s200_joint_2: limit lower=0.820304748437 upper=5.46288055874 effort=2000 velocity=1 -> lower=0.820304748437 upper=5.46288055874 effort=2000 velocity=1.4
- joint j2n6s200_joint_3: limit lower=0.331612557879 upper=5.9515727493 effort=2000 velocity=1 -> lower=0.331612557879 upper=5.9515727493 effort=2000 velocity=1.4
- joint j2n6s200_joint_4: limit lower=-6.28318530718 upper=6.28318530718 effort=2000 velocity=1 -> lower=-6.28318530718 upper=6.28318530718 effort=2000 velocity=1.4
- joint j2n6s200_joint_5: limit lower=-6.28318530718 upper=6.28318530718 effort=2000 velocity=1 -> lower=-6.28318530718 upper=6.28318530718 effort=2000 velocity=1.4
- joint j2n6s200_joint_6: limit lower=-6.28318530718 upper=6.28318530718 effort=2000 velocity=1 -> lower=-6.28318530718 upper=6.28318530718 effort=2000 velocity=1.4
- joint j2n6s200_joint_base: limit lower=0 upper=0 effort=2000 velocity=1 -> lower=0 upper=0 effort=2000 velocity=1.4

File: robots_urdf/ada_with_forque.urdf (robot description, URDF)
Before this commit: robot j2n6s200, 16 links, 15 joints
Joints:
- joint j2n6s200_joint_1: limit lower=-6.28318530718 upper=6.28318530718 effort=2000 velocity=1 -> lower=-6.28318530718 upper=6.28318530718 effort=2000 velocity=1.4
- joint j2n6s200_joint_2: limit lower=0.820304748437 upper=5.46288055874 effort=2000 velocity=1 -> lower=0.820304748437 upper=5.46288055874 effort=2000 velocity=1.4
- joint j2n6s200_joint_3: limit lower=0.331612557879 upper=5.9515727493 effort=2000 velocity=1 -> lower=0.331612557879 upper=5.9515727493 effort=2000 velocity=1.4
- joint j2n6s200_joint_4: limit lower=-6.28318530718 upper=6.28318530718 effort=2000 velocity=1 -> lower=-6.28318530718 upper=6.28318530718 effort=2000 velocity=1.4
- joint j2n6s200_joint_5: limit lower=-6.28318530718 upper=6.28318530718 effort=2000 velocity=1 -> lower=-6.28318530718 upper=6.28318530718 effort=2000 velocity=1.4
- joint j2n6s200_joint_6: limit lower=-6.28318530718 upper=6.28318530718 effort=2000 velocity=1 -> lower=-6.28318530718 upper=6.28318530718 effort=2000 velocity=1.4
- joint j2n6s200_joint_base: limit lower=0 upper=0 effort=2000 velocity=1 -> lower=0 upper=0 effort=2000 velocity=1.4

Commit message: fixed joule collision model and forque translation

File: robots/camera.xacro (robot description, xacro)
@@ -8,5 +8,6 @@
         <origin  rpy="0 0 0" xyz="-0.014 -0.062 -0.023"  />
         <geometry>
-          <mesh filename="package://ada_description/meshes/camera_joule.dae" scale="0.001 0.001 0.001"/>
+          <!-- <mesh filename="package://ada_description/meshes/camera_joule.dae" scale="0.001 0.001 0.001"/> -->
+          <mesh filename="package://ada_description/meshes/collision_camera_joule.dae" scale="0.001 0.001 0.00098"/>
         </geometry>
       <material name="carbon_fiber">
@@ -15,5 +16,5 @@
       </visual>
       <collision>
-        <origin  rpy="0 0 0" xyz="-0.014 -0.072 -0.033"/>
+        <origin  rpy="0 0 0" xyz="-0.014 -0.062 -0.023"  />
         <geometry>
           <mesh filename="package://ada_description/meshes/collision_camera_joule.dae" scale="0.001 0.001 0.00098"/>

File: robots/forque.xacro (robot description, xacro)
@@ -23,5 +23,5 @@
       <child link="j2n6s200_forque"/>
       <axis xyz="0 0 1"/>
-      <origin rpy="3.14 0 0" xyz="0.01 -0.000 0.078"/>
+      <origin rpy="3.14 0 0" xyz="-0.003 -0.0013 0.065"/>
       <limit effort="2000" lower="0" upper="2" velocity="1"/>
     </joint>

File: robots_urdf/ada_with_camera.urdf (robot description, URDF)
Before this commit: robot j2n6s200, 16 links, 15 joints
Links:
- link j2n6s200_joule: geometry collision mesh filename=package://ada_description/meshes/collision_camera_joule.dae scale=0.001 0.001 0.00098; visual mesh filename=package://ada_description/meshes/collision_camera_joule.dae scale=0.001 0.001 0.00098

File: robots_urdf/ada_with_camera_forque.urdf (robot description, URDF)
Before this commit: robot j2n6s200, 19 links, 18 joints
Links:
- link j2n6s200_joule: geometry collision mesh filename=package://ada_description/meshes/collision_camera_joule.dae scale=0.001 0.001 0.00098; visual mesh filename=package://ada_description/meshes/collision_camera_joule.dae scale=0.001 0.001 0.00098
Joints:
- joint j2n6s200_joint_forque: origin xyz=0.01 -0.000 0.078 rpy=3.14 0 0 -> xyz=-0.003 -0.0013 0.065 rpy=3.14 0 0

File: robots_urdf/ada_with_forque.urdf (robot description, URDF)
Before this commit: robot j2n6s200, 18 links, 17 joints
Joints:
- joint j2n6s200_joint_forque: origin xyz=0.01 -0.000 0.078 rpy=3.14 0 0 -> xyz=-0.003 -0.0013 0.065 rpy=3.14 0 0
