Commit message: removed camera model, changed position of forque

File: robots/camera.xacro (robot description, xacro)
@@ -7,8 +7,8 @@
       <visual>
         <origin  rpy="0 0 0" xyz="-0.014 -0.062 -0.023"  />
-        <geometry>
+        <!-- <geometry> -->
           <!-- <mesh filename="package://ada_description/meshes/camera_joule.dae" scale="0.001 0.001 0.001"/> -->
-          <mesh filename="package://ada_description/meshes/collision_camera_joule.dae" scale="0.001 0.001 0.00098"/>
-        </geometry>
+          <!-- <mesh filename="package://ada_description/meshes/collision_camera_joule.dae" scale="0.001 0.001 0.00098"/> -->
+        <!-- </geometry> -->
       <material name="carbon_fiber">
           <color rgba="0.792156862745098 0.819607843137255 0.933333333333333 1"/>

File: robots/forque.xacro (robot description, xacro)
@@ -23,5 +23,5 @@
       <child link="j2n6s200_forque"/>
       <axis xyz="0 0 1"/>
-      <origin rpy="3.14 0 0" xyz="-0.003 -0.0013 0.065"/>
+      <origin rpy="3.14 0 0" xyz="0.008 0.0018 0.0582"/>
       <limit effort="2000" lower="0" upper="2" velocity="1"/>
     </joint>

File: robots/j2n6s200.xacro (robot description, xacro)
@@ -5,80 +5,80 @@
     <xacro:include filename="$(find ada_description)/robots/kinova_common.xacro" />
     <xacro:include filename="$(find ada_description)/robots/kinova_finger_set.xacro" />
-    <property name="link_base_mesh" value="base" />
-    <property name="link_1_mesh" value="shoulder" />
-    <property name="link_2_mesh" value="arm" />
-    <property name="link_3_mesh" value="forearm" />
-    <property name="link_4_mesh" value="wrist" />
-    <property name="link_5_mesh" value="wrist" />
-    <property name="link_6_mesh" value="hand_2finger" />
-    <property name="link_base_mesh_no" value="0" />
-    <property name="link_1_mesh_no" value="1" />
-    <property name="link_2_mesh_no" value="2" />
-    <property name="link_3_mesh_no" value="3" />
-    <property name="link_4_mesh_no" value="4" />
-    <property name="link_5_mesh_no" value="4" />
-    <property name="link_6_mesh_no" value="56" />
-    <property name="joint_base" value="joint_base" />
-    <property name="joint_base_type" value="fixed" />
-    <property name="joint_base_axis_xyz" value="0 0 0" />
-    <property name="joint_base_origin_xyz" value="0 0 0" />
-    <property name="joint_base_origin_rpy" value="0 0 0" />
-    <property name="joint_1" value="joint_1" />
-    <property name="joint_1_type" value="revolute" />
-    <property name="joint_1_axis_xyz" value="0 0 1" />
-    <property name="joint_1_origin_xyz" value="0 0 0.15675" />
-    <property name="joint_1_origin_rpy" value="0 ${J_PI} 0" />
-    <property name="joint_1_lower_limit" value="${-2*J_PI}" />
-    <property name="joint_1_upper_limit" value="${2*J_PI}" />
-    <property name="joint_2" value="joint_2" />
-    <property name="joint_2_type" value="revolute" />
-    <property name="joint_2_axis_xyz" value="0 0 1" />
-    <property name="joint_2_origin_xyz" value="0 0.0016 -0.11875" />
-    <property name="joint_2_origin_rpy" value="-${J_PI/2} 0 ${J_PI}" />
-    <property name="joint_2_lower_limit" value="${47/180*J_PI}" />
-    <property name="joint_2_upper_limit" value="${313/180*J_PI}" />
-    <property name="joint_3" value="joint_3" />
-    <property name="joint_3_type" value="revolute" />
-    <property name="joint_3_axis_xyz" value="0 0 1" />
-    <property name="joint_3_origin_xyz" value="0 -0.410 0" />
-    <property name="joint_3_origin_rpy" value="0 ${J_PI} 0" />
-    <property name="joint_3_lower_limit" value="${19/180*J_PI}" />
-    <property name="joint_3_upper_limit" value="${341/180*J_PI}" />
-    <property name="joint_4" value="joint_4" />
-    <property name="joint_4_type" value="revolute" />
-    <property name="joint_4_axis_xyz" value="0 0 1" />
-    <property name="joint_4_origin_xyz" value="0 0.2073 -0.0114" />
-    <property name="joint_4_origin_rpy" value="-${J_PI/2} 0 ${J_PI}" />
-    <property name="joint_4_lower_limit" value="${-2*J_PI}" />
-    <property name="joint_4_upper_limit" value="${2*J_PI}" />
-    <property name="joint_5" value="joint_5" />
-    <property name="joint_5_type" value="revolute" />
-    <property name="joint_5_axis_xyz" value="0 0 1" />
-    <property name="joint_5_origin_xyz" value="0 -0.03703 -0.06414" />
-    <property name="joint_5_origin_rpy" value="${J_PI/3} 0 ${J_PI}" />
-    <property name="joint_5_lower_limit" value="${-2*J_PI}" />
-    <property name="joint_5_upper_limit" value="${2*J_PI}" />
-    <property name="joint_6" value="joint_6" />
-    <property name="joint_6_type" value="revolute" />
-    <property name="joint_6_axis_xyz" value="0 0 1" />
-    <property name="joint_6_origin_xyz" value="0 -0.03703 -0.06414" />
-    <property name="joint_6_origin_rpy" value="${J_PI/3} 0 ${J_PI}" />
-    <property name="joint_6_lower_limit" value="${-2*J_PI}" />
-    <property name="joint_6_upper_limit" value="${2*J_PI}" />
-    <property name="joint_end_effector" value="end_effector_offset" />
-    <property name="joint_end_effector_type" value="fixed" />
-    <property name="joint_end_effector_axis_xyz" value="0 0 0" />
-    <property name="joint_end_effector_origin_xyz" value="0 0 -0.1600" />
-    <property name="joint_end_effector_origin_rpy" value="${J_PI} 0 0" />
-    <property name="joint_hand_tip" value="end_effector_offset" />
-    <property name="joint_hand_tip_type" value="fixed" />
-    <property name="joint_hand_tip_axis_xyz" value="0 0 0" />
-    <property name="joint_hand_tip_origin_xyz" value="0 0 0.0370" />
-    <property name="joint_hand_tip_origin_rpy" value="0 0 0" />
-    <property name="joint_hand_base" value="hand_base" />
-    <property name="joint_hand_base_type" value="fixed" />
-    <property name="joint_hand_base_axis_xyz" value="0 0 0" />
-    <property name="joint_hand_base_origin_xyz" value="0 0 0" />
-    <property name="joint_hand_base_origin_rpy" value="0 0 0" />
+    <xacro:property name="link_base_mesh" value="base" />
+    <xacro:property name="link_1_mesh" value="shoulder" />
+    <xacro:property name="link_2_mesh" value="arm" />
+    <xacro:property name="link_3_mesh" value="forearm" />
+    <xacro:property name="link_4_mesh" value="wrist" />
+    <xacro:property name="link_5_mesh" value="wrist" />
+    <xacro:property name="link_6_mesh" value="hand_2finger" />
+    <xacro:property name="link_base_mesh_no" value="0" />
+    <xacro:property name="link_1_mesh_no" value="1" />
+    <xacro:property name="link_2_mesh_no" value="2" />
+    <xacro:property name="link_3_mesh_no" value="3" />
+    <xacro:property name="link_4_mesh_no" value="4" />
+    <xacro:property name="link_5_mesh_no" value="4" />
+    <xacro:property name="link_6_mesh_no" value="56" />
+    <xacro:property name="joint_base" value="joint_base" />
+    <xacro:property name="joint_base_type" value="fixed" />
+    <xacro:property name="joint_base_axis_xyz" value="0 0 0" />
+    <xacro:property name="joint_base_origin_xyz" value="0 0 0" />
+    <xacro:property name="joint_base_origin_rpy" value="0 0 0" />
+    <xacro:property name="joint_1" value="joint_1" />
+    <xacro:property name="joint_1_type" value="revolute" />
+    <xacro:property name="joint_1_axis_xyz" value="0 0 1" />
+    <xacro:property name="joint_1_origin_xyz" value="0 0 0.15675" />
+    <xacro:property name="joint_1_origin_rpy" value="0 ${J_PI} 0" />
+    <xacro:property name="joint_1_lower_limit" value="${-2*J_PI}" />
+    <xacro:property name="joint_1_upper_limit" value="${2*J_PI}" />
+    <xacro:property name="joint_2" value="joint_2" />
+    <xacro:property name="joint_2_type" value="revolute" />
+    <xacro:property name="joint_2_axis_xyz" value="0 0 1" />
+    <xacro:property name="joint_2_origin_xyz" value="0 0.0016 -0.11875" />
+    <xacro:property name="joint_2_origin_rpy" value="-${J_PI/2} 0 ${J_PI}" />
+    <xacro:property name="joint_2_lower_limit" value="${47/180*J_PI}" />
+    <xacro:property name="joint_2_upper_limit" value="${313/180*J_PI}" />
+    <xacro:property name="joint_3" value="joint_3" />
+    <xacro:property name="joint_3_type" value="revolute" />
+    <xacro:property name="joint_3_axis_xyz" value="0 0 1" />
+    <xacro:property name="joint_3_origin_xyz" value="0 -0.410 0" />
+    <xacro:property name="joint_3_origin_rpy" value="0 ${J_PI} 0" />
+    <xacro:property name="joint_3_lower_limit" value="${19/180*J_PI}" />
+    <xacro:property name="joint_3_upper_limit" value="${341/180*J_PI}" />
+    <xacro:property name="joint_4" value="joint_4" />
+    <xacro:property name="joint_4_type" value="revolute" />
+    <xacro:property name="joint_4_axis_xyz" value="0 0 1" />
+    <xacro:property name="joint_4_origin_xyz" value="0 0.2073 -0.0114" />
+    <xacro:property name="joint_4_origin_rpy" value="-${J_PI/2} 0 ${J_PI}" />
+    <xacro:property name="joint_4_lower_limit" value="${-2*J_PI}" />
+    <xacro:property name="joint_4_upper_limit" value="${2*J_PI}" />
+    <xacro:property name="joint_5" value="joint_5" />
+    <xacro:property name="joint_5_type" value="revolute" />
+    <xacro:property name="joint_5_axis_xyz" value="0 0 1" />
+    <xacro:property name="joint_5_origin_xyz" value="0 -0.03703 -0.06414" />
+    <xacro:property name="joint_5_origin_rpy" value="${J_PI/3} 0 ${J_PI}" />
+    <xacro:property name="joint_5_lower_limit" value="${-2*J_PI}" />
+    <xacro:property name="joint_5_upper_limit" value="${2*J_PI}" />
+    <xacro:property name="joint_6" value="joint_6" />
+    <xacro:property name="joint_6_type" value="revolute" />
+    <xacro:property name="joint_6_axis_xyz" value="0 0 1" />
+    <xacro:property name="joint_6_origin_xyz" value="0 -0.03703 -0.06414" />
+    <xacro:property name="joint_6_origin_rpy" value="${J_PI/3} 0 ${J_PI}" />
+    <xacro:property name="joint_6_lower_limit" value="${-2*J_PI}" />
+    <xacro:property name="joint_6_upper_limit" value="${2*J_PI}" />
+    <xacro:property name="joint_end_effector" value="end_effector_offset" />
+    <xacro:property name="joint_end_effector_type" value="fixed" />
+    <xacro:property name="joint_end_effector_axis_xyz" value="0 0 0" />
+    <xacro:property name="joint_end_effector_origin_xyz" value="0 0 -0.1600" />
+    <xacro:property name="joint_end_effector_origin_rpy" value="${J_PI} 0 0" />
+    <xacro:property name="joint_hand_tip" value="end_effector_offset" />
+    <xacro:property name="joint_hand_tip_type" value="fixed" />
+    <xacro:property name="joint_hand_tip_axis_xyz" value="0 0 0" />
+    <xacro:property name="joint_hand_tip_origin_xyz" value="0 0 0.0370" />
+    <xacro:property name="joint_hand_tip_origin_rpy" value="0 0 0" />
+    <xacro:property name="joint_hand_base" value="hand_base" />
+    <xacro:property name="joint_hand_base_type" value="fixed" />
+    <xacro:property name="joint_hand_base_axis_xyz" value="0 0 0" />
+    <xacro:property name="joint_hand_base_origin_xyz" value="0 0 0" />
+    <xacro:property name="joint_hand_base_origin_rpy" value="0 0 0" />
     <xacro:macro name="j2n6s200" params="base_parent hide_final_ring:=false prefix:=j2n6s200">
         <!--xacro:gazebo_config robot_namespace="${prefix}"/-->

File: robots/j2n6s200_standalone.xacro (robot description, xacro)
@@ -9,6 +9,6 @@
   <xacro:arg name="with_forque" default="false" />
   <link name="world"/>
-  <property name="robot_root" value="world" />
-  <property name="prefix" value="j2n6s200" />
+  <xacro:property name="robot_root" value="world" />
+  <xacro:property name="prefix" value="j2n6s200" />
   <xacro:j2n6s200  base_parent="${robot_root}" hide_final_ring="$(arg with_camera)"/>
   <!--xacro:j2n6s200  base_parent="${robot_root}" /-->

File: robots/kinova_common.xacro (robot description, xacro)
@@ -3,5 +3,5 @@
 	xmlns:xacro="http://ros.org/wiki/xacro">
 <xacro:include filename="$(find ada_description)/robots/kinova_inertial.xacro" />
-    <property name="J_PI" value="3.1415926535897931" />
+    <xacro:property name="J_PI" value="3.1415926535897931" />
     <xacro:macro name="kinova_armlink" params="link_name link_mesh ring_mesh:=ring_big use_ring_mesh:=false mesh_no">
         <link name="${link_name}">
@@ -38,5 +38,5 @@
         <child link="${child}"/>
         <axis xyz="${joint_axis_xyz}"/>
-        <limit effort="2000" velocity="0.8" lower="${joint_lower_limit}" upper="${joint_upper_limit}"/>
+        <limit effort="2000" velocity="1.0" lower="${joint_lower_limit}" upper="${joint_upper_limit}"/>
         <origin xyz="${joint_origin_xyz}" rpy="${joint_origin_rpy}"/>
         <dynamics damping="0.0" friction="0.0"/>

File: robots_urdf/ada.urdf (robot description, URDF)
Before this commit: robot j2n6s200, 15 links, 14 joints
Joints:
- joint j2n6s200_joint_1: limit lower=-6.28318530718 upper=6.28318530718 effort=2000 velocity=0.8 -> lower=-6.28318530718 upper=6.28318530718 effort=2000 velocity=1.0
- joint j2n6s200_joint_2: limit lower=0.820304748437 upper=5.46288055874 effort=2000 velocity=0.8 -> lower=0.820304748437 upper=5.46288055874 effort=2000 velocity=1.0
- joint j2n6s200_joint_3: limit lower=0.331612557879 upper=5.9515727493 effort=2000 velocity=0.8 -> lower=0.331612557879 upper=5.9515727493 effort=2000 velocity=1.0
- joint j2n6s200_joint_4: limit lower=-6.28318530718 upper=6.28318530718 effort=2000 velocity=0.8 -> lower=-6.28318530718 upper=6.28318530718 effort=2000 velocity=1.0
- joint j2n6s200_joint_5: limit lower=-6.28318530718 upper=6.28318530718 effort=2000 velocity=0.8 -> lower=-6.28318530718 upper=6.28318530718 effort=2000 velocity=1.0
- joint j2n6s200_joint_6: limit lower=-6.28318530718 upper=6.28318530718 effort=2000 velocity=0.8 -> lower=-6.28318530718 upper=6.28318530718 effort=2000 velocity=1.0
- joint j2n6s200_joint_base: limit lower=0 upper=0 effort=2000 velocity=0.8 -> lower=0 upper=0 effort=2000 velocity=1.0

File: robots_urdf/ada_with_camera.urdf (robot description, URDF)
Before this commit: robot j2n6s200, 16 links, 15 joints
Links:
- link j2n6s200_joule: geometry collision mesh filename=package://ada_description/meshes/collision_camera_joule.dae scale=0.001 0.001 0.00098
Joints:
- joint j2n6s200_joint_1: limit lower=-6.28318530718 upper=6.28318530718 effort=2000 velocity=0.8 -> lower=-6.28318530718 upper=6.28318530718 effort=2000 velocity=1.0
- joint j2n6s200_joint_2: limit lower=0.820304748437 upper=5.46288055874 effort=2000 velocity=0.8 -> lower=0.820304748437 upper=5.46288055874 effort=2000 velocity=1.0
- joint j2n6s200_joint_3: limit lower=0.331612557879 upper=5.9515727493 effort=2000 velocity=0.8 -> lower=0.331612557879 upper=5.9515727493 effort=2000 velocity=1.0
- joint j2n6s200_joint_4: limit lower=-6.28318530718 upper=6.28318530718 effort=2000 velocity=0.8 -> lower=-6.28318530718 upper=6.28318530718 effort=2000 velocity=1.0
- joint j2n6s200_joint_5: limit lower=-6.28318530718 upper=6.28318530718 effort=2000 velocity=0.8 -> lower=-6.28318530718 upper=6.28318530718 effort=2000 velocity=1.0
- joint j2n6s200_joint_6: limit lower=-6.28318530718 upper=6.28318530718 effort=2000 velocity=0.8 -> lower=-6.28318530718 upper=6.28318530718 effort=2000 velocity=1.0
- joint j2n6s200_joint_base: limit lower=0 upper=0 effort=2000 velocity=0.8 -> lower=0 upper=0 effort=2000 velocity=1.0

File: robots_urdf/ada_with_camera_forque.urdf (robot description, URDF)
Before this commit: robot j2n6s200, 19 links, 18 joints
Links:
- link j2n6s200_joule: geometry collision mesh filename=package://ada_description/meshes/collision_camera_joule.dae scale=0.001 0.001 0.00098
Joints:
- joint j2n6s200_joint_1: limit lower=-6.28318530718 upper=6.28318530718 effort=2000 velocity=0.8 -> lower=-6.28318530718 upper=6.28318530718 effort=2000 velocity=1.0
- joint j2n6s200_joint_2: limit lower=0.820304748437 upper=5.46288055874 effort=2000 velocity=0.8 -> lower=0.820304748437 upper=5.46288055874 effort=2000 velocity=1.0
- joint j2n6s200_joint_3: limit lower=0.331612557879 upper=5.9515727493 effort=2000 velocity=0.8 -> lower=0.331612557879 upper=5.9515727493 effort=2000 velocity=1.0
- joint j2n6s200_joint_4: limit lower=-6.28318530718 upper=6.28318530718 effort=2000 velocity=0.8 -> lower=-6.28318530718 upper=6.28318530718 effort=2000 velocity=1.0
- joint j2n6s200_joint_5: limit lower=-6.28318530718 upper=6.28318530718 effort=2000 velocity=0.8 -> lower=-6.28318530718 upper=6.28318530718 effort=2000 velocity=1.0
- joint j2n6s200_joint_6: limit lower=-6.28318530718 upper=6.28318530718 effort=2000 velocity=0.8 -> lower=-6.28318530718 upper=6.28318530718 effort=2000 velocity=1.0
- joint j2n6s200_joint_base: limit lower=0 upper=0 effort=2000 velocity=0.8 -> lower=0 upper=0 effort=2000 velocity=1.0
- joint j2n6s200_joint_forque: origin xyz=-0.003 -0.0013 0.065 rpy=3.14 0 0 -> xyz=0.008 0.0018 0.0582 rpy=3.14 0 0

File: robots_urdf/ada_with_forque.urdf (robot description, URDF)
Before this commit: robot j2n6s200, 18 links, 17 joints
Joints:
- joint j2n6s200_joint_1: limit lower=-6.28318530718 upper=6.28318530718 effort=2000 velocity=0.8 -> lower=-6.28318530718 upper=6.28318530718 effort=2000 velocity=1.0
- joint j2n6s200_joint_2: limit lower=0.820304748437 upper=5.46288055874 effort=2000 velocity=0.8 -> lower=0.820304748437 upper=5.46288055874 effort=2000 velocity=1.0
- joint j2n6s200_joint_3: limit lower=0.331612557879 upper=5.9515727493 effort=2000 velocity=0.8 -> lower=0.331612557879 upper=5.9515727493 effort=2000 velocity=1.0
- joint j2n6s200_joint_4: limit lower=-6.28318530718 upper=6.28318530718 effort=2000 velocity=0.8 -> lower=-6.28318530718 upper=6.28318530718 effort=2000 velocity=1.0
- joint j2n6s200_joint_5: limit lower=-6.28318530718 upper=6.28318530718 effort=2000 velocity=0.8 -> lower=-6.28318530718 upper=6.28318530718 effort=2000 velocity=1.0
- joint j2n6s200_joint_6: limit lower=-6.28318530718 upper=6.28318530718 effort=2000 velocity=0.8 -> lower=-6.28318530718 upper=6.28318530718 effort=2000 velocity=1.0
- joint j2n6s200_joint_base: limit lower=0 upper=0 effort=2000 velocity=0.8 -> lower=0 upper=0 effort=2000 velocity=1.0
- joint j2n6s200_joint_forque: origin xyz=-0.003 -0.0013 0.065 rpy=3.14 0 0 -> xyz=0.008 0.0018 0.0582 rpy=3.14 0 0

Commit message: new joule model

File: robots/camera.xacro (robot description, xacro)
@@ -8,6 +8,6 @@
         <origin  rpy="0 0 0" xyz="-0.014 -0.062 -0.023"  />
         <geometry>
-          <!-- <mesh filename="package://ada_description/meshes/camera_joule.dae" scale="0.001 0.001 0.001"/> -->
-          <mesh filename="package://ada_description/meshes/collision_camera_joule.dae" scale="0.001 0.001 0.00098"/>
+          <mesh filename="package://ada_description/meshes/camera_joule.dae" scale="0.001 0.001 0.001"/>
+          <!-- <mesh filename="package://ada_description/meshes/collision_camera_joule.dae" scale="0.001 0.001 0.00098"/> -->
         </geometry>
       <material name="carbon_fiber">

File: robots_urdf/ada_with_camera.urdf (robot description, URDF)
Before this commit: robot j2n6s200, 16 links, 15 joints
Links:
- link j2n6s200_joule: geometry collision mesh filename=package://ada_description/meshes/collision_camera_joule.dae scale=0.001 0.001 0.00098; visual mesh filename=package://ada_description/meshes/camera_joule.dae scale=0.001 0.001 0.001

File: robots_urdf/ada_with_camera_forque.urdf (robot description, URDF)
Before this commit: robot j2n6s200, 19 links, 18 joints
Links:
- link j2n6s200_joule: geometry collision mesh filename=package://ada_description/meshes/collision_camera_joule.dae scale=0.001 0.001 0.00098; visual mesh filename=package://ada_description/meshes/camera_joule.dae scale=0.001 0.001 0.001
Joints:
- joint j2n6s200_joint_1: type continuous -> revolute
- joint j2n6s200_joint_4: type continuous -> revolute
- joint j2n6s200_joint_5: type continuous -> revolute
- joint j2n6s200_joint_6: type continuous -> revolute

Commit message: Update xacro files to match manual edits to ada_with_camera_forque

File: robots/camera.xacro (robot description, xacro)
@@ -16,7 +16,7 @@
       </visual>
       <collision>
-        <origin  rpy="0 0 0" xyz="-0.014 -0.062 -0.023"  />
+        <origin rpy="0 0 0" xyz="-0.008 -0.055 0.01"/>
         <geometry>
-          <mesh filename="package://ada_description/meshes/collision_camera_joule.dae" scale="0.001 0.001 0.00098"/>
+          <mesh filename="package://ada_description/meshes/collision_camera_joule.dae" scale="0.0008 0.00076 0.0006"/>
         </geometry>
       </collision>

File: robots/kinova_common.xacro (robot description, xacro)
@@ -33,10 +33,10 @@
       </link>
     </xacro:macro>
-  <xacro:macro name="kinova_armjoint" params="joint_name type parent child joint_axis_xyz joint_origin_xyz joint_origin_rpy joint_lower_limit joint_upper_limit fixed:=false">
+  <xacro:macro name="kinova_armjoint" params="joint_name type parent child joint_axis_xyz joint_origin_xyz joint_origin_rpy joint_lower_limit joint_upper_limit joint_velocity_limit=1.0 fixed:=false">
     <joint name="${joint_name}" type="${type}">
         <parent link="${parent}"/>
         <child link="${child}"/>
         <axis xyz="${joint_axis_xyz}"/>
-        <limit effort="2000" velocity="0.8" lower="${joint_lower_limit}" upper="${joint_upper_limit}"/>
+        <limit effort="2000" velocity="${joint_velocity_limit}" lower="${joint_lower_limit}" upper="${joint_upper_limit}"/>
         <origin xyz="${joint_origin_xyz}" rpy="${joint_origin_rpy}"/>
         <dynamics damping="0.0" friction="0.0"/>
