Commit message: make the joints continuous

File: robots_urdf/ada_with_camera_forque.urdf (robot description, URDF)
Before this commit: robot j2n6s200, 19 links, 18 joints
Joints:
- joint j2n6s200_joint_1: type revolute -> continuous
- joint j2n6s200_joint_4: type revolute -> continuous
- joint j2n6s200_joint_5: type revolute -> continuous
- joint j2n6s200_joint_6: type revolute -> continuous

Commit message: Make camera smaller

File: robots_urdf/ada_with_camera_forque.urdf (robot description, URDF)
Before this commit: robot j2n6s200, 19 links, 18 joints
Links:
- link j2n6s200_joule: geometry collision mesh filename=package://ada_description/meshes/collision_camera_joule.dae scale=0.0008 0.00076 0.0006; visual mesh filename=package://ada_description/meshes/camera_joule.dae scale=0.001 0.001 0.001

Commit message: Low velocity

File: robots_urdf/ada_with_camera_forque.urdf (robot description, URDF)
Before this commit: robot j2n6s200, 19 links, 18 joints
Joints:
- joint j2n6s200_joint_1: limit lower=-6.28318530718 upper=6.28318530718 effort=2000 velocity=0.8 -> lower=-6.28318530718 upper=6.28318530718 effort=2000 velocity=0.3
- joint j2n6s200_joint_2: limit lower=0.820304748437 upper=5.46288055874 effort=2000 velocity=0.8 -> lower=0.820304748437 upper=5.46288055874 effort=2000 velocity=0.3
- joint j2n6s200_joint_3: limit lower=0.331612557879 upper=5.9515727493 effort=2000 velocity=0.8 -> lower=0.331612557879 upper=5.9515727493 effort=2000 velocity=0.3
- joint j2n6s200_joint_4: limit lower=-6.28318530718 upper=6.28318530718 effort=2000 velocity=0.8 -> lower=-6.28318530718 upper=6.28318530718 effort=2000 velocity=0.3
- joint j2n6s200_joint_5: limit lower=-6.28318530718 upper=6.28318530718 effort=2000 velocity=0.8 -> lower=-6.28318530718 upper=6.28318530718 effort=2000 velocity=0.3
- joint j2n6s200_joint_6: limit lower=-6.28318530718 upper=6.28318530718 effort=2000 velocity=0.8 -> lower=-6.28318530718 upper=6.28318530718 effort=2000 velocity=0.3
- joint j2n6s200_joint_base: limit lower=0 upper=0 effort=2000 velocity=0.8 -> lower=0 upper=0 effort=2000 velocity=0.3

Commit message: use .dae for the visualization

File: robots_urdf/ada_with_camera_forque.urdf (robot description, URDF)
Before this commit: robot j2n6s200, 19 links, 18 joints
Links:
- link j2n6s200_joule: geometry collision mesh filename=package://ada_description/meshes/nano_coll.dae scale=0.001 0.001 0.001; visual mesh filename=package://ada_description/meshes/nano_all.dae scale=0.001 0.001 0.001

Commit message: minor fix on location of nano

File: robots_urdf/ada_with_camera_forque.urdf (robot description, URDF)
Before this commit: robot j2n6s200, 19 links, 18 joints
Joints:
- joint j2n6s200_joule: origin xyz=0.06 0.051 0.0140 rpy=1.57079632679 1.57079632679 0 -> xyz=0.06 0.016 0.0160 rpy=1.57079632679 1.57079632679 0

Commit message: Velocity limits too low

File: robots_urdf/ada_with_camera_forque.urdf (robot description, URDF)
Before this commit: robot j2n6s200, 19 links, 18 joints
Joints:
- joint j2n6s200_joint_1: limit lower=-6.28318530718 upper=6.28318530718 effort=2000 velocity=0.3 -> lower=-6.28318530718 upper=6.28318530718 effort=2000 velocity=1.0
- joint j2n6s200_joint_2: limit lower=0.820304748437 upper=5.46288055874 effort=2000 velocity=0.3 -> lower=0.820304748437 upper=5.46288055874 effort=2000 velocity=1.0
- joint j2n6s200_joint_3: limit lower=0.331612557879 upper=5.9515727493 effort=2000 velocity=0.3 -> lower=0.331612557879 upper=5.9515727493 effort=2000 velocity=1.0
- joint j2n6s200_joint_4: limit lower=-6.28318530718 upper=6.28318530718 effort=2000 velocity=0.3 -> lower=-6.28318530718 upper=6.28318530718 effort=2000 velocity=1.0
- joint j2n6s200_joint_5: limit lower=-6.28318530718 upper=6.28318530718 effort=2000 velocity=0.3 -> lower=-6.28318530718 upper=6.28318530718 effort=2000 velocity=1.0
- joint j2n6s200_joint_6: limit lower=-6.28318530718 upper=6.28318530718 effort=2000 velocity=0.3 -> lower=-6.28318530718 upper=6.28318530718 effort=2000 velocity=1.0
- joint j2n6s200_joint_base: limit lower=0 upper=0 effort=2000 velocity=0.3 -> lower=0 upper=0 effort=2000 velocity=1.0
