Commit message: added xacros

File: robots_urdf/ada.urdf (robot description, URDF)
Before this commit: robot j2n6s200, 13 links, 12 joints
Links:
- removed link j2n6s200_joule
- added link j2n6s200_hand_base
- added link world
- link j2n6s200_end_effector: geometry 
Joints:
- removed joint j2n6s200_joule
- added joint j2n6s200_joint_base: type fixed, parent world, child j2n6s200_link_base, origin xyz=0 0 0 rpy=0 0 0, axis 0 0 0, limit lower=0 upper=0 effort=2000 velocity=1
- added joint j2n6s200_joint_hand_base: type fixed, parent j2n6s200_link_6, child j2n6s200_hand_base, origin xyz=0 0 0 rpy=$0 0 0, axis 0 0 0, limit lower=0 upper=0 effort=2000 velocity=1
- joint j2n6s200_joint_1: limit lower=-3.141592 upper=3.141592 effort=2000 velocity=1 -> lower=-6.28318530718 upper=6.28318530718 effort=2000 velocity=1; type continuous -> revolute
- joint j2n6s200_joint_2: limit lower=-3.8451785 upper=0.7035858 effort=2000 velocity=1 -> lower=0.820304748437 upper=5.46288055874 effort=2000 velocity=1
- joint j2n6s200_joint_3: limit lower=-4.104090 upper=0.9515727493 effort=2000 velocity=1 -> lower=0.331612557879 upper=5.9515727493 effort=2000 velocity=1
- joint j2n6s200_joint_4: limit lower=-3.141592 upper=3.141592 effort=2000 velocity=1 -> lower=-6.28318530718 upper=6.28318530718 effort=2000 velocity=1; type continuous -> revolute
- joint j2n6s200_joint_5: limit lower=-3.141592 upper=3.141592 effort=2000 velocity=1 -> lower=-6.28318530718 upper=6.28318530718 effort=2000 velocity=1; type continuous -> revolute
- joint j2n6s200_joint_6: limit lower=-3.141592 upper=3.141592 effort=2000 velocity=1 -> lower=-6.28318530718 upper=6.28318530718 effort=2000 velocity=1; type continuous -> revolute
- joint j2n6s200_joint_finger_1: parent j2n6s200_link_6 -> j2n6s200_hand_base
- joint j2n6s200_joint_finger_2: parent j2n6s200_link_6 -> j2n6s200_hand_base
- joint j2n6s200_joint_finger_tip_1: limit lower=0 upper=2 effort=2000 velocity=1 -> lower=0 upper=2 effort=0 velocity=1; type revolute -> fixed
- joint j2n6s200_joint_finger_tip_2: limit lower=0 upper=2 effort=2000 velocity=1 -> lower=0 upper=2 effort=0 velocity=1; type revolute -> fixed

File: robots_urdf/ada_with_camera.urdf (robot description, URDF)
Before this commit: robot j2n6s200, 17 links, 16 joints
Links:
- removed link j2n6s200_forque
- removed link j2n6s200_forque_end_effector
Joints:
- removed joint j2n6s200_joint_forque
- removed joint j2n6s200_joint_forque_end_effector
- joint j2n6s200_joint_1: limit lower=-10 upper=10 effort=2000 velocity=1 -> lower=-6.28318530718 upper=6.28318530718 effort=2000 velocity=1
- joint j2n6s200_joint_2: limit lower=0.82030474843 upper=5.46288055874 effort=2000 velocity=1 -> lower=0.820304748437 upper=5.46288055874 effort=2000 velocity=1
- joint j2n6s200_joint_3: limit lower=0.33161255787 upper=5.9515727493 effort=2000 velocity=1 -> lower=0.331612557879 upper=5.9515727493 effort=2000 velocity=1
- joint j2n6s200_joint_4: limit lower=-10 upper=10 effort=2000 velocity=1 -> lower=-6.28318530718 upper=6.28318530718 effort=2000 velocity=1
- joint j2n6s200_joint_5: limit lower=-10 upper=10 effort=2000 velocity=1 -> lower=-6.28318530718 upper=6.28318530718 effort=2000 velocity=1
- joint j2n6s200_joint_6: limit lower=-10 upper=10 effort=2000 velocity=1 -> lower=-6.28318530718 upper=6.28318530718 effort=2000 velocity=1
- joint j2n6s200_joint_base: axis (none) -> 0 0 0; limit (none) -> lower=0 upper=0 effort=2000 velocity=1
- joint j2n6s200_joint_hand_base: limit (none) -> lower=0 upper=0 effort=2000 velocity=1; origin xyz=0 0 0 rpy=0 0 0 -> xyz=0 0 0 rpy=$0 0 0

File: robots_urdf/ada_with_camera_forque.urdf (robot description, URDF)
Before this commit: robot j2n6s200, 15 links, 14 joints
Links:
- added link j2n6s200_hand_base
- added link world
- link j2n6s200_end_effector: geometry 
- link j2n6s200_forque_end_effector: geometry 
Joints:
- added joint j2n6s200_joint_base: type fixed, parent world, child j2n6s200_link_base, origin xyz=0 0 0 rpy=0 0 0, axis 0 0 0, limit lower=0 upper=0 effort=2000 velocity=1
- added joint j2n6s200_joint_hand_base: type fixed, parent j2n6s200_link_6, child j2n6s200_hand_base, origin xyz=0 0 0 rpy=$0 0 0, axis 0 0 0, limit lower=0 upper=0 effort=2000 velocity=1
- joint j2n6s200_joint_1: limit lower=-3.141592 upper=3.141592 effort=2000 velocity=1 -> lower=-6.28318530718 upper=6.28318530718 effort=2000 velocity=1; type continuous -> revolute
- joint j2n6s200_joint_2: limit lower=-3.8451785 upper=0.7035858 effort=2000 velocity=1 -> lower=0.820304748437 upper=5.46288055874 effort=2000 velocity=1
- joint j2n6s200_joint_3: limit lower=-4.104090 upper=0.9515727493 effort=2000 velocity=1 -> lower=0.331612557879 upper=5.9515727493 effort=2000 velocity=1
- joint j2n6s200_joint_4: limit lower=-3.141592 upper=3.141592 effort=2000 velocity=1 -> lower=-6.28318530718 upper=6.28318530718 effort=2000 velocity=1; type continuous -> revolute
- joint j2n6s200_joint_5: limit lower=-3.141592 upper=3.141592 effort=2000 velocity=1 -> lower=-6.28318530718 upper=6.28318530718 effort=2000 velocity=1; type continuous -> revolute
- joint j2n6s200_joint_6: limit lower=-3.141592 upper=3.141592 effort=2000 velocity=1 -> lower=-6.28318530718 upper=6.28318530718 effort=2000 velocity=1; type continuous -> revolute
- joint j2n6s200_joint_finger_1: origin xyz=-0.0025 0.03095 -0.11482 rpy=-1.570796327 1.75 1.57079632679490 -> xyz=-0.0025 0.03095 -0.11482 rpy=-1.570796327 .649262481663582 1.57079632679490; parent j2n6s200_link_6 -> j2n6s200_hand_base
- joint j2n6s200_joint_finger_2: origin xyz=-0.0025 -0.03095 -0.11482 rpy=-1.570796327 1.75 -1.57079632679490 -> xyz=-0.0025 -0.03095 -0.11482 rpy=-1.570796327 .649262481663582 -1.57079632679490; parent j2n6s200_link_6 -> j2n6s200_hand_base
- joint j2n6s200_joint_finger_tip_1: limit lower=0 upper=2 effort=2000 velocity=1 -> lower=0 upper=2 effort=0 velocity=1; type revolute -> fixed
- joint j2n6s200_joint_finger_tip_2: limit lower=0 upper=2 effort=2000 velocity=1 -> lower=0 upper=2 effort=0 velocity=1; type revolute -> fixed

File: robots_urdf/ada_with_forque.urdf (robot description, URDF)
Before this commit: robot j2n6s200, 12 links, 11 joints
Links:
- added link j2n6s200_forque; collision mesh filename=package://ada_description/meshes/collision_forque_kinova.dae scale=0.001 0.001 0.001; visual mesh filename=package://ada_description/meshes/forque_kinova.dae scale=0.001 0.001 0.001
- added link j2n6s200_forque_end_effector
- added link j2n6s200_hand_base
- added link world
- link j2n6s200_end_effector: geometry 
Joints:
- added joint j2n6s200_joint_base: type fixed, parent world, child j2n6s200_link_base, origin xyz=0 0 0 rpy=0 0 0, axis 0 0 0, limit lower=0 upper=0 effort=2000 velocity=1
- added joint j2n6s200_joint_forque: type fixed, parent j2n6s200_end_effector, child j2n6s200_forque, origin xyz=-0.001 -0.000 0.09 rpy=3.14 0 0, axis 0 0 1, limit lower=0 upper=2 effort=2000 velocity=1
- added joint j2n6s200_joint_forque_end_effector: type fixed, parent j2n6s200_forque, child j2n6s200_forque_end_effector, origin xyz=0 0 -0.1 rpy=3.1415 0 0, axis 0 0 0, limit lower=0 upper=0 effort=2000 velocity=1
- added joint j2n6s200_joint_hand_base: type fixed, parent j2n6s200_link_6, child j2n6s200_hand_base, origin xyz=0 0 0 rpy=$0 0 0, axis 0 0 0, limit lower=0 upper=0 effort=2000 velocity=1
- joint j2n6s200_joint_1: limit lower=-3.141592 upper=3.141592 effort=2000 velocity=1 -> lower=-6.28318530718 upper=6.28318530718 effort=2000 velocity=1; type continuous -> revolute
- joint j2n6s200_joint_2: limit lower=-3.8451785 upper=0.7035858 effort=2000 velocity=1 -> lower=0.820304748437 upper=5.46288055874 effort=2000 velocity=1
- joint j2n6s200_joint_3: limit lower=-4.104090 upper=0.9515727493 effort=2000 velocity=1 -> lower=0.331612557879 upper=5.9515727493 effort=2000 velocity=1
- joint j2n6s200_joint_4: limit lower=-3.141592 upper=3.141592 effort=2000 velocity=1 -> lower=-6.28318530718 upper=6.28318530718 effort=2000 velocity=1; type continuous -> revolute
- joint j2n6s200_joint_5: limit lower=-3.141592 upper=3.141592 effort=2000 velocity=1 -> lower=-6.28318530718 upper=6.28318530718 effort=2000 velocity=1; type continuous -> revolute
- joint j2n6s200_joint_6: limit lower=-3.141592 upper=3.141592 effort=2000 velocity=1 -> lower=-6.28318530718 upper=6.28318530718 effort=2000 velocity=1; type continuous -> revolute
- joint j2n6s200_joint_finger_1: parent j2n6s200_link_6 -> j2n6s200_hand_base
- joint j2n6s200_joint_finger_2: parent j2n6s200_link_6 -> j2n6s200_hand_base
- joint j2n6s200_joint_finger_tip_1: limit lower=0 upper=2 effort=2000 velocity=1 -> lower=0 upper=2 effort=0 velocity=1; type revolute -> fixed
- joint j2n6s200_joint_finger_tip_2: limit lower=0 upper=2 effort=2000 velocity=1 -> lower=0 upper=2 effort=0 velocity=1; type revolute -> fixed

Commit message: Change joint 1, 4, 5, 6 from revolute to continuous

File: robots_urdf/ada.urdf (robot description, URDF)
Before this commit: robot j2n6s200, 15 links, 14 joints
Joints:
- joint j2n6s200_joint_1: type revolute -> continuous
- joint j2n6s200_joint_4: type revolute -> continuous
- joint j2n6s200_joint_5: type revolute -> continuous
- joint j2n6s200_joint_6: type revolute -> continuous

File: robots_urdf/ada_with_camera.urdf (robot description, URDF)
Before this commit: robot j2n6s200, 16 links, 15 joints
Joints:
- joint j2n6s200_joint_1: type revolute -> continuous
- joint j2n6s200_joint_4: type revolute -> continuous
- joint j2n6s200_joint_5: type revolute -> continuous
- joint j2n6s200_joint_6: type revolute -> continuous

File: robots_urdf/ada_with_camera_forque.urdf (robot description, URDF)
Before this commit: robot j2n6s200, 19 links, 18 joints
Joints:
- joint j2n6s200_joint_1: type revolute -> continuous
- joint j2n6s200_joint_4: type revolute -> continuous
- joint j2n6s200_joint_5: type revolute -> continuous
- joint j2n6s200_joint_6: type revolute -> continuous

File: robots_urdf/ada_with_forque.urdf (robot description, URDF)
Before this commit: robot j2n6s200, 18 links, 17 joints
Joints:
- joint j2n6s200_joint_1: type revolute -> continuous
- joint j2n6s200_joint_4: type revolute -> continuous
- joint j2n6s200_joint_5: type revolute -> continuous
- joint j2n6s200_joint_6: type revolute -> continuous

Commit message: Regenerate urdfs with xacro

File: robots_urdf/ada.urdf (robot description, URDF)
Before this commit: robot j2n6s200, 15 links, 14 joints
Links:
- link j2n6s200_link_6: geometry collision mesh filename=package://ada_description/meshes/collision_hand_2finger.dae; visual mesh filename=package://ada_description/meshes/hand_2finger.dae
Joints:
- joint j2n6s200_joint_1: limit lower=-6.28318530718 upper=6.28318530718 effort=2000 velocity=0.8 -> lower=-6.283185307179586 upper=6.283185307179586 effort=2000 velocity=1.0; origin xyz=0 0 0.15675 rpy=0 3.14159265359 0 -> xyz=0 0 0.15675 rpy=0 3.141592653589793 0
- joint j2n6s200_joint_2: limit lower=0.820304748437 upper=5.46288055874 effort=2000 velocity=0.8 -> lower=0.8203047484373349 upper=5.462880558742252 effort=2000 velocity=1.0; origin xyz=0 0.0016 -0.11875 rpy=-1.57079632679 0 3.14159265359 -> xyz=0 0.0016 -0.11875 rpy=-1.5707963267948966 0 3.141592653589793
- joint j2n6s200_joint_3: limit lower=0.331612557879 upper=5.9515727493 effort=2000 velocity=0.8 -> lower=0.33161255787892263 upper=5.951572749300664 effort=2000 velocity=1.0; origin xyz=0 -0.410 0 rpy=0 3.14159265359 0 -> xyz=0 -0.410 0 rpy=0 3.141592653589793 0
- joint j2n6s200_joint_4: limit lower=-6.28318530718 upper=6.28318530718 effort=2000 velocity=0.8 -> lower=-6.283185307179586 upper=6.283185307179586 effort=2000 velocity=1.0; origin xyz=0 0.2073 -0.0114 rpy=-1.57079632679 0 3.14159265359 -> xyz=0 0.2073 -0.0114 rpy=-1.5707963267948966 0 3.141592653589793
- joint j2n6s200_joint_5: limit lower=-6.28318530718 upper=6.28318530718 effort=2000 velocity=0.8 -> lower=-6.283185307179586 upper=6.283185307179586 effort=2000 velocity=1.0; origin xyz=0 -0.03703 -0.06414 rpy=1.0471975512 0 3.14159265359 -> xyz=0 -0.03703 -0.06414 rpy=1.0471975511965976 0 3.141592653589793
- joint j2n6s200_joint_6: limit lower=-6.28318530718 upper=6.28318530718 effort=2000 velocity=0.8 -> lower=-6.283185307179586 upper=6.283185307179586 effort=2000 velocity=1.0; origin xyz=0 -0.03703 -0.06414 rpy=1.0471975512 0 3.14159265359 -> xyz=0 -0.03703 -0.06414 rpy=1.0471975511965976 0 3.141592653589793
- joint j2n6s200_joint_base: limit lower=0 upper=0 effort=2000 velocity=0.8 -> lower=0 upper=0 effort=2000 velocity=1.0
- joint j2n6s200_joint_end_effector: origin xyz=0 0 -0.1600 rpy=3.14159265359 0 0 -> xyz=0 0 -0.1600 rpy=3.141592653589793 0 0

File: robots_urdf/ada_with_camera.urdf (robot description, URDF)
Before this commit: robot j2n6s200, 16 links, 15 joints
Links:
- link j2n6s200_joule: geometry collision mesh filename=package://ada_description/meshes/collision_camera_joule.dae scale=0.0008 0.00076 0.0006; visual mesh filename=package://ada_description/meshes/camera_joule.dae scale=0.001 0.001 0.001
Joints:
- joint j2n6s200_joint_1: limit lower=-6.28318530718 upper=6.28318530718 effort=2000 velocity=0.8 -> lower=-6.283185307179586 upper=6.283185307179586 effort=2000 velocity=1.0; origin xyz=0 0 0.15675 rpy=0 3.14159265359 0 -> xyz=0 0 0.15675 rpy=0 3.141592653589793 0
- joint j2n6s200_joint_2: limit lower=0.820304748437 upper=5.46288055874 effort=2000 velocity=0.8 -> lower=0.8203047484373349 upper=5.462880558742252 effort=2000 velocity=1.0; origin xyz=0 0.0016 -0.11875 rpy=-1.57079632679 0 3.14159265359 -> xyz=0 0.0016 -0.11875 rpy=-1.5707963267948966 0 3.141592653589793
- joint j2n6s200_joint_3: limit lower=0.331612557879 upper=5.9515727493 effort=2000 velocity=0.8 -> lower=0.33161255787892263 upper=5.951572749300664 effort=2000 velocity=1.0; origin xyz=0 -0.410 0 rpy=0 3.14159265359 0 -> xyz=0 -0.410 0 rpy=0 3.141592653589793 0
- joint j2n6s200_joint_4: limit lower=-6.28318530718 upper=6.28318530718 effort=2000 velocity=0.8 -> lower=-6.283185307179586 upper=6.283185307179586 effort=2000 velocity=1.0; origin xyz=0 0.2073 -0.0114 rpy=-1.57079632679 0 3.14159265359 -> xyz=0 0.2073 -0.0114 rpy=-1.5707963267948966 0 3.141592653589793
- joint j2n6s200_joint_5: limit lower=-6.28318530718 upper=6.28318530718 effort=2000 velocity=0.8 -> lower=-6.283185307179586 upper=6.283185307179586 effort=2000 velocity=1.0; origin xyz=0 -0.03703 -0.06414 rpy=1.0471975512 0 3.14159265359 -> xyz=0 -0.03703 -0.06414 rpy=1.0471975511965976 0 3.141592653589793
- joint j2n6s200_joint_6: limit lower=-6.28318530718 upper=6.28318530718 effort=2000 velocity=0.8 -> lower=-6.283185307179586 upper=6.283185307179586 effort=2000 velocity=1.0; origin xyz=0 -0.03703 -0.06414 rpy=1.0471975512 0 3.14159265359 -> xyz=0 -0.03703 -0.06414 rpy=1.0471975511965976 0 3.141592653589793
- joint j2n6s200_joint_base: limit lower=0 upper=0 effort=2000 velocity=0.8 -> lower=0 upper=0 effort=2000 velocity=1.0
- joint j2n6s200_joint_end_effector: origin xyz=0 0 -0.1600 rpy=3.14159265359 0 0 -> xyz=0 0 -0.1600 rpy=3.141592653589793 0 0

File: robots_urdf/ada_with_camera_forque.urdf (robot description, URDF)
Before this commit: robot j2n6s200, 19 links, 18 joints
Joints:
- joint j2n6s200_joint_1: limit lower=-6.28318530718 upper=6.28318530718 effort=2000 velocity=1.0 -> lower=-6.283185307179586 upper=6.283185307179586 effort=2000 velocity=1.0; origin xyz=0 0 0.15675 rpy=0 3.14159265359 0 -> xyz=0 0 0.15675 rpy=0 3.141592653589793 0
- joint j2n6s200_joint_2: limit lower=0.820304748437 upper=5.46288055874 effort=2000 velocity=1.0 -> lower=0.8203047484373349 upper=5.462880558742252 effort=2000 velocity=1.0; origin xyz=0 0.0016 -0.11875 rpy=-1.57079632679 0 3.14159265359 -> xyz=0 0.0016 -0.11875 rpy=-1.5707963267948966 0 3.141592653589793
- joint j2n6s200_joint_3: limit lower=0.331612557879 upper=5.9515727493 effort=2000 velocity=1.0 -> lower=0.33161255787892263 upper=5.951572749300664 effort=2000 velocity=1.0; origin xyz=0 -0.410 0 rpy=0 3.14159265359 0 -> xyz=0 -0.410 0 rpy=0 3.141592653589793 0
- joint j2n6s200_joint_4: limit lower=-6.28318530718 upper=6.28318530718 effort=2000 velocity=1.0 -> lower=-6.283185307179586 upper=6.283185307179586 effort=2000 velocity=1.0; origin xyz=0 0.2073 -0.0114 rpy=-1.57079632679 0 3.14159265359 -> xyz=0 0.2073 -0.0114 rpy=-1.5707963267948966 0 3.141592653589793
- joint j2n6s200_joint_5: limit lower=-6.28318530718 upper=6.28318530718 effort=2000 velocity=1.0 -> lower=-6.283185307179586 upper=6.283185307179586 effort=2000 velocity=1.0; origin xyz=0 -0.03703 -0.06414 rpy=1.0471975512 0 3.14159265359 -> xyz=0 -0.03703 -0.06414 rpy=1.0471975511965976 0 3.141592653589793
- joint j2n6s200_joint_6: limit lower=-6.28318530718 upper=6.28318530718 effort=2000 velocity=1.0 -> lower=-6.283185307179586 upper=6.283185307179586 effort=2000 velocity=1.0; origin xyz=0 -0.03703 -0.06414 rpy=1.0471975512 0 3.14159265359 -> xyz=0 -0.03703 -0.06414 rpy=1.0471975511965976 0 3.141592653589793
- joint j2n6s200_joint_end_effector: origin xyz=0 0 -0.1600 rpy=3.14159265359 0 0 -> xyz=0 0 -0.1600 rpy=3.141592653589793 0 0

File: robots_urdf/ada_with_forque.urdf (robot description, URDF)
Before this commit: robot j2n6s200, 18 links, 17 joints
Links:
- link j2n6s200_link_6: geometry collision mesh filename=package://ada_description/meshes/collision_hand_2finger.dae; visual mesh filename=package://ada_description/meshes/hand_2finger.dae
Joints:
- joint j2n6s200_joint_1: limit lower=-6.28318530718 upper=6.28318530718 effort=2000 velocity=0.8 -> lower=-6.283185307179586 upper=6.283185307179586 effort=2000 velocity=1.0; origin xyz=0 0 0.15675 rpy=0 3.14159265359 0 -> xyz=0 0 0.15675 rpy=0 3.141592653589793 0
- joint j2n6s200_joint_2: limit lower=0.820304748437 upper=5.46288055874 effort=2000 velocity=0.8 -> lower=0.8203047484373349 upper=5.462880558742252 effort=2000 velocity=1.0; origin xyz=0 0.0016 -0.11875 rpy=-1.57079632679 0 3.14159265359 -> xyz=0 0.0016 -0.11875 rpy=-1.5707963267948966 0 3.141592653589793
- joint j2n6s200_joint_3: limit lower=0.331612557879 upper=5.9515727493 effort=2000 velocity=0.8 -> lower=0.33161255787892263 upper=5.951572749300664 effort=2000 velocity=1.0; origin xyz=0 -0.410 0 rpy=0 3.14159265359 0 -> xyz=0 -0.410 0 rpy=0 3.141592653589793 0
- joint j2n6s200_joint_4: limit lower=-6.28318530718 upper=6.28318530718 effort=2000 velocity=0.8 -> lower=-6.283185307179586 upper=6.283185307179586 effort=2000 velocity=1.0; origin xyz=0 0.2073 -0.0114 rpy=-1.57079632679 0 3.14159265359 -> xyz=0 0.2073 -0.0114 rpy=-1.5707963267948966 0 3.141592653589793
- joint j2n6s200_joint_5: limit lower=-6.28318530718 upper=6.28318530718 effort=2000 velocity=0.8 -> lower=-6.283185307179586 upper=6.283185307179586 effort=2000 velocity=1.0; origin xyz=0 -0.03703 -0.06414 rpy=1.0471975512 0 3.14159265359 -> xyz=0 -0.03703 -0.06414 rpy=1.0471975511965976 0 3.141592653589793
- joint j2n6s200_joint_6: limit lower=-6.28318530718 upper=6.28318530718 effort=2000 velocity=0.8 -> lower=-6.283185307179586 upper=6.283185307179586 effort=2000 velocity=1.0; origin xyz=0 -0.03703 -0.06414 rpy=1.0471975512 0 3.14159265359 -> xyz=0 -0.03703 -0.06414 rpy=1.0471975511965976 0 3.141592653589793
- joint j2n6s200_joint_base: limit lower=0 upper=0 effort=2000 velocity=0.8 -> lower=0 upper=0 effort=2000 velocity=1.0
- joint j2n6s200_joint_end_effector: origin xyz=0 0 -0.1600 rpy=3.14159265359 0 0 -> xyz=0 0 -0.1600 rpy=3.141592653589793 0 0
