Commit message: replace joule with nano

File: robots_urdf/ada_with_camera.urdf (robot description, URDF)
Before this commit: robot j2n6s200, 16 links, 15 joints
Links:
- link j2n6s200_joule: geometry collision mesh filename=package://ada_description/meshes/nano_coll.dae scale=0.001 0.001 0.001; visual mesh filename=package://ada_description/meshes/nano_all.STL scale=0.001 0.001 0.001

File: robots_urdf/ada_with_camera_forque.urdf (robot description, URDF)
Before this commit: robot j2n6s200, 19 links, 18 joints
Links:
- link j2n6s200_joule: geometry collision mesh filename=package://ada_description/meshes/nano_coll.dae scale=0.001 0.001 0.001; visual mesh filename=package://ada_description/meshes/nano_all.STL scale=0.001 0.001 0.001

Commit message: Save edits for sniyaz thesis that show coll geom in rviz.

File: robots_urdf/ada_with_camera.urdf (robot description, URDF)
Before this commit: robot j2n6s200, 16 links, 15 joints
Links:
- link j2n6s200_joule: geometry collision mesh filename=package://ada_description/meshes/collision_camera_joule.dae scale=0.001 0.001 0.00098; visual mesh filename=package://ada_description/meshes/collision_camera_joule.dae scale=0.001 0.001 0.00098
- link j2n6s200_link_3: geometry collision mesh filename=package://ada_description/meshes/collision_forearm.dae; visual mesh filename=package://ada_description/meshes/collision_forearm.dae
- link j2n6s200_link_5: geometry collision mesh filename=package://ada_description/meshes/collision_wrist.dae; visual mesh filename=package://ada_description/meshes/collision_wrist.dae
- link j2n6s200_link_6: geometry collision mesh filename=package://ada_description/meshes/collision_hand_2finger.dae; visual mesh filename=package://ada_description/meshes/collision_hand_2finger.dae
