Commit message: Moved JACO and MICO meshes/robots to subfolders

File: jaco/robots/camera.xacro (robot description, xacro)
@@ -8,6 +8,6 @@
         <origin  rpy="0 0 0" xyz="-0.014 -0.062 -0.023"  />
         <geometry>
-          <mesh filename="package://ada_description/meshes/camera_joule.dae" scale="0.001 0.001 0.001"/>
-          <!-- <mesh filename="package://ada_description/meshes/collision_camera_joule.dae" scale="0.001 0.001 0.00098"/> -->
+          <mesh filename="package://ada_description/jaco/meshes/camera_joule.dae" scale="0.001 0.001 0.001"/>
+          <!-- <mesh filename="package://ada_description/jaco/meshes/collision_camera_joule.dae" scale="0.001 0.001 0.00098"/> -->
         </geometry>
       <material name="carbon_fiber">
@@ -18,5 +18,5 @@
         <origin  rpy="0 0 0" xyz="-0.014 -0.062 -0.023"  />
         <geometry>
-          <mesh filename="package://ada_description/meshes/collision_camera_joule.dae" scale="0.001 0.001 0.00098"/>
+          <mesh filename="package://ada_description/jaco/meshes/collision_camera_joule.dae" scale="0.001 0.001 0.00098"/>
         </geometry>
       </collision>

File: jaco/robots/forque.xacro (robot description, xacro)
@@ -7,5 +7,5 @@
       <visual>
         <geometry>
-            <mesh filename="package://ada_description/meshes/forque_kinova.dae" scale="0.001 0.001 0.001"/>
+            <mesh filename="package://ada_description/jaco/meshes/forque_kinova.dae" scale="0.001 0.001 0.001"/>
         </geometry>
         <material name="carbon_fiber">
@@ -15,5 +15,5 @@
       <collision>
         <geometry>
-          <mesh filename="package://ada_description/meshes/collision_forque_kinova.dae" scale="0.001 0.001 0.001"/>
+          <mesh filename="package://ada_description/jaco/meshes/collision_forque_kinova.dae" scale="0.001 0.001 0.001"/>
         </geometry>
       </collision>

File: jaco/robots/j2n6s200.xacro (robot description, xacro)
@@ -3,82 +3,82 @@
 <root xmlns:xi="http://www.w3.org/2001/XInclude"
     xmlns:xacro="http://ros.org/wiki/xacro">
-    <xacro:include filename="$(find ada_description)/robots/kinova_common.xacro" />
-    <xacro:include filename="$(find ada_description)/robots/kinova_finger_set.xacro" />
-    <property name="link_base_mesh" value="base" />
-    <property name="link_1_mesh" value="shoulder" />
-    <property name="link_2_mesh" value="arm" />
-    <property name="link_3_mesh" value="forearm" />
-    <property name="link_4_mesh" value="wrist" />
-    <property name="link_5_mesh" value="wrist" />
-    <property name="link_6_mesh" value="hand_2finger" />
-    <property name="link_base_mesh_no" value="0" />
-    <property name="link_1_mesh_no" value="1" />
-    <property name="link_2_mesh_no" value="2" />
-    <property name="link_3_mesh_no" value="3" />
-    <property name="link_4_mesh_no" value="4" />
-    <property name="link_5_mesh_no" value="4" />
-    <property name="link_6_mesh_no" value="56" />
-    <property name="joint_base" value="joint_base" />
-    <property name="joint_base_type" value="fixed" />
-    <property name="joint_base_axis_xyz" value="0 0 0" />
-    <property name="joint_base_origin_xyz" value="0 0 0" />
-    <property name="joint_base_origin_rpy" value="0 0 0" />
-    <property name="joint_1" value="joint_1" />
-    <property name="joint_1_type" value="continuous" />
-    <property name="joint_1_axis_xyz" value="0 0 1" />
-    <property name="joint_1_origin_xyz" value="0 0 0.15675" />
-    <property name="joint_1_origin_rpy" value="0 ${J_PI} 0" />
-    <property name="joint_1_lower_limit" value="${-2*J_PI}" />
-    <property name="joint_1_upper_limit" value="${2*J_PI}" />
-    <property name="joint_2" value="joint_2" />
-    <property name="joint_2_type" value="revolute" />
-    <property name="joint_2_axis_xyz" value="0 0 1" />
-    <property name="joint_2_origin_xyz" value="0 0.0016 -0.11875" />
-    <property name="joint_2_origin_rpy" value="-${J_PI/2} 0 ${J_PI}" />
-    <property name="joint_2_lower_limit" value="${47/180*J_PI}" />
-    <property name="joint_2_upper_limit" value="${313/180*J_PI}" />
-    <property name="joint_3" value="joint_3" />
-    <property name="joint_3_type" value="revolute" />
-    <property name="joint_3_axis_xyz" value="0 0 1" />
-    <property name="joint_3_origin_xyz" value="0 -0.410 0" />
-    <property name="joint_3_origin_rpy" value="0 ${J_PI} 0" />
-    <property name="joint_3_lower_limit" value="${19/180*J_PI}" />
-    <property name="joint_3_upper_limit" value="${341/180*J_PI}" />
-    <property name="joint_4" value="joint_4" />
-    <property name="joint_4_type" value="continuous" />
-    <property name="joint_4_axis_xyz" value="0 0 1" />
-    <property name="joint_4_origin_xyz" value="0 0.2073 -0.0114" />
-    <property name="joint_4_origin_rpy" value="-${J_PI/2} 0 ${J_PI}" />
-    <property name="joint_4_lower_limit" value="${-2*J_PI}" />
-    <property name="joint_4_upper_limit" value="${2*J_PI}" />
-    <property name="joint_5" value="joint_5" />
-    <property name="joint_5_type" value="continuous" />
-    <property name="joint_5_axis_xyz" value="0 0 1" />
-    <property name="joint_5_origin_xyz" value="0 -0.03703 -0.06414" />
-    <property name="joint_5_origin_rpy" value="${J_PI/3} 0 ${J_PI}" />
-    <property name="joint_5_lower_limit" value="${-2*J_PI}" />
-    <property name="joint_5_upper_limit" value="${2*J_PI}" />
-    <property name="joint_6" value="joint_6" />
-    <property name="joint_6_type" value="continuous" />
-    <property name="joint_6_axis_xyz" value="0 0 1" />
-    <property name="joint_6_origin_xyz" value="0 -0.03703 -0.06414" />
-    <property name="joint_6_origin_rpy" value="${J_PI/3} 0 ${J_PI}" />
-    <property name="joint_6_lower_limit" value="${-2*J_PI}" />
-    <property name="joint_6_upper_limit" value="${2*J_PI}" />
-    <property name="joint_end_effector" value="end_effector_offset" />
-    <property name="joint_end_effector_type" value="fixed" />
-    <property name="joint_end_effector_axis_xyz" value="0 0 0" />
-    <property name="joint_end_effector_origin_xyz" value="0 0 -0.1600" />
-    <property name="joint_end_effector_origin_rpy" value="${J_PI} 0 0" />
-    <property name="joint_hand_tip" value="end_effector_offset" />
-    <property name="joint_hand_tip_type" value="fixed" />
-    <property name="joint_hand_tip_axis_xyz" value="0 0 0" />
-    <property name="joint_hand_tip_origin_xyz" value="0 0 0.0370" />
-    <property name="joint_hand_tip_origin_rpy" value="0 0 0" />
-    <property name="joint_hand_base" value="hand_base" />
-    <property name="joint_hand_base_type" value="fixed" />
-    <property name="joint_hand_base_axis_xyz" value="0 0 0" />
-    <property name="joint_hand_base_origin_xyz" value="0 0 0" />
-    <property name="joint_hand_base_origin_rpy" value="0 0 0" />
+    <xacro:include filename="$(find ada_description)/jaco/robots/kinova_common.xacro" />
+    <xacro:include filename="$(find ada_description)/jaco/robots/kinova_finger_set.xacro" />
+    <xacro:property name="link_base_mesh" value="base" />
+    <xacro:property name="link_1_mesh" value="shoulder" />
+    <xacro:property name="link_2_mesh" value="arm" />
+    <xacro:property name="link_3_mesh" value="forearm" />
+    <xacro:property name="link_4_mesh" value="wrist" />
+    <xacro:property name="link_5_mesh" value="wrist" />
+    <xacro:property name="link_6_mesh" value="hand_2finger" />
+    <xacro:property name="link_base_mesh_no" value="0" />
+    <xacro:property name="link_1_mesh_no" value="1" />
+    <xacro:property name="link_2_mesh_no" value="2" />
+    <xacro:property name="link_3_mesh_no" value="3" />
+    <xacro:property name="link_4_mesh_no" value="4" />
+    <xacro:property name="link_5_mesh_no" value="4" />
+    <xacro:property name="link_6_mesh_no" value="56" />
+    <xacro:property name="joint_base" value="joint_base" />
+    <xacro:property name="joint_base_type" value="fixed" />
+    <xacro:property name="joint_base_axis_xyz" value="0 0 0" />
+    <xacro:property name="joint_base_origin_xyz" value="0 0 0" />
+    <xacro:property name="joint_base_origin_rpy" value="0 0 0" />
+    <xacro:property name="joint_1" value="joint_1" />
+    <xacro:property name="joint_1_type" value="continuous" />
+    <xacro:property name="joint_1_axis_xyz" value="0 0 1" />
+    <xacro:property name="joint_1_origin_xyz" value="0 0 0.15675" />
+    <xacro:property name="joint_1_origin_rpy" value="0 ${J_PI} 0" />
+    <xacro:property name="joint_1_lower_limit" value="${-2*J_PI}" />
+    <xacro:property name="joint_1_upper_limit" value="${2*J_PI}" />
+    <xacro:property name="joint_2" value="joint_2" />
+    <xacro:property name="joint_2_type" value="revolute" />
+    <xacro:property name="joint_2_axis_xyz" value="0 0 1" />
+    <xacro:property name="joint_2_origin_xyz" value="0 0.0016 -0.11875" />
+    <xacro:property name="joint_2_origin_rpy" value="-${J_PI/2} 0 ${J_PI}" />
+    <xacro:property name="joint_2_lower_limit" value="${47/180*J_PI}" />
+    <xacro:property name="joint_2_upper_limit" value="${313/180*J_PI}" />
+    <xacro:property name="joint_3" value="joint_3" />
+    <xacro:property name="joint_3_type" value="revolute" />
+    <xacro:property name="joint_3_axis_xyz" value="0 0 1" />
+    <xacro:property name="joint_3_origin_xyz" value="0 -0.410 0" />
+    <xacro:property name="joint_3_origin_rpy" value="0 ${J_PI} 0" />
+    <xacro:property name="joint_3_lower_limit" value="${19/180*J_PI}" />
+    <xacro:property name="joint_3_upper_limit" value="${341/180*J_PI}" />
+    <xacro:property name="joint_4" value="joint_4" />
+    <xacro:property name="joint_4_type" value="continuous" />
+    <xacro:property name="joint_4_axis_xyz" value="0 0 1" />
+    <xacro:property name="joint_4_origin_xyz" value="0 0.2073 -0.0114" />
+    <xacro:property name="joint_4_origin_rpy" value="-${J_PI/2} 0 ${J_PI}" />
+    <xacro:property name="joint_4_lower_limit" value="${-2*J_PI}" />
+    <xacro:property name="joint_4_upper_limit" value="${2*J_PI}" />
+    <xacro:property name="joint_5" value="joint_5" />
+    <xacro:property name="joint_5_type" value="continuous" />
+    <xacro:property name="joint_5_axis_xyz" value="0 0 1" />
+    <xacro:property name="joint_5_origin_xyz" value="0 -0.03703 -0.06414" />
+    <xacro:property name="joint_5_origin_rpy" value="${J_PI/3} 0 ${J_PI}" />
+    <xacro:property name="joint_5_lower_limit" value="${-2*J_PI}" />
+    <xacro:property name="joint_5_upper_limit" value="${2*J_PI}" />
+    <xacro:property name="joint_6" value="joint_6" />
+    <xacro:property name="joint_6_type" value="continuous" />
+    <xacro:property name="joint_6_axis_xyz" value="0 0 1" />
+    <xacro:property name="joint_6_origin_xyz" value="0 -0.03703 -0.06414" />
+    <xacro:property name="joint_6_origin_rpy" value="${J_PI/3} 0 ${J_PI}" />
+    <xacro:property name="joint_6_lower_limit" value="${-2*J_PI}" />
+    <xacro:property name="joint_6_upper_limit" value="${2*J_PI}" />
+    <xacro:property name="joint_end_effector" value="end_effector_offset" />
+    <xacro:property name="joint_end_effector_type" value="fixed" />
+    <xacro:property name="joint_end_effector_axis_xyz" value="0 0 0" />
+    <xacro:property name="joint_end_effector_origin_xyz" value="0 0 -0.1600" />
+    <xacro:property name="joint_end_effector_origin_rpy" value="${J_PI} 0 0" />
+    <xacro:property name="joint_hand_tip" value="end_effector_offset" />
+    <xacro:property name="joint_hand_tip_type" value="fixed" />
+    <xacro:property name="joint_hand_tip_axis_xyz" value="0 0 0" />
+    <xacro:property name="joint_hand_tip_origin_xyz" value="0 0 0.0370" />
+    <xacro:property name="joint_hand_tip_origin_rpy" value="0 0 0" />
+    <xacro:property name="joint_hand_base" value="hand_base" />
+    <xacro:property name="joint_hand_base_type" value="fixed" />
+    <xacro:property name="joint_hand_base_axis_xyz" value="0 0 0" />
+    <xacro:property name="joint_hand_base_origin_xyz" value="0 0 0" />
+    <xacro:property name="joint_hand_base_origin_rpy" value="0 0 0" />
     <xacro:macro name="j2n6s200" params="base_parent hide_final_ring:=false prefix:=j2n6s200">
         <!--xacro:gazebo_config robot_namespace="${prefix}"/-->

File: jaco/robots/j2n6s200_standalone.xacro (robot description, xacro)
@@ -3,12 +3,12 @@
 <robot xmlns:xi="http://www.w3.org/2001/XInclude"
 	xmlns:xacro="http://ros.org/wiki/xacro" name="j2n6s200">
-  <xacro:include filename="$(find ada_description)/robots/j2n6s200.xacro"/>
-  <xacro:include filename="$(find ada_description)/robots/camera.xacro"/>
-  <xacro:include filename="$(find ada_description)/robots/forque.xacro"/>
+  <xacro:include filename="$(find ada_description)/jaco/robots/j2n6s200.xacro"/>
+  <xacro:include filename="$(find ada_description)/jaco/robots/camera.xacro"/>
+  <xacro:include filename="$(find ada_description)/jaco/robots/forque.xacro"/>
   <xacro:arg name="with_camera" default="false" />
   <xacro:arg name="with_forque" default="false" />
   <link name="world"/>
-  <property name="robot_root" value="world" />
-  <property name="prefix" value="j2n6s200" />
+  <xacro:property name="robot_root" value="world" />
+  <xacro:property name="prefix" value="j2n6s200" />
   <xacro:j2n6s200  base_parent="${robot_root}" hide_final_ring="$(arg with_camera)"/>
   <!--xacro:j2n6s200  base_parent="${robot_root}" /-->

File: jaco/robots/kinova_common.xacro (robot description, xacro)
@@ -2,6 +2,6 @@
 <root xmlns:xi="http://www.w3.org/2001/XInclude"
 	xmlns:xacro="http://ros.org/wiki/xacro">
-<xacro:include filename="$(find ada_description)/robots/kinova_inertial.xacro" />
-    <property name="J_PI" value="3.1415926535897931" />
+<xacro:include filename="$(find ada_description)/jaco/robots/kinova_inertial.xacro" />
+    <xacro:property name="J_PI" value="3.1415926535897931" scope="global" />
     <xacro:macro name="kinova_armlink" params="link_name link_mesh ring_mesh:=ring_big use_ring_mesh:=false mesh_no">
         <link name="${link_name}">
@@ -9,5 +9,5 @@
                 <geometry>
                     <mesh
-                        filename="package://ada_description/meshes/${link_mesh}.dae"/>
+                        filename="package://ada_description/jaco/meshes/${link_mesh}.dae"/>
                 </geometry>
                 <material name="carbon_fiber">
@@ -20,5 +20,5 @@
                 <geometry>
                     <mesh
-                        filename="package://ada_description/meshes/${ring_mesh}.dae"/>
+                        filename="package://ada_description/jaco/meshes/${ring_mesh}.dae"/>
                 </geometry>
              </visual>
@@ -27,5 +27,5 @@
                 <geometry>
                     <mesh
-                        filename="package://ada_description/meshes/collision_${link_mesh}.dae"/>
+                        filename="package://ada_description/jaco/meshes/collision_${link_mesh}.dae"/>
                 </geometry>
             </collision>

File: jaco/robots/kinova_finger_set.xacro (robot description, xacro)
@@ -14,5 +14,5 @@
     xmlns:physics="http://playerstage.sourceforge.net/gazebo/xmlschema/#physics"
     xmlns:xacro="http://ros.org/wiki/xacro">
-    <xacro:include filename="$(find ada_description)/robots/kinova_common.xacro" />
+    <xacro:include filename="$(find ada_description)/jaco/robots/kinova_common.xacro" />
     <xacro:macro name="kinova_2fingers" params="link_hand prefix">
         <!-- finger1 Rot := Ry((1/2)*Pi) . Rx(Pi) . Rz(-52.8*((1/180)*Pi)) -->

File: jaco/urdf/ada.urdf (robot description, URDF)
Before this commit: robot j2n6s200, 19 links, 18 joints
Links:
- removed link j2n6s200_forque
- removed link j2n6s200_forque_end_effector
- removed link j2n6s200_forque_tip
- removed link j2n6s200_joule
- link j2n6s200_link_1: geometry collision mesh filename=package://ada_description/jaco/meshes/collision_shoulder.dae; visual mesh filename=package://ada_description/jaco/meshes/ring_big.dae
- link j2n6s200_link_2: geometry collision mesh filename=package://ada_description/jaco/meshes/collision_arm.dae; visual mesh filename=package://ada_description/jaco/meshes/arm.dae
- link j2n6s200_link_3: geometry collision mesh filename=package://ada_description/jaco/meshes/collision_forearm.dae; visual mesh filename=package://ada_description/jaco/meshes/forearm.dae
- link j2n6s200_link_4: geometry collision mesh filename=package://ada_description/jaco/meshes/collision_wrist.dae; visual mesh filename=package://ada_description/jaco/meshes/ring_small.dae
- link j2n6s200_link_5: geometry collision mesh filename=package://ada_description/jaco/meshes/collision_wrist.dae; visual mesh filename=package://ada_description/jaco/meshes/ring_small.dae
- link j2n6s200_link_6: geometry collision mesh filename=package://ada_description/jaco/meshes/collision_hand_2finge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; visual mesh filename=package://ada_description/jaco/meshes/hand_2finger.dae
- link j2n6s200_link_base: geometry collision mesh filename=package://ada_description/jaco/meshes/collision_base.dae; visual mesh filename=package://ada_description/jaco/meshes/base.dae
- link j2n6s200_link_finger_1: geometry collision mesh filename=package://ada_description/jaco/meshes/collision_finger_prox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; visual mesh filename=package://ada_description/jaco/meshes/finger_proximal.dae
- link j2n6s200_link_finger_2: geometry collision mesh filename=package://ada_description/jaco/meshes/collision_finger_prox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; visual mesh filename=package://ada_description/jaco/meshes/finger_proximal.dae
- link j2n6s200_link_finger_tip_1: geometry collision mesh filename=package://ada_description/jaco/meshes/collision_finger_dist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; visual mesh filename=package://ada_description/jaco/meshes/finger_distal.dae
- link j2n6s200_link_finger_tip_2: geometry collision mesh filename=package://ada_description/jaco/meshes/collision_finger_dist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; visual mesh filename=package://ada_description/jaco/meshes/finger_distal.dae
Joints:
- removed joint j2n6s200_joint_forque
- removed joint j2n6s200_joint_forque_end_effector
- removed joint j2n6s200_joint_forque_tip
- removed joint j2n6s200_joule
- joint j2n6s200_joint_1: limit lower=-6.28318530718 upper=6.28318530718 effort=2000 velocity=1.0 -> lower=-6.283185307179586 upper=6.283185307179586 effort=2000 velocity=0.8; origin xyz=0 0 0.15675 rpy=0 3.14159265359 0 -> xyz=0 0 0.15675 rpy=0 3.141592653589793 0
- joint j2n6s200_joint_2: limit lower=0.820304748437 upper=5.46288055874 effort=2000 velocity=1.0 -> lower=0.8203047484373349 upper=5.462880558742252 effort=2000 velocity=0.8; origin xyz=0 0.0016 -0.11875 rpy=-1.57079632679 0 3.14159265359 -> xyz=0 0.0016 -0.11875 rpy=-1.5707963267948966 0 3.141592653589793
- joint j2n6s200_joint_3: limit lower=0.331612557879 upper=5.9515727493 effort=2000 velocity=1.0 -> lower=0.33161255787892263 upper=5.951572749300664 effort=2000 velocity=0.8; origin xyz=0 -0.410 0 rpy=0 3.14159265359 0 -> xyz=0 -0.410 0 rpy=0 3.141592653589793 0
- joint j2n6s200_joint_4: limit lower=-6.28318530718 upper=6.28318530718 effort=2000 velocity=1.0 -> lower=-6.283185307179586 upper=6.283185307179586 effort=2000 velocity=0.8; origin xyz=0 0.2073 -0.0114 rpy=-1.57079632679 0 3.14159265359 -> xyz=0 0.2073 -0.0114 rpy=-1.5707963267948966 0 3.141592653589793
- joint j2n6s200_joint_5: limit lower=-6.28318530718 upper=6.28318530718 effort=2000 velocity=1.0 -> lower=-6.283185307179586 upper=6.283185307179586 effort=2000 velocity=0.8; origin xyz=0 -0.03703 -0.06414 rpy=1.0471975512 0 3.14159265359 -> xyz=0 -0.03703 -0.06414 rpy=1.0471975511965976 0 3.141592653589793
- joint j2n6s200_joint_6: limit lower=-6.28318530718 upper=6.28318530718 effort=2000 velocity=1.0 -> lower=-6.283185307179586 upper=6.283185307179586 effort=2000 velocity=0.8; origin xyz=0 -0.03703 -0.06414 rpy=1.0471975512 0 3.14159265359 -> xyz=0 -0.03703 -0.06414 rpy=1.0471975511965976 0 3.141592653589793
- joint j2n6s200_joint_base: limit lower=0 upper=0 effort=2000 velocity=1.0 -> lower=0 upper=0 effort=2000 velocity=0.8
- joint j2n6s200_joint_end_effector: origin xyz=0 0 -0.1600 rpy=3.14159265359 0 0 -> xyz=0 0 -0.1600 rpy=3.141592653589793 0 0
