Commit message: Moved JACO and MICO meshes/robots to subfolders

File: jaco/urdf/ada_with_camera.urdf (robot description, URDF)
Before this commit: robot j2n6s200, 16 links, 15 joints
Links:
- link j2n6s200_joule: geometry collision mesh filename=package://ada_description/jaco/meshes/collision_camera_joul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 scale=0.001 0.001 0.00098; visual mesh filename=package://ada_description/jaco/meshes/camera_joule.dae scale=0.001 0.001 0.001
- link j2n6s200_link_1: geometry collision mesh filename=package://ada_description/jaco/meshes/collision_shoulder.dae; visual mesh filename=package://ada_description/jaco/meshes/ring_big.dae
- link j2n6s200_link_2: geometry collision mesh filename=package://ada_description/jaco/meshes/collision_arm.dae; visual mesh filename=package://ada_description/jaco/meshes/arm.dae
- link j2n6s200_link_3: geometry collision mesh filename=package://ada_description/jaco/meshes/collision_forearm.dae; visual mesh filename=package://ada_description/jaco/meshes/forearm.dae
- link j2n6s200_link_4: geometry collision mesh filename=package://ada_description/jaco/meshes/collision_wrist.dae; visual mesh filename=package://ada_description/jaco/meshes/ring_small.dae
- link j2n6s200_link_5: geometry collision mesh filename=package://ada_description/jaco/meshes/collision_wrist.dae; visual mesh filename=package://ada_description/jaco/meshes/ring_small.dae
- link j2n6s200_link_6: geometry collision mesh filename=package://ada_description/jaco/meshes/collision_hand_2finge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; visual mesh filename=package://ada_description/jaco/meshes/hand_2finger.dae
- link j2n6s200_link_base: geometry collision mesh filename=package://ada_description/jaco/meshes/collision_base.dae; visual mesh filename=package://ada_description/jaco/meshes/base.dae
- link j2n6s200_link_finger_1: geometry collision mesh filename=package://ada_description/jaco/meshes/collision_finger_prox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; visual mesh filename=package://ada_description/jaco/meshes/finger_proximal.dae
- link j2n6s200_link_finger_2: geometry collision mesh filename=package://ada_description/jaco/meshes/collision_finger_prox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; visual mesh filename=package://ada_description/jaco/meshes/finger_proximal.dae
- link j2n6s200_link_finger_tip_1: geometry collision mesh filename=package://ada_description/jaco/meshes/collision_finger_dist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; visual mesh filename=package://ada_description/jaco/meshes/finger_distal.dae
- link j2n6s200_link_finger_tip_2: geometry collision mesh filename=package://ada_description/jaco/meshes/collision_finger_dist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; visual mesh filename=package://ada_description/jaco/meshes/finger_distal.dae
Joints:
- joint j2n6s200_joint_1: limit lower=-6.28318530718 upper=6.28318530718 effort=2000 velocity=0.8 -> lower=-6.283185307179586 upper=6.283185307179586 effort=2000 velocity=0.8; origin xyz=0 0 0.15675 rpy=0 3.14159265359 0 -> xyz=0 0 0.15675 rpy=0 3.141592653589793 0
- joint j2n6s200_joint_2: limit lower=0.820304748437 upper=5.46288055874 effort=2000 velocity=0.8 -> lower=0.8203047484373349 upper=5.462880558742252 effort=2000 velocity=0.8; origin xyz=0 0.0016 -0.11875 rpy=-1.57079632679 0 3.14159265359 -> xyz=0 0.0016 -0.11875 rpy=-1.5707963267948966 0 3.141592653589793
- joint j2n6s200_joint_3: limit lower=0.331612557879 upper=5.9515727493 effort=2000 velocity=0.8 -> lower=0.33161255787892263 upper=5.951572749300664 effort=2000 velocity=0.8; origin xyz=0 -0.410 0 rpy=0 3.14159265359 0 -> xyz=0 -0.410 0 rpy=0 3.141592653589793 0
- joint j2n6s200_joint_4: limit lower=-6.28318530718 upper=6.28318530718 effort=2000 velocity=0.8 -> lower=-6.283185307179586 upper=6.283185307179586 effort=2000 velocity=0.8; origin xyz=0 0.2073 -0.0114 rpy=-1.57079632679 0 3.14159265359 -> xyz=0 0.2073 -0.0114 rpy=-1.5707963267948966 0 3.141592653589793
- joint j2n6s200_joint_5: limit lower=-6.28318530718 upper=6.28318530718 effort=2000 velocity=0.8 -> lower=-6.283185307179586 upper=6.283185307179586 effort=2000 velocity=0.8; origin xyz=0 -0.03703 -0.06414 rpy=1.0471975512 0 3.14159265359 -> xyz=0 -0.03703 -0.06414 rpy=1.0471975511965976 0 3.141592653589793
- joint j2n6s200_joint_6: limit lower=-6.28318530718 upper=6.28318530718 effort=2000 velocity=0.8 -> lower=-6.283185307179586 upper=6.283185307179586 effort=2000 velocity=0.8; origin xyz=0 -0.03703 -0.06414 rpy=1.0471975512 0 3.14159265359 -> xyz=0 -0.03703 -0.06414 rpy=1.0471975511965976 0 3.141592653589793
- joint j2n6s200_joint_end_effector: origin xyz=0 0 -0.1600 rpy=3.14159265359 0 0 -> xyz=0 0 -0.1600 rpy=3.141592653589793 0 0

File: jaco/urdf/ada_with_camera_forque.urdf (robot description, URDF)
Before this commit: robot j2n6s200, 18 links, 17 joints
Links:
- added link j2n6s200_joule; collision mesh filename=package://ada_description/jaco/meshes/collision_camera_joul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 scale=0.001 0.001 0.00098; visual mesh filename=package://ada_description/jaco/meshes/camera_joule.dae scale=0.001 0.001 0.001
- link j2n6s200_forque: geometry collision mesh filename=package://ada_description/jaco/meshes/collision_forque_kino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 scale=0.001 0.001 0.001; visual mesh filename=package://ada_description/jaco/meshes/forque_kinova.dae scale=0.001 0.001 0.001
- link j2n6s200_link_1: geometry collision mesh filename=package://ada_description/jaco/meshes/collision_shoulder.dae; visual mesh filename=package://ada_description/jaco/meshes/ring_big.dae
- link j2n6s200_link_2: geometry collision mesh filename=package://ada_description/jaco/meshes/collision_arm.dae; visual mesh filename=package://ada_description/jaco/meshes/arm.dae
- link j2n6s200_link_3: geometry collision mesh filename=package://ada_description/jaco/meshes/collision_forearm.dae; visual mesh filename=package://ada_description/jaco/meshes/forearm.dae
- link j2n6s200_link_4: geometry collision mesh filename=package://ada_description/jaco/meshes/collision_wrist.dae; visual mesh filename=package://ada_description/jaco/meshes/ring_small.dae
- link j2n6s200_link_5: geometry collision mesh filename=package://ada_description/jaco/meshes/collision_wrist.dae; visual mesh filename=package://ada_description/jaco/meshes/ring_small.dae
- link j2n6s200_link_6: geometry collision mesh filename=package://ada_description/jaco/meshes/collision_hand_2finge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; visual mesh filename=package://ada_description/jaco/meshes/hand_2finger.dae
- link j2n6s200_link_base: geometry collision mesh filename=package://ada_description/jaco/meshes/collision_base.dae; visual mesh filename=package://ada_description/jaco/meshes/base.dae
- link j2n6s200_link_finger_1: geometry collision mesh filename=package://ada_description/jaco/meshes/collision_finger_prox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; visual mesh filename=package://ada_description/jaco/meshes/finger_proximal.dae
- link j2n6s200_link_finger_2: geometry collision mesh filename=package://ada_description/jaco/meshes/collision_finger_prox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; visual mesh filename=package://ada_description/jaco/meshes/finger_proximal.dae
- link j2n6s200_link_finger_tip_1: geometry collision mesh filename=package://ada_description/jaco/meshes/collision_finger_dist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; visual mesh filename=package://ada_description/jaco/meshes/finger_distal.dae
- link j2n6s200_link_finger_tip_2: geometry collision mesh filename=package://ada_description/jaco/meshes/collision_finger_dist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; visual mesh filename=package://ada_description/jaco/meshes/finger_distal.dae
Joints:
- added joint j2n6s200_joule: type fixed, parent j2n6s200_link_6, child j2n6s200_joule, origin xyz=0.06 0.051 0.0140 rpy=1.57079632679 1.57079632679 0, axis 0 0 1, limit lower=-6.28318530718 upper=6.28318530718 effort=2000 velocity=1
- joint j2n6s200_joint_1: limit lower=-6.28318530718 upper=6.28318530718 effort=2000 velocity=0.8 -> lower=-6.283185307179586 upper=6.283185307179586 effort=2000 velocity=0.8; origin xyz=0 0 0.15675 rpy=0 3.14159265359 0 -> xyz=0 0 0.15675 rpy=0 3.141592653589793 0
- joint j2n6s200_joint_2: limit lower=0.820304748437 upper=5.46288055874 effort=2000 velocity=0.8 -> lower=0.8203047484373349 upper=5.462880558742252 effort=2000 velocity=0.8; origin xyz=0 0.0016 -0.11875 rpy=-1.57079632679 0 3.14159265359 -> xyz=0 0.0016 -0.11875 rpy=-1.5707963267948966 0 3.141592653589793
- joint j2n6s200_joint_3: limit lower=0.331612557879 upper=5.9515727493 effort=2000 velocity=0.8 -> lower=0.33161255787892263 upper=5.951572749300664 effort=2000 velocity=0.8; origin xyz=0 -0.410 0 rpy=0 3.14159265359 0 -> xyz=0 -0.410 0 rpy=0 3.141592653589793 0
- joint j2n6s200_joint_4: limit lower=-6.28318530718 upper=6.28318530718 effort=2000 velocity=0.8 -> lower=-6.283185307179586 upper=6.283185307179586 effort=2000 velocity=0.8; origin xyz=0 0.2073 -0.0114 rpy=-1.57079632679 0 3.14159265359 -> xyz=0 0.2073 -0.0114 rpy=-1.5707963267948966 0 3.141592653589793
- joint j2n6s200_joint_5: limit lower=-6.28318530718 upper=6.28318530718 effort=2000 velocity=0.8 -> lower=-6.283185307179586 upper=6.283185307179586 effort=2000 velocity=0.8; origin xyz=0 -0.03703 -0.06414 rpy=1.0471975512 0 3.14159265359 -> xyz=0 -0.03703 -0.06414 rpy=1.0471975511965976 0 3.141592653589793
- joint j2n6s200_joint_6: limit lower=-6.28318530718 upper=6.28318530718 effort=2000 velocity=0.8 -> lower=-6.283185307179586 upper=6.283185307179586 effort=2000 velocity=0.8; origin xyz=0 -0.03703 -0.06414 rpy=1.0471975512 0 3.14159265359 -> xyz=0 -0.03703 -0.06414 rpy=1.0471975511965976 0 3.141592653589793
- joint j2n6s200_joint_end_effector: origin xyz=0 0 -0.1600 rpy=3.14159265359 0 0 -> xyz=0 0 -0.1600 rpy=3.141592653589793 0 0

File: jaco/urdf/ada_with_forque.urdf (robot description, URDF)
Before this commit: robot j2n6s200, 15 links, 14 joints
Links:
- added link j2n6s200_forque; collision mesh filename=package://ada_description/jaco/meshes/collision_forque_kino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 scale=0.001 0.001 0.001; visual mesh filename=package://ada_description/jaco/meshes/forque_kinova.dae scale=0.001 0.001 0.001
- added link j2n6s200_forque_end_effector
- added link j2n6s200_forque_tip
- link j2n6s200_link_1: geometry collision mesh filename=package://ada_description/jaco/meshes/collision_shoulder.dae; visual mesh filename=package://ada_description/jaco/meshes/ring_big.dae
- link j2n6s200_link_2: geometry collision mesh filename=package://ada_description/jaco/meshes/collision_arm.dae; visual mesh filename=package://ada_description/jaco/meshes/arm.dae
- link j2n6s200_link_3: geometry collision mesh filename=package://ada_description/jaco/meshes/collision_forearm.dae; visual mesh filename=package://ada_description/jaco/meshes/forearm.dae
- link j2n6s200_link_4: geometry collision mesh filename=package://ada_description/jaco/meshes/collision_wrist.dae; visual mesh filename=package://ada_description/jaco/meshes/ring_small.dae
- link j2n6s200_link_5: geometry collision mesh filename=package://ada_description/jaco/meshes/collision_wrist.dae; visual mesh filename=package://ada_description/jaco/meshes/ring_small.dae
- link j2n6s200_link_6: geometry collision mesh filename=package://ada_description/jaco/meshes/collision_hand_2finge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; visual mesh filename=package://ada_description/jaco/meshes/hand_2finger.dae
- link j2n6s200_link_base: geometry collision mesh filename=package://ada_description/jaco/meshes/collision_base.dae; visual mesh filename=package://ada_description/jaco/meshes/base.dae
- link j2n6s200_link_finger_1: geometry collision mesh filename=package://ada_description/jaco/meshes/collision_finger_prox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; visual mesh filename=package://ada_description/jaco/meshes/finger_proximal.dae
- link j2n6s200_link_finger_2: geometry collision mesh filename=package://ada_description/jaco/meshes/collision_finger_prox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; visual mesh filename=package://ada_description/jaco/meshes/finger_proximal.dae
- link j2n6s200_link_finger_tip_1: geometry collision mesh filename=package://ada_description/jaco/meshes/collision_finger_dist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; visual mesh filename=package://ada_description/jaco/meshes/finger_distal.dae
- link j2n6s200_link_finger_tip_2: geometry collision mesh filename=package://ada_description/jaco/meshes/collision_finger_dist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; visual mesh filename=package://ada_description/jaco/meshes/finger_distal.dae
Joints:
- added joint j2n6s200_joint_forque: type fixed, parent j2n6s200_end_effector, child j2n6s200_forque, origin xyz=-0.003 -0.0013 0.065 rpy=3.14 0 0, axis 0 0 1, limit lower=0 upper=2 effort=2000 velocity=1
- added joint j2n6s200_joint_forque_end_effector: type fixed, parent j2n6s200_forque, child j2n6s200_forque_end_effector, origin xyz=0.007 0 -0.093 rpy=3.1415 0 1.57075, axis 0 0 0, limit lower=0 upper=0 effort=2000 velocity=1
- added joint j2n6s200_joint_forque_tip: type fixed, parent j2n6s200_forque, child j2n6s200_forque_tip, origin xyz=0.007 0 -0.093 rpy=2.6415 0 1.57075, axis 0 0 0, limit lower=0 upper=0 effort=2000 velocity=1
- joint j2n6s200_joint_1: limit lower=-6.28318530718 upper=6.28318530718 effort=2000 velocity=0.8 -> lower=-6.283185307179586 upper=6.283185307179586 effort=2000 velocity=0.8; origin xyz=0 0 0.15675 rpy=0 3.14159265359 0 -> xyz=0 0 0.15675 rpy=0 3.141592653589793 0
- joint j2n6s200_joint_2: limit lower=0.820304748437 upper=5.46288055874 effort=2000 velocity=0.8 -> lower=0.8203047484373349 upper=5.462880558742252 effort=2000 velocity=0.8; origin xyz=0 0.0016 -0.11875 rpy=-1.57079632679 0 3.14159265359 -> xyz=0 0.0016 -0.11875 rpy=-1.5707963267948966 0 3.141592653589793
- joint j2n6s200_joint_3: limit lower=0.331612557879 upper=5.9515727493 effort=2000 velocity=0.8 -> lower=0.33161255787892263 upper=5.951572749300664 effort=2000 velocity=0.8; origin xyz=0 -0.410 0 rpy=0 3.14159265359 0 -> xyz=0 -0.410 0 rpy=0 3.141592653589793 0
- joint j2n6s200_joint_4: limit lower=-6.28318530718 upper=6.28318530718 effort=2000 velocity=0.8 -> lower=-6.283185307179586 upper=6.283185307179586 effort=2000 velocity=0.8; origin xyz=0 0.2073 -0.0114 rpy=-1.57079632679 0 3.14159265359 -> xyz=0 0.2073 -0.0114 rpy=-1.5707963267948966 0 3.141592653589793
- joint j2n6s200_joint_5: limit lower=-6.28318530718 upper=6.28318530718 effort=2000 velocity=0.8 -> lower=-6.283185307179586 upper=6.283185307179586 effort=2000 velocity=0.8; origin xyz=0 -0.03703 -0.06414 rpy=1.0471975512 0 3.14159265359 -> xyz=0 -0.03703 -0.06414 rpy=1.0471975511965976 0 3.141592653589793
- joint j2n6s200_joint_6: limit lower=-6.28318530718 upper=6.28318530718 effort=2000 velocity=0.8 -> lower=-6.283185307179586 upper=6.283185307179586 effort=2000 velocity=0.8; origin xyz=0 -0.03703 -0.06414 rpy=1.0471975512 0 3.14159265359 -> xyz=0 -0.03703 -0.06414 rpy=1.0471975511965976 0 3.141592653589793
- joint j2n6s200_joint_end_effector: origin xyz=0 0 -0.1600 rpy=3.14159265359 0 0 -> xyz=0 0 -0.1600 rpy=3.141592653589793 0 0
