Commit message: use dummy world link for both sim and real

File: kortex_description/robots/kortex_robot.xacro (robot description, xacro)
@@ -16,13 +16,11 @@
         </xacro:if>
         <!-- Run the macros -->
-        <!-- For gazebo-->
-        <xacro:if value="${sim}">
-            <link name="world" />
-            <joint name="world_to_root" type="fixed">
-                <child link="${prefix}base_link" />
-                <parent link="world" />
-                <origin xyz="0 0 0" rpy="0 0 0" />
-            </joint>
-        </xacro:if>
+        <!-- For gazebo and DART -->
+        <link name="world" />
+        <joint name="world_to_root" type="fixed">
+            <child link="${prefix}base_link" />
+            <parent link="world" />
+            <origin xyz="0 0 0" rpy="0 0 0" />
+        </joint>
         <!-- Load the arm -->
         <xacro:load_arm parent="" dof="${dof}" vision="${vision}" prefix="${prefix}">
