Commit message: Added link named world (+ fixed link between world and base_link) to adhere to DART rules

File: kortex_description/robots/gen3_6dof_vision.urdf (robot description, URDF)
Before this commit: robot gen3_robotiq_2f_85, 22 links, 21 joints
Links:
- added link world
Joints:
- added joint base_link_joint_world: type fixed, parent world, child base_link, origin xyz=0 0 0 rpy=0 0 0, axis 0 0 0, limit lower=0 upper=0 effort=2000 velocity=1.0

Commit message: Rotate Gen3 base to match Jaco2 base, i.e., contorl panel towards +y axis

File: kortex_description/robots/gen3_6dof_vision.urdf (robot description, URDF)
Before this commit: robot gen3_robotiq_2f_85, 23 links, 22 joints
Joints:
- joint world_to_root: origin xyz=0 0 0 rpy=0 0 0 -> xyz=0 0 0 rpy=0 0 -1.57079632679

File: kortex_description/robots/kortex_robot.xacro (robot description, xacro)
@@ -21,5 +21,5 @@
             <child link="${prefix}base_link" />
             <parent link="world" />
-            <origin xyz="0 0 0" rpy="0 0 0" />
+            <origin xyz="0 0 0" rpy="0 0 -1.57079632679" />
         </joint>
         <!-- Load the arm -->
