Commit message: Added forque params

File: kortex_description/robots/gen3_6dof_vision_forque.urdf (robot description, URDF)
Before this commit: robot gen3_robotiq_2f_85, 27 links, 26 joints
Links:
- link forque: mass 0 -> 0.113

File: kortex_description/tools/forque/forque.xacro (robot description, xacro)
@@ -9,6 +9,6 @@
   <link name="${prefix}forque">
     <inertial>
-        <origin xyz="0 0 0" rpy="0 0 0" />
-        <mass value="0" />
+        <origin xyz="0 0 0.091" rpy="0 0 0" />
+        <mass value="0.113" />
         <inertia ixx="0" ixy="0" ixz="0" iyy="0" iyz="0" izz="0" />
     </inertial>
