Commit message: add gen3 xacro changes

File: kortex_description/robots/gen3_robotiq_2f_85.xacro (robot description, xacro)
@@ -7,7 +7,9 @@
     <xacro:arg name="gripper" default="robotiq_2f_85" />
     <xacro:arg name="forque" default="true" />
+    <xacro:arg name="realsense_cam" default="true" />
+    <xacro:arg name="reflect_cam" default="true" />
     <xacro:arg name="sim" default="false" />
     <xacro:arg name="prefix" default="" />
     <xacro:include filename="$(find kortex_description)/robots/kortex_robot.xacro" />
-    <xacro:load_robot arm="$(arg arm)" gripper="$(arg gripper)" forque="$(arg forque)" dof="$(arg dof)" vision="$(arg vision)" sim="$(arg sim)" prefix="$(arg prefix)" />
+    <xacro:load_robot arm="$(arg arm)" gripper="$(arg gripper)" forque="$(arg forque)" reflect_cam="$(arg reflect_cam)" realsense_cam="$(arg realsense_cam)" dof="$(arg dof)" vision="$(arg vision)" sim="$(arg sim)" prefix="$(arg prefix)" />
 </robot>

File: kortex_description/robots/kortex_robot.xacro (robot description, xacro)
@@ -1,5 +1,5 @@
 <?xml version="1.0"?>
 <robot xmlns:xacro="http://ros.org/wiki/xacro">
-    <xacro:macro name="load_robot" params="arm gripper forque dof vision sim prefix">
+    <xacro:macro name="load_robot" params="arm gripper forque reflect_cam realsense_cam dof vision sim prefix">
         <!-- Files to include -->
         <xacro:include filename="$(find kortex_description)/arms/${arm}/${dof}dof/urdf/${arm}_macro.xacro" />
@@ -54,4 +54,15 @@
             <xacro:load_forque parent="${prefix}${last_arm_link}"  prefix="${prefix}"/>
         </xacro:unless>
+        <!-- Load the realsense_camera -->
+        <xacro:unless value="${not realsense_cam}">
+            <!-- last_arm_link is defined in "$(find kortex_description)/arms/${arm}/urdf/${arm}_macro.xacro" -->
+            <xacro:include filename="$(find kortex_description)/tools/realsense_cam/realsense_cam_mount.xacro" />
+            <xacro:load_realsense_cam parent="${prefix}${last_arm_link}"  prefix="${prefix}" reflect="1"/>
+        </xacro:unless>
+        <xacro:unless value="${not reflect_cam}">
+            <!-- last_arm_link is defined in "$(find kortex_description)/arms/${arm}/urdf/${arm}_macro.xacro" -->
+            <xacro:include filename="$(find kortex_description)/tools/realsense_cam/realsense_cam_mount.xacro" />
+            <xacro:load_realsense_cam parent="${prefix}${last_arm_link}"  prefix="${prefix}" reflect="-1"/>
+        </xacro:unless>
         <!-- Load the Gazebo transmissions and gazebo_ros_control plugin -->
         <xacro:if value="${sim}">
