Commit message: add camera link

File: kortex_description/arms/gen3/6dof/urdf/gen3_macro.xacro (robot description, xacro)
@@ -238,4 +238,34 @@
         xyz="0 0 0" />
     </joint>
+    <xacro:if value="${vision}">
+    <link name="${prefix}color_camera_link">
+      <visual>
+        <origin xyz="0 0 0" rpy="0 0 0" />
+        <geometry>
+          <box size="0 0 0" />
+        </geometry>
+      </visual>
+    </link>
+    <link name="${prefix}depth_camera_link">
+      <visual>
+        <origin xyz="0 0 0" rpy="0 0 0" />
+        <geometry>
+          <box size="0 0 0" />
+        </geometry>
+      </visual>
+    </link>
+    <joint name="${prefix}camera_color_joint" type="fixed">
+      <origin xyz="0 0.05639 -0.00305" rpy="0 0 0" />
+      <parent link="${prefix}end_effector_link" />
+      <child link="${prefix}color_camera_link" />
+      <axis xyz="0 0 0" />
+    </joint>
+    <joint name="${prefix}camera_depth_joint" type="fixed">
+      <origin xyz="0.0275 0.06600 -0.00305" rpy="0 0 0" />
+      <parent link="${prefix}end_effector_link" />
+      <child link="${prefix}depth_camera_link" />
+      <axis xyz="0 0 0" />
+    </joint>
+    </xacro:if>
   </xacro:macro>
 </robot>

Commit message: add camera joint changes to xacro and urdf

File: kortex_description/arms/gen3/6dof/urdf/gen3_macro.xacro (robot description, xacro)
@@ -243,5 +243,5 @@
         <origin xyz="0 0 0" rpy="0 0 0" />
         <geometry>
-          <box size="0 0 0" />
+          <box size="0.001 0.001 0.001" />
         </geometry>
       </visual>
@@ -251,5 +251,5 @@
         <origin xyz="0 0 0" rpy="0 0 0" />
         <geometry>
-          <box size="0 0 0" />
+          <box size="0.001 0.001 0.001" />
         </geometry>
       </visual>
@@ -259,5 +259,5 @@
       <parent link="${prefix}end_effector_link" />
       <child link="${prefix}color_camera_link" />
-      <axis xyz="0 0 0" />
+      <axis xyz="0.001 0.001 0.001" />
     </joint>
     <joint name="${prefix}camera_depth_joint" type="fixed">
@@ -265,5 +265,5 @@
       <parent link="${prefix}end_effector_link" />
       <child link="${prefix}depth_camera_link" />
-      <axis xyz="0 0 0" />
+      <axis xyz="0.001 0.001 0.001" />
     </joint>
     </xacro:if>

File: kortex_description/robots/gen3_6dof_vision.urdf (robot description, URDF)
Before this commit: robot gen3_robotiq_2f_85, 23 links, 22 joints
Links:
- link left_inner_finger: geometry collision mesh filename=package://kortex_description/grippers/robotiq_2f_85/meshes/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 scale=0.001 0.001 0.001; visual mesh filename=package://kortex_description/grippers/robotiq_2f_85/meshes/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 scale=0.001 0.001 0.001
- link left_inner_finger_pad: geometry collision box size=0.022 0.00635 0.0375; visual box size=0.022 0.00635 0.0375
- link left_inner_knuckle: geometry collision mesh filename=package://kortex_description/grippers/robotiq_2f_85/meshes/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 scale=0.001 0.001 0.001; visual mesh filename=package://kortex_description/grippers/robotiq_2f_85/meshes/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 scale=0.001 0.001 0.001
- link left_outer_finger: geometry collision mesh filename=package://kortex_description/grippers/robotiq_2f_85/meshes/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 scale=0.001 0.001 0.001; visual mesh filename=package://kortex_description/grippers/robotiq_2f_85/meshes/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 scale=0.001 0.001 0.001
- link left_outer_knuckle: geometry collision mesh filename=package://kortex_description/grippers/robotiq_2f_85/meshes/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 scale=0.001 0.001 0.001; visual mesh filename=package://kortex_description/grippers/robotiq_2f_85/meshes/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 scale=0.001 0.001 0.001
- link right_inner_finger: geometry collision mesh filename=package://kortex_description/grippers/robotiq_2f_85/meshes/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 scale=0.001 0.001 0.001; visual mesh filename=package://kortex_description/grippers/robotiq_2f_85/meshes/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 scale=0.001 0.001 0.001
- link right_inner_finger_pad: geometry collision box size=0.022 0.00635 0.0375; visual box size=0.022 0.00635 0.0375
- link right_inner_knuckle: geometry collision mesh filename=package://kortex_description/grippers/robotiq_2f_85/meshes/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 scale=0.001 0.001 0.001; visual mesh filename=package://kortex_description/grippers/robotiq_2f_85/meshes/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 scale=0.001 0.001 0.001
- link right_outer_finger: geometry collision mesh filename=package://kortex_description/grippers/robotiq_2f_85/meshes/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 scale=0.001 0.001 0.001; visual mesh filename=package://kortex_description/grippers/robotiq_2f_85/meshes/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 scale=0.001 0.001 0.001
- link right_outer_knuckle: geometry collision mesh filename=package://kortex_description/grippers/robotiq_2f_85/meshes/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 scale=0.001 0.001 0.001; visual mesh filename=package://kortex_description/grippers/robotiq_2f_85/meshes/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 scale=0.001 0.001 0.001
Joints:
- removed joint base_link_joint_world
- added joint world_to_root: type fixed, parent world, child base_link, origin xyz=0 0 0 rpy=0 0 0
- joint camera_color_joint: axis 0 0 0 -> 0.001 0.001 0.001
- joint camera_depth_joint: axis 0 0 0 -> 0.001 0.001 0.001
- joint right_outer_knuckle_joint: type revolute -> fixed

Commit message: Switch to camera link

File: kortex_description/arms/gen3/6dof/urdf/gen3_macro.xacro (robot description, xacro)
@@ -239,5 +239,5 @@
     </joint>
     <xacro:if value="${vision}">
-    <link name="${prefix}color_camera_link">
+    <link name="${prefix}camera_link">
       <visual>
         <origin xyz="0 0 0" rpy="0 0 0" />

File: kortex_description/robots/gen3_6dof_vision.urdf (robot description, URDF)
Before this commit: robot gen3_robotiq_2f_85, 23 links, 22 joints
Links:
- removed link color_camera_link
- added link camera_link; visual box size=0.001 0.001 0.001

Commit message: Actually switched to camera link

File: kortex_description/arms/gen3/6dof/urdf/gen3_macro.xacro (robot description, xacro)
@@ -258,5 +258,5 @@
       <origin xyz="0 0.05639 -0.00305" rpy="0 0 0" />
       <parent link="${prefix}end_effector_link" />
-      <child link="${prefix}color_camera_link" />
+      <child link="${prefix}camera_link" />
       <axis xyz="0.001 0.001 0.001" />
     </joint>

File: kortex_description/robots/gen3_6dof_vision.urdf (robot description, URDF)
Before this commit: robot gen3_robotiq_2f_85, 23 links, 22 joints
Joints:
- joint camera_color_joint: child color_camera_link -> camera_link

Commit message: Fixed yaw in camera link

File: kortex_description/arms/gen3/6dof/urdf/gen3_macro.xacro (robot description, xacro)
@@ -256,5 +256,5 @@
     </link>
     <joint name="${prefix}camera_color_joint" type="fixed">
-      <origin xyz="0 0.05639 -0.00305" rpy="0 0 0" />
+      <origin xyz="0 0.05639 -0.00305" rpy="0 0 3.14" />
       <parent link="${prefix}end_effector_link" />
       <child link="${prefix}camera_link" />
@@ -262,5 +262,5 @@
     </joint>
     <joint name="${prefix}camera_depth_joint" type="fixed">
-      <origin xyz="0.0275 0.06600 -0.00305" rpy="0 0 0" />
+      <origin xyz="0.0275 0.06600 -0.00305" rpy="0 0 3.14" />
       <parent link="${prefix}end_effector_link" />
       <child link="${prefix}depth_camera_link" />

File: kortex_description/robots/gen3_6dof_vision.urdf (robot description, URDF)
Before this commit: robot gen3_robotiq_2f_85, 23 links, 22 joints
Joints:
- joint camera_color_joint: origin xyz=0 0.05639 -0.00305 rpy=0 0 0 -> xyz=0 0.05639 -0.00305 rpy=0 0 3.14
- joint camera_depth_joint: origin xyz=0.0275 0.06600 -0.00305 rpy=0 0 0 -> xyz=0.0275 0.06600 -0.00305 rpy=0 0 3.14

Commit message: Corrected rotation between world & base + added forque to urdf

File: kortex_description/arms/gen3/6dof/urdf/gen3_macro.xacro (robot description, xacro)
@@ -11,5 +11,5 @@
       </inertial>
       <visual>
-        <origin xyz="0 0 0" rpy="0 0 0" />
+        <origin xyz="0 0 0" rpy="0 0 -1.5708" />
         <geometry>
           <mesh filename="package://kortex_description/arms/gen3/${dof}dof/meshes/base_link.STL" />
@@ -20,5 +20,5 @@
       </visual>
       <collision>
-        <origin xyz="0 0 0" rpy="0 0 0" />
+        <origin xyz="0 0 0" rpy="0 0 -1.5708" />
         <geometry>
           <mesh filename="package://kortex_description/arms/gen3/${dof}dof/meshes/base_link.STL" />
@@ -49,5 +49,5 @@
     </link>
     <joint name="${prefix}joint_1" type="continuous">
-      <origin xyz="0 0 0.15643" rpy="-3.1416 0.0 0.0" />
+      <origin xyz="0 0 0.15643" rpy="-3.1416 0.0 -1.5708" />
       <parent link="${prefix}base_link" />
       <child link="${prefix}shoulder_link" />

File: kortex_description/robots/gen3_6dof_vision.urdf (robot description, URDF)
Before this commit: robot gen3_robotiq_2f_85, 23 links, 22 joints
Joints:
- joint joint_1: origin xyz=0 0 0.15643 rpy=-3.1416 0.0 0.0 -> xyz=0 0 0.15643 rpy=-3.1416 0.0 -1.5708
- joint world_to_root: origin xyz=0 0 0 rpy=0 0 -1.57079632679 -> xyz=0 0 0 rpy=0 0 0

File: kortex_description/robots/gen3_robotiq_2f_85.xacro (robot description, xacro)
@@ -6,7 +6,8 @@
     <xacro:arg name="vision" default="true" />
     <xacro:arg name="gripper" default="robotiq_2f_85" />
+    <xacro:arg name="forque" default="true" />
     <xacro:arg name="sim" default="false" />
     <xacro:arg name="prefix" default="" />
     <xacro:include filename="$(find kortex_description)/robots/kortex_robot.xacro" />
-    <xacro:load_robot arm="$(arg arm)" gripper="$(arg gripper)" dof="$(arg dof)" vision="$(arg vision)" sim="$(arg sim)" prefix="$(arg prefix)" />
+    <xacro:load_robot arm="$(arg arm)" gripper="$(arg gripper)" forque="$(arg forque)" dof="$(arg dof)" vision="$(arg vision)" sim="$(arg sim)" prefix="$(arg prefix)" />
 </robot>

File: kortex_description/robots/kortex_robot.xacro (robot description, xacro)
@@ -1,5 +1,5 @@
 <?xml version="1.0"?>
 <robot xmlns:xacro="http://ros.org/wiki/xacro">
-    <xacro:macro name="load_robot" params="arm gripper dof vision sim prefix">
+    <xacro:macro name="load_robot" params="arm gripper forque dof vision sim prefix">
         <!-- Files to include -->
         <xacro:include filename="$(find kortex_description)/arms/${arm}/${dof}dof/urdf/${arm}_macro.xacro" />
@@ -21,5 +21,5 @@
             <child link="${prefix}base_link" />
             <parent link="world" />
-            <origin xyz="0 0 0" rpy="0 0 -1.57079632679" />
+            <origin xyz="0 0 0" rpy="0 0 0" />
         </joint>
         <!-- Load the arm -->
@@ -42,4 +42,10 @@
             </joint>
         </xacro:if>
+        <!-- Load the forque -->
+        <xacro:unless value="${not forque}">
+            <!-- last_arm_link is defined in "$(find kortex_description)/arms/${arm}/urdf/${arm}_macro.xacro" -->
+            <xacro:include filename="$(find kortex_description)/tools/forque/forque.xacro" />
+            <xacro:load_forque parent="${prefix}${last_arm_link}"  prefix="${prefix}"/>
+        </xacro:unless>
         <!-- Load the Gazebo transmissions and gazebo_ros_control plugin -->
         <xacro:if value="${sim}">
