Commit message: Currently used inertia

File: kortex_description/arms/gen3/6dof/urdf/gen3_macro.xacro (robot description, xacro)
@@ -116,5 +116,5 @@
       <inertial>
         <origin xyz="-1E-06 0.008486 -0.062937" rpy="0 0 0" />
-        <mass value="0.6781" />
+        <mass value="0.678" />
         <inertia ixx="0.001645" ixy="0" ixz="0" iyy="0.001666" iyz="-0.000234" izz="0.000389" />
       </inertial>
@@ -226,5 +226,11 @@
       <limit effort="9" velocity="1.2218" />
     </joint>
-    <link name="${prefix}end_effector_link" />
+    <link name="${prefix}end_effector_link">
+      <inertial>
+        <origin xyz="0 0 0" rpy="0 0 0" />
+        <mass value="0" />
+        <inertia ixx="0" ixy="0" ixz="0" iyy="0" iyz="0" izz="0" />
+      </inertial>
+    </link>
     <joint
       name="${prefix}end_effector"
@@ -240,4 +246,9 @@
     <xacro:if value="${vision}">
     <link name="${prefix}camera_link">
+      <inertial>
+        <origin xyz="0 0 0" rpy="0 0 0" />
+        <mass value="0" />
+        <inertia ixx="0" ixy="0" ixz="0" iyy="0" iyz="0" izz="0" />
+      </inertial>
       <visual>
         <origin xyz="0 0 0" rpy="0 0 0" />
@@ -248,4 +259,9 @@
     </link>
     <link name="${prefix}depth_camera_link">
+      <inertial>
+        <origin xyz="0 0 0" rpy="0 0 0" />
+        <mass value="0" />
+        <inertia ixx="0" ixy="0" ixz="0" iyy="0" iyz="0" izz="0" />
+      </inertial>
       <visual>
         <origin xyz="0 0 0" rpy="0 0 0" />

File: kortex_description/grippers/robotiq_2f_85/urdf/robotiq_arg2f.xacro (robot description, xacro)
@@ -9,8 +9,13 @@
     </joint>
     <link name="${prefix}robotiq_arg2f_base_link">
-      <inertial>
+<!--       <inertial>
         <origin xyz="8.625E-08 -4.6583E-06 0.03145" rpy="0 0 0" />
         <mass value="0.22652" />
         <inertia ixx="0.00020005" ixy="-4.2442E-10" ixz="-2.9069E-10" iyy="0.00017832" iyz="-3.4402E-08" izz="0.00013478" />
+      </inertial> -->
+      <inertial>
+        <origin xyz="0 0 0" rpy="0 0 0" />
+        <mass value="0" />
+        <inertia ixx="0" ixy="0" ixz="0" iyy="0" iyz="0" izz="0" />
       </inertial>
       <visual>
@@ -32,4 +37,16 @@
       </collision>
     </link>
+    <joint name="${prefix}gripper_inertia_base_joint" type="fixed">
+        <parent link="${parent}"/>
+        <child link="${prefix}inertia_link"/>
+        <origin rpy="0.0 0.0 0.0" xyz="0.0 0.0 0.0"/>
+    </joint>
+    <link name="${prefix}inertia_link">
+        <inertial>
+            <origin xyz="0 0 0.058" rpy="0 0 0"/>
+            <mass value="0.925"/>
+            <inertia ixx="0.000000" ixy="0.000000" ixz="0.000000" iyy="0.000000" iyz="0.000000" izz="0.000000"/>
+        </inertial>
+    </link>
     <gazebo reference="${prefix}robotiq_arg2f_base_link">
       <material>Gazebo/Black</material>

File: kortex_description/grippers/robotiq_2f_85/urdf/robotiq_arg2f_85_model_macro.xacro (robot description, xacro)
@@ -5,8 +5,13 @@
   <xacro:macro name="outer_knuckle" params="prefix fingerprefix stroke">
     <link name="${prefix}${fingerprefix}_outer_knuckle">
-      <inertial>
+<!--       <inertial>
         <origin xyz="-0.000200000000003065 0.0199435877845359 0.0292245259211331" rpy="0 0 0" />
         <mass value="0.00853198276973456" />
         <inertia ixx="2.89328108496468E-06" ixy="-1.57935047237397E-19" ixz="-1.93980378593255E-19" iyy="1.86719750325683E-06" iyz="-1.21858577871576E-06" izz="1.21905238907251E-06" />
+      </inertial> -->
+      <inertial>
+        <origin xyz="0 0 0" rpy="0 0 0" />
+        <mass value="0" />
+        <inertia ixx="0" ixy="0" ixz="0" iyy="0" iyz="0" izz="0" />
       </inertial>
       <visual>
@@ -29,8 +34,13 @@
   <xacro:macro name="outer_finger" params="prefix fingerprefix stroke">
     <link name="${prefix}${fingerprefix}_outer_finger">
-      <inertial>
+<!--       <inertial>
         <origin xyz="0.00030115855001899 0.0373907951953854 -0.0208027427000385" rpy="0 0 0" />
         <mass value="0.022614240507152" />
         <inertia ixx="1.52518312458174E-05" ixy="9.76583423954399E-10" ixz="-5.43838577022588E-10" iyy="6.17694243867776E-06" iyz="6.78636130740228E-06" izz="1.16494917907219E-05" />
+      </inertial> -->
+      <inertial>
+        <origin xyz="0 0 0" rpy="0 0 0" />
+        <mass value="0" />
+        <inertia ixx="0" ixy="0" ixz="0" iyy="0" iyz="0" izz="0" />
       </inertial>
       <visual>
@@ -53,8 +63,13 @@
   <xacro:macro name="inner_knuckle" params="prefix fingerprefix stroke">
     <link name="${prefix}${fingerprefix}_inner_knuckle">
-      <inertial>
+<!--       <inertial>
         <origin xyz="0.000123011831763771 0.0507850843201817 0.00103968640075166" rpy="0 0 0" />
        <mass value="0.0271177346495152" />
         <inertia ixx="2.61910379223783E-05" ixy="-2.43616858946494E-07" ixz="-6.37789906117123E-09" iyy="2.8270243746167E-06" iyz="-5.37200748039765E-07" izz="2.83695868220296E-05" />
+      </inertial> -->
+      <inertial>
+        <origin xyz="0 0 0" rpy="0 0 0" />
+        <mass value="0" />
+        <inertia ixx="0" ixy="0" ixz="0" iyy="0" iyz="0" izz="0" />
       </inertial>
       <visual>
@@ -77,8 +92,13 @@
   <xacro:macro name="inner_finger" params="prefix fingerprefix stroke">
     <link name="${prefix}${fingerprefix}_inner_finger">
-      <inertial>
+<!--       <inertial>
         <origin xyz="0.000299999999999317 0.0160078233491243 -0.0136945669206257" rpy="0 0 0" />
         <mass value="0.0104003125914103" />
         <inertia ixx="2.71909453810972E-06" ixy="1.35402465472579E-21" ixz="-7.1817349065269E-22" iyy="7.69100314106116E-07" iyz="6.74715432769696E-07" izz="2.30315190420171E-06" />
+      </inertial>  -->
+      <inertial>
+        <origin xyz="0 0 0" rpy="0 0 0" />
+        <mass value="0" />
+        <inertia ixx="0" ixy="0" ixz="0" iyy="0" iyz="0" izz="0" />
       </inertial>
       <visual>
@@ -102,4 +122,9 @@
   <xacro:macro name="inner_finger_pad" params="prefix fingerprefix">
     <link name="${prefix}${fingerprefix}_inner_finger_pad">
+      <inertial>
+        <origin xyz="0 0 0" rpy="0 0 0" />
+        <mass value="0" />
+        <inertia ixx="0" ixy="0" ixz="0" iyy="0" iyz="0" izz="0" />
+      </inertial>
       <visual>
         <origin xyz="0 0 0" rpy="0 0 0" />
@@ -161,5 +186,5 @@
   <xacro:include filename="$(find kortex_description)/grippers/robotiq_2f_85/urdf/robotiq_arg2f.xacro" />
   <xacro:macro name="finger_joint" params="prefix">
-    <joint name="${prefix}finger_joint" type="revolute">
+    <joint name="${prefix}finger_joint" type="fixed">
       <origin xyz="0 -0.0306011 0.054904" rpy="0 0 ${pi}"/>
       <parent link="${prefix}robotiq_arg2f_base_link" />
@@ -184,5 +209,11 @@
   <xacro:macro name="robotiq_arg2f_85" params="prefix parent">
     <!-- Tool frame used by the arm -->
-    <link name="${prefix}tool_frame"/>
+    <link name="${prefix}tool_frame">
+      <inertial>
+        <origin xyz="0 0 0" rpy="0 0 0" />
+        <mass value="0" />
+        <inertia ixx="0" ixy="0" ixz="0" iyy="0" iyz="0" izz="0" />
+      </inertial>
+    </link>
     <joint name="${prefix}tool_frame_joint" type="fixed">
         <origin xyz="0 0 0.120" rpy="0 0 0" />

File: kortex_description/robots/gen3_6dof_vision_forque.urdf (robot description, URDF)
Before this commit: robot gen3_robotiq_2f_85, 26 links, 25 joints
Links:
- added link inertia_link, mass 0.925
- link camera_link: mass None -> 0
- link depth_camera_link: mass None -> 0
- link end_effector_link: mass None -> 0
- link forque: mass None -> 0
- link forque_end_effector: mass None -> 0
- link forque_tip: mass None -> 0
- link left_inner_finger: mass 0.0104003125914103 -> 0
- link left_inner_finger_pad: mass None -> 0
- link left_inner_knuckle: mass 0.0271177346495152 -> 0
- link left_outer_finger: mass 0.022614240507152 -> 0
- link left_outer_knuckle: mass 0.00853198276973456 -> 0
- link right_inner_finger: mass 0.0104003125914103 -> 0
- link right_inner_finger_pad: mass None -> 0
- link right_inner_knuckle: mass 0.0271177346495152 -> 0
- link right_outer_finger: mass 0.022614240507152 -> 0
- link right_outer_knuckle: mass 0.00853198276973456 -> 0
- link robotiq_arg2f_base_link: mass 0.22652 -> 0
- link spherical_wrist_1_link: mass 0.6781 -> 0.678
- link tool_frame: mass None -> 0
Joints:
- added joint gripper_inertia_base_joint: type fixed, parent end_effector_link, child inertia_link, origin xyz=0.0 0.0 0.0 rpy=0.0 0.0 0.0
- joint finger_joint: type revolute -> fixed

File: kortex_description/robots/gen3_7dof_vision.urdf (robot description, URDF)
Before this commit: robot gen3_robotiq_2f_85, 23 links, 22 joints
Links:
- removed link bicep_link
- removed link depth_camera_link
- added link camera_color_frame
- added link camera_depth_frame
- added link forque, mass 0; collision mesh filename=package://kortex_description/tools/forque/forque.stl scale=0.001 0.001 0.001; visual mesh filename=package://kortex_description/tools/forque/forque.stl scale=0.001 0.001 0.001
- added link forque_end_effector, mass 0
- added link forque_tip, mass 0
- added link half_arm_1_link, mass 1.1636; collision mesh filename=package://kortex_description/arms/gen3/7dof/meshes/half_arm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; visual mesh filename=package://kortex_description/arms/gen3/7dof/meshes/half_arm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
- added link half_arm_2_link, mass 1.1636; collision mesh filename=package://kortex_description/arms/gen3/7dof/meshes/half_arm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; visual mesh filename=package://kortex_description/arms/gen3/7dof/meshes/half_arm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
- added link inertia_link, mass 0.925
- link base_link: geometry collision mesh filename=package://kortex_description/arms/gen3/7dof/meshes/base_lin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; visual mesh filename=package://kortex_description/arms/gen3/7dof/meshes/base_lin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
- link bracelet_link: geometry collision mesh filename=package://kortex_description/arms/gen3/7dof/meshes/bracelet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; visual mesh filename=package://kortex_description/arms/gen3/7dof/meshes/bracelet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
- link camera_link: geometry 
- link forearm_link: mass 0.93 -> 0.9302; geometry collision mesh filename=package://kortex_description/arms/gen3/7dof/meshes/forearm_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; visual mesh filename=package://kortex_description/arms/gen3/7dof/meshes/forearm_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
- link left_inner_finger: mass 0.0104003125914103 -> 0
- link left_inner_finger_pad: mass None -> 0
- link left_inner_knuckle: mass 0.0271177346495152 -> 0
- link left_outer_finger: mass 0.022614240507152 -> 0
- link left_outer_knuckle: mass 0.00853198276973456 -> 0
- link right_inner_finger: mass 0.0104003125914103 -> 0
- link right_inner_finger_pad: mass None -> 0
- link right_inner_knuckle: mass 0.0271177346495152 -> 0
- link right_outer_finger: mass 0.022614240507152 -> 0
- link right_outer_knuckle: mass 0.00853198276973456 -> 0
- link robotiq_arg2f_base_link: mass 0.22652 -> 0
- link shoulder_link: mass 1.377 -> 1.3773; geometry collision mesh filename=package://kortex_description/arms/gen3/7dof/meshes/shoulder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; visual mesh filename=package://kortex_description/arms/gen3/7dof/meshes/shoulder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
- link spherical_wrist_1_link: geometry collision mesh filename=package://kortex_description/arms/gen3/7dof/meshes/spherica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; visual mesh filename=package://kortex_description/arms/gen3/7dof/meshes/spherica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
- link spherical_wrist_2_link: mass 0.678 -> 0.6781; geometry collision mesh filename=package://kortex_description/arms/gen3/7dof/meshes/spherica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; visual mesh filename=package://kortex_description/arms/gen3/7dof/meshes/spherica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
- link tool_frame: mass None -> 0
Joints:
- removed joint camera_color_joint
- removed joint camera_depth_joint
- added joint camera_module: type fixed, parent end_effector_link, child camera_link, origin xyz=0 0.05639 -0.00305 rpy=3.14159265358979 3.14159265358979 0
- added joint color_module: type fixed, parent end_effector_link, child camera_color_frame, origin xyz=0 0.05639 -0.00305 rpy=3.14159265358979 3.14159265358979 0
- added joint depth_module: type fixed, parent end_effector_link, child camera_depth_frame, origin xyz=0.0275 0.066 -0.00305 rpy=3.14159265358979 3.14159265358979 0
- added joint forque_joint: type fixed, parent end_effector_link, child forque, origin xyz=0.0 0.0 0.11 rpy=0.0 0.0 0
- added joint gripper_inertia_base_joint: type fixed, parent end_effector_link, child inertia_link, origin xyz=0.0 0.0 0.0 rpy=0.0 0.0 0.0
- added joint joint_7: type continuous, parent spherical_wrist_2_link, child bracelet_link, origin xyz=0 -0.10593 -0.00017505 rpy=-1.5708 -5.5511E-17 9.6396E-17, axis 0 0 1, limit effort=9 velocity=1.2218
- added joint joint_forque_end_effector: type fixed, parent forque, child forque_end_effector, origin xyz=0 0.007 0.18 rpy=0 0 0, axis 0 0 0, limit lower=0 upper=0 effort=2000 velocity=1
- added joint joint_forque_tip: type fixed, parent forque, child forque_tip, origin xyz=0.0 0.007 0.18 rpy=-0.5 0 0, axis 0 0 0, limit lower=0 upper=0 effort=2000 velocity=1
- joint end_effector: origin xyz=0 0 -0.0615250000000001 rpy=3.14159265358979 1.09937075168372E-32 3.14159265358979 -> xyz=0 0 -0.0615250000000001 rpy=3.14159265358979 1.09937075168372E-32 0
- joint finger_joint: type revolute -> fixed
- joint joint_1: origin xyz=0 0 0.15643 rpy=-3.1416 0.0 -1.5708 -> xyz=0 0 0.15643 rpy=3.1416 2.7629E-18 -4.9305E-36
- joint joint_2: child bicep_link -> half_arm_1_link; origin xyz=0 0.005375 -0.12838 rpy=1.5708 0.0 0.0 -> xyz=0 0.005375 -0.12838 rpy=1.5708 2.1343E-17 -1.1102E-16
- joint joint_3: child forearm_link -> half_arm_2_link; limit lower=-2.66 upper=2.66 effort=39 velocity=1.3963 -> effort=39 velocity=1.3963; origin xyz=0 -0.41 0 rpy=3.1416 0 0 -> xyz=0 -0.21038 -0.006375 rpy=-1.5708 1.2326E-32 -2.9122E-16; parent bicep_link -> half_arm_1_link; type revolute -> continuous
- joint joint_4: child spherical_wrist_1_link -> forearm_link; limit effort=9 velocity=1.2218 -> lower=-2.66 upper=2.66 effort=39 velocity=1.3963; origin xyz=0 0.20843 -0.006375 rpy=1.5708 0.0 0.0 -> xyz=0 0.006375 -0.21038 rpy=1.5708 -6.6954E-17 -1.6653E-16; parent forearm_link -> half_arm_2_link; type continuous -> revolute
- joint joint_5: child spherical_wrist_2_link -> spherical_wrist_1_link; limit lower=-2.23 upper=2.23 effort=9 velocity=1.2218 -> effort=9 velocity=1.2218; origin xyz=0 -0.00017505 -0.10593 rpy=-1.5708 0.0 0.0 -> xyz=0 -0.20843 -0.006375 rpy=-1.5708 2.2204E-16 -6.373E-17; parent spherical_wrist_1_link -> forearm_link; type revolute -> continuous
- joint joint_6: child bracelet_link -> spherical_wrist_2_link; limit effort=9 velocity=1.2218 -> lower=-2.23 upper=2.23 effort=9 velocity=1.2218; origin xyz=0 0.10593 -0.00017505 rpy=1.5708 0.0 0.0 -> xyz=0 0.00017505 -0.10593 rpy=1.5708 9.2076E-28 -8.2157E-15; parent spherical_wrist_2_link -> spherical_wrist_1_link; type continuous -> revolute

File: kortex_description/robots/kortex_robot.xacro (robot description, xacro)
@@ -34,5 +34,11 @@
         <!-- If no gripper, define tool frame here -->
         <xacro:if value="${not gripper}">
-            <link name="${prefix}tool_frame"/>
+            <link name="${prefix}tool_frame">
+                <inertial>
+                    <origin xyz="0 0 0" rpy="0 0 0" />
+                    <mass value="0" />
+                    <inertia ixx="0" ixy="0" ixz="0" iyy="0" iyz="0" izz="0" />
+                </inertial>
+            </link>
             <joint name="${prefix}tool_frame_joint" type="fixed">
                 <origin xyz="0 0 0" rpy="0 0 0" />

File: kortex_description/tools/forque/forque.xacro (robot description, xacro)
@@ -8,4 +8,9 @@
   </joint>
   <link name="${prefix}forque">
+    <inertial>
+        <origin xyz="0 0 0" rpy="0 0 0" />
+        <mass value="0" />
+        <inertia ixx="0" ixy="0" ixz="0" iyy="0" iyz="0" izz="0" />
+    </inertial>
     <visual>
       <origin xyz="0 0 0" rpy="0 0 0" />
@@ -28,4 +33,9 @@
   </gazebo>
   <link name="${prefix}forque_end_effector">
+    <inertial>
+      <origin xyz="0 0 0" rpy="0 0 0" />
+      <mass value="0" />
+      <inertia ixx="0" ixy="0" ixz="0" iyy="0" iyz="0" izz="0" />
+    </inertial>
   </link>
     <joint name="${prefix}joint_forque_end_effector" type="fixed">
@@ -36,5 +46,10 @@
       <origin rpy="0 0 0" xyz="0 0.007 0.18"/>
     </joint>
-    <link name="${prefix}forque_tip">
+  <link name="${prefix}forque_tip">
+    <inertial>
+      <origin xyz="0 0 0" rpy="0 0 0" />
+      <mass value="0" />
+      <inertia ixx="0" ixy="0" ixz="0" iyy="0" iyz="0" izz="0" />
+    </inertial>
   </link>
     <joint name="${prefix}joint_forque_tip" type="fixed">
