Commit message: Small forque tip shift to correct for bending

File: ada_description/robots_urdf/ada_with_camera_forque.urdf (robot description, URDF)
Before this commit: robot j2n6s200, 19 links, 18 joints
Joints:
- joint j2n6s200_joint_forque_end_effector: origin xyz=0.007 0 -0.093 rpy=3.1415 0 1.57075 -> xyz=0.002 0.005 -0.093 rpy=3.1415 0 1.57075
- joint j2n6s200_joint_forque_tip: origin xyz=0.007 0 -0.093 rpy=2.6415 0 1.57075 -> xyz=0.002 0.005 -0.093 rpy=2.6415 0 1.57075

File: ada_description/robots_urdf/ada_with_forque.urdf (robot description, URDF)
Before this commit: robot j2n6s200, 18 links, 17 joints
Joints:
- joint j2n6s200_joint_forque_end_effector: origin xyz=0.007 0 -0.093 rpy=3.1415 0 1.57075 -> xyz=0.002 0.005 -0.093 rpy=3.1415 0 1.57075
- joint j2n6s200_joint_forque_tip: origin xyz=0.007 0 -0.093 rpy=2.6415 0 1.57075 -> xyz=0.002 0.005 -0.093 rpy=2.6415 0 1.57075

Commit message: Revert "Merge pull request #28 from personalrobotics/egordon/forque_tip_fix"
The core issue that the "fix" was addressing was a camera calibration issue, not a bent fork issue. Now that the camera calibration has been fixed, this change is no longer necessary/desirable.

This reverts commit 607e0925aebdd0729e7a9cf9d5535487759f52b5, reversing
changes made to f649c4e3298c2e6339e71454b2f586efe0835c49.

File: ada_description/robots_urdf/ada_with_camera_forque.urdf (robot description, URDF)
Before this commit: robot j2n6s200, 19 links, 18 joints
Joints:
- joint j2n6s200_joint_forque_end_effector: origin xyz=0.002 0.005 -0.093 rpy=3.1415 0 1.57075 -> xyz=0.007 0 -0.093 rpy=3.1415 0 1.57075
- joint j2n6s200_joint_forque_tip: origin xyz=0.002 0.005 -0.093 rpy=2.6415 0 1.57075 -> xyz=0.007 0 -0.093 rpy=2.6415 0 1.57075

File: ada_description/robots_urdf/ada_with_forque.urdf (robot description, URDF)
Before this commit: robot j2n6s200, 18 links, 17 joints
Joints:
- joint j2n6s200_joint_forque_end_effector: origin xyz=0.002 0.005 -0.093 rpy=3.1415 0 1.57075 -> xyz=0.007 0 -0.093 rpy=3.1415 0 1.57075
- joint j2n6s200_joint_forque_tip: origin xyz=0.002 0.005 -0.093 rpy=2.6415 0 1.57075 -> xyz=0.007 0 -0.093 rpy=2.6415 0 1.57075
